File: UTSVT_Design_Blocks.kicad_blocks/Power_Mux.kicad_block/Power_Mux.kicad_sch (KiCad schematic)
At the start: 6 parts, among them U1 TPS2117DRLR

Commit message: added all footprints + 3d models to design blocks
Parts:
- U1: footprint pretty:TPS2117DRLR -> UTSVT_Power:TPS2117DRLR
