File: UTSVT_Design_Blocks.kicad_blocks/usb_pd_boost.kicad_block/usb_pd_boost.kicad_sch (KiCad schematic)
At the start: 17 parts, among them IC101 TPS55340PWP

Commit message: addressed comments, pls review
Parts:
- removed C107, C108: 4.7uF, symbol Device:C
- removed C109: 1uF, symbol Device:C
- removed D101: 5A, symbol Device:D
- added C11: 1uF, Capacitor_SMD:C_0603_1608Metric, symbol Device:C
- added C2: 10uF, Capacitor_SMD:C_0805_2012Metric, symbol Device:C
- added C7, C9: 4.7uF, Capacitor_SMD:C_0805_2012Metric, symbol Device:C
- added D1: 5A, B540C-13-F:DIOM7959X250N, symbol Device:D_Schottky
- added R4: 0, Resistor_SMD:R_0603_1608Metric, symbol Device:R_US
- added R6: 300k, Resistor_SMD:R_0603_1608Metric, symbol Device:R_US
- added R7: 45.3k, Resistor_SMD:R_0603_1608Metric, symbol Device:R_US
- C1: renamed from C102; footprint (none) -> Capacitor_SMD:C_0805_2012Metric
- C10: renamed from C110; footprint (none) -> Capacitor_SMD:C_0603_1608Metric
- C3: renamed from C103; footprint (none) -> Capacitor_SMD:C_0603_1608Metric
- C4: renamed from C104; value 100nF -> 0.1uF; footprint (none) -> Capacitor_SMD:C_0603_1608Metric
- C5: renamed from C105; value 2.2nF -> 100pF; footprint (none) -> Capacitor_SMD:C_0603_1608Metric
- C6: renamed from C101; value 22nF -> 0.047uF; footprint (none) -> Capacitor_SMD:C_0603_1608Metric; P/N GRM155R71C223KA01D -> MSASU105SB5473KFNA01
- C8: renamed from C106; footprint (none) -> Capacitor_SMD:C_0805_2012Metric
- IC1: renamed from IC101; footprint (none) -> TPS55340PWP:SOP65P640X120-15N
- L1: renamed from L101; footprint (none) -> SDR1307-100ML:SDR1307100ML
- R1: renamed from R104; footprint (none) -> Resistor_SMD:R_0603_1608Metric; P/N CRCW0402187KFKED -> RT0603FRE07187KL
- R2: renamed from R103; footprint (none) -> Resistor_SMD:R_0603_1608Metric
- R3: renamed from R102; value 1.37k -> 2.49k; footprint (none) -> Resistor_SMD:R_0603_1608Metric; P/N CRCW04021K37FKED -> CRCW06032K49FKEAC
- R5: renamed from R101; value 60.4k -> 78.7k; footprint (none) -> Resistor_SMD:R_0603_1608Metric; P/N CRCW040260K4FKED -> RT0603BRE0778K7L
Connections:
- net GND: now also IC1.11 (NC), IC1.6 (SYNC), C11.2, C2.2, C7.2, C9.2, R4.1, R7.2
- net at IC1.1 (SW_1), IC1.2 (SW_2), L1.2: now also D1.2 (A)
- net at IC1.8 (COMP), R3.1: now also C5.1; no longer C4.1
- net at R3.2: now also C4.1; no longer C5.1
- net +24V: no longer names the net of C10.1, C8.1, R1.1
- net +24V: now also C11.1, C7.1, C9.1, D1.1 (K)
- net +9V renamed +USB_PD
- net +USB_PD: now also C2.1, R6.1; no longer IC1.4 (EN)
- new net: IC1.4 (EN), R4.2, R6.2, R7.1
- no-connect marks 1 -> 0
Other:
- note added: "3*4.7uF + 2x1uF > Cout"
- note added: "COMP Network"
- note added: "Dmax = 0.6625 IOUT = 1A fSW = 600kHz COUT_nominal = 3×4.7µF + 2×1µF = 16.1µF Vripple = Dmax*Iout/fsw*Cout Vripple ≈ 68.6 mV"
- note added: "Dmax = 1 - (Vin*efficiency/Vout) Dmax = 1 - ((9*0.9)/24) Dmax = 0.6625"
- note added: "EN pin calculation"
- note added: "Freq Calculation"
- note added: "IOUT_MAX = 9*(5.25-0.994/2)*0.9/24 IOUT_MAX ≈ 1.60A"
- note added: "Input Bypass caps"
- note added: "Note: Pin 15: EP = exposed pad, powerPAD The PowerPAD should be soldered to the AGND. If possible, use thermal vias to connect to internal ground plane for improved power dissipation."
- note added: "Output Bypass Capacitor Calculation"
- note added: "R1 = 187k R2 = 10k fBW ~= fSW/10 to fSW/20 fSW = 600k, fBW = 6.2kHZ Gea = 440 µA/V R3 = 1 / (0.00044 × 0.0508 × 10^(Kps/20)) R3 ~= 2.2k --> 2.49k, common passives"
- note added: "R3 = 2.2k fBW ~= fSW/10 to fSW/20 fSW = 600k, fBW = 6.2kHZ C4 = 0.1uF"
- note added: "Resr = 13.7mΩ Cout = ~16.1uF R3 = 2.2k C5 = 104pF ~= 100pF"
- note added: "Rfreq = 57500 * fsw(kHz)^-1.03 Rfreq = 57000 * (600)^-1.03 Rfreq = 78.4k"
- note added: "Ven = 8V Ven = Vin * Rbot/(Rtop+Rbottom) Ratio of Rbottom/(Rtop+Rbottom)=1.08/8≈0.135 Standardized Passives: ratio = 45.3k / (300k + 45.3k) = 45.3k / 300k ≈ 0.131 Vin,on = 1.08 / 0.131 ≈ 8.24V Vin,off = 0.92/0.131 = 7V R4 as a DNP 0 ohm resistor to force boost off in some cases"
- note added: "Vin(min) = 9V Vout = 24V L = 10uH fSW = 600kHZ nest = 90% = 0.9 ILIM = 5.25A (data sheet pg 16)"
- note added: "Vout/Iout calculations"
- note added: "ΔIL = 9*0.6625/(10µH*600kHz) ΔIL = 5.9625 / 6 ΔIL ≈ 0.994A"
- note added: "ΔIL = VIN × D / (L × fSW) ΔIL = 9 × 0.6625 / (10µH × 600kHz) ΔIL ≈ 0.994A ICIN,rms = ΔIL / √12 ICIN,rms = 0.994 / 3.464 ICIN,rms ≈ 0.287A Allowing 50mV ripple CIN ≥ 0.994 / (4 × 600k × 0.05) CIN ≥ 8.3µF effective"
- moved on the sheet: C1, C10, C3, C4, C5, C6, C8, L1, R3, R5

Commit message: for review again
Parts:
- added TP1: Vin, symbol Connector:TestPoint
- added TP2: EN, symbol Connector:TestPoint
- added TP3: GND, symbol Connector:TestPoint
- added TP4: Vout, symbol Connector:TestPoint
- added TP5: SW, symbol Connector:TestPoint
- added TP6: FB, symbol Connector:TestPoint
- added TP7: SS, symbol Connector:TestPoint
- added TP8: COMP, symbol Connector:TestPoint
- C1, C2: LCSC P/N (none) -> C3840574
- C10, C11: LCSC P/N (none) -> C559769; P/N MLASU168SB5105KTNA01 -> CC0603KRX7R9BB105
- C3: value 100nF -> 0.1uF; LCSC P/N (none) -> C6666325
- C4: LCSC P/N (none) -> C6666325
- C5: LCSC P/N (none) -> C14665; P/N CL21C222JBFNNNE -> CC0603JRNPO9BN101
- C6: LCSC P/N (none) -> C107093; P/N MSASU105SB5473KFNA01 -> CC0603KRX7R9BB473
- C7, C8, C9: LCSC P/N (none) -> C6962403
- D1: LCSC P/N (none) -> C72264
- IC1: LCSC P/N (none) -> C43862
- L1: LCSC P/N (none) -> C49672242
- R1: LCSC P/N (none) -> C2085290; P/N RT0603FRE07187KL -> CRCW0603187KFKEA
- R2: LCSC P/N (none) -> C843841
- R3: value 2.49k -> 2.55k; LCSC P/N (none) -> C844547; P/N CRCW06032K49FKEAC -> CRCW06032K55FKEA
- R4: LCSC P/N (none) -> C95177; P/N CRCW06030000Z0EE -> RC0603JR-070RL
- R5: LCSC P/N (none) -> C3961380; P/N RT0603BRE0778K7L -> RC0603DR-0778K7L
- R6: value 300k -> 301k; LCSC P/N (none) -> C273742; P/N CRCW0603300KJNTA -> RC0603FR-07301KL
- R7: value 45.3k -> 51.1k; LCSC P/N (none) -> C844575; P/N CRCW060345K3FKEAHP -> CRCW060351K1FKEA
Connections:
- net +USB_PD: now also TP1.1
- net GND: now also TP3.1
- net +24V: now reaches C10.1, C11.1, C7.1, C8.1, C9.1, D1.1 (K), R1.1
- net +24V: now also TP4.1
- net at IC1.4 (EN), R4.2, R6.2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: now also TP2.1
- net at C6.1, IC1.5 (SS): now also TP7.1
- net at D1.2 (A), IC1.1 (SW_1), IC1.2 (SW_2)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: now also TP5.1
- net at C5.1, IC1.8 (COMP), R3.1: now also TP8.1
- net at IC1.9 (FB), R1.2, R2.1: now also TP6.1
- no-connect marks 0 -> 1
Other:
- note added: "- 8V-20V to 24.00V @ 1A-2.25A - Internal 5-A, 40-V low-side MOSFET switch"
- note added: "9V: IOUT_MAX = 9*(5.25-0.994/2)*0.9/24 IOUT_MAX ≈ 1.60A (IC Limit) IOUT (90% efficient) = 1A 20V: IOUT_MAX ≈ 3.62A (IC Limit) Real (90% efficient) = 2.25A IOUT = 54W / 24V IOUT ≈ 2.25A 95% → 57W out → 24V @ 2.38A"
- note added: "C7 = Vin bypass caps"
- note added: "Vin = 9V Dmax = 1 - (Vin*efficiency/Vout) Dmax = 1 - ((9*0.9)/24) Dmax = 0.6625 Vin = 20V D = 1 - (VIN × η / VOUT) D = 1 - (20 × 0.9 / 24) D = 1 - 0.75 D = 0.25"
- note added: "Vin(min) = 9V or 20V Vout = 24V L = 10uH fSW = 600kHZ nest = 90% = 0.9 ILIM = 5.25A (data sheet pg 16)"
- note added: "Vout = 1.229V * (R1/R2 + 1) Vout = 1.229V * (Rsh/Rsl + 1) Vout = 1.229V * (187k/10k + 1) Vout = 24.2113 volts"
- note added: "ΔIL = 9*0.6625/(10µH*600kHz) ΔIL = 5.9625 / 6 ΔIL ≈ 0.994A (9V) ΔIL ≈ 0.833A (20V)"
- note removed: "- 8V-20V to 24.00V @ 1A - Internal 5-A, 40-V low-side MOSFET switch"
- note removed: "Dmax = 1 - (Vin*efficiency/Vout) Dmax = 1 - ((9*0.9)/24) Dmax = 0.6625"
- note removed: "IOUT_MAX = 9*(5.25-0.994/2)*0.9/24 IOUT_MAX ≈ 1.60A"
- note removed: "Vin(min) = 9V Vout = 24V L = 10uH fSW = 600kHZ nest = 90% = 0.9 ILIM = 5.25A (data sheet pg 16)"
- note removed: "Vout = 1.229V * (R1/R2 + 1) Vout = 1.229V * (Rsh/Rsl + 1) Vout = 1.229V * (R(104)/R(103) + 1) Vout = 1.229V * (187k/10k + 1) Vout = 24.2113 volts"
- note removed: "ΔIL = 9*0.6625/(10µH*600kHz) ΔIL = 5.9625 / 6 ΔIL ≈ 0.994A"

Commit message: addressedyurp
Parts:
- removed TP3: GND, symbol Connector:TestPoint
- C5: value 100pF -> 0.1nF
- R3: value 2.55k -> 2.21k; LCSC P/N C844547 -> C705758; P/N CRCW06032K55FKEA -> RT0603BRD072K21L
Connections:
- net GND renamed AGND
- net AGND: no longer IC1.12 (PGND_1), IC1.13 (PGND_2), IC1.14 (PGND_3), IC1.15 (EP)
- new net PGND: IC1.12 (PGND_1), IC1.13 (PGND_2), IC1.14 (PGND_3), IC1.15 (EP)
- no-connect marks 1 -> 0
Changed lines of the file:
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@@
 	(rectangle
 		(start 17.272 34.036)
-		(end 282.448 105.918)
+		(end 247.396 105.918)
 		(stroke
 			(width 0)
@@
 	)
 	(rectangle
-		(start 17.526 112.522)
-		(end 77.216 147.32)
+		(start 17.526 108.966)
+		(end 77.216 143.764)
 		(stroke
 			(width 0)
@@
 	)
 	(rectangle
-		(start 17.78 149.86)
-		(end 77.47 195.58)
+		(start 17.78 146.304)
+		(end 77.47 192.024)
 		(stroke
 			(width 0)
@@
 	(text "C7 = Vin bypass caps"
 		(exclude_from_sim no)
-		(at 30.734 193.294 0)
+		(at 30.734 189.738 0)
 		(effects
 			(font
@@
 	(text "ΔIL = VIN × D / (L × fSW)\nΔIL = 9 × 0.6625 / (10µH × 600kHz)\nΔIL ≈ 0.994A\n\nICIN,rms = ΔIL / √12\nICIN,rms = 0.994 / 3.464\nICIN,rms ≈ 0.287A\n\nAllowing 50mV ripple\nCIN ≥ 0.994 / (4 × 600k × 0.05)\nCIN ≥ 8.3µF effective"
 		(exclude_from_sim no)
-		(at 19.304 178.562 0)
+		(at 19.304 175.006 0)
 		(effects
 			(font
@@
 	(text "Input Bypass caps"
 		(exclude_from_sim no)
-		(at 27.94 151.892 0)
+		(at 27.94 148.336 0)
 		(effects
 			(font
@@
 	(text "EN pin calculation"
 		(exclude_from_sim no)
-		(at 27.686 114.808 0)
+		(at 27.686 111.252 0)
 		(effects
 			(font
@@
 	(text "Ven = 8V\nVen = Vin * Rbot/(Rtop+Rbottom)\nRatio of Rbottom/(Rtop+Rbottom)=1.08/8≈0.135\n\nStandardized Passives:\nratio = 45.3k / (300k + 45.3k) = 45.3k / 300k ≈ 0.131\n\nVin,on = 1.08 / 0.131 ≈ 8.24V\n\nVin,off = 0.92/0.131 = 7V\n\nR4 as a DNP 0 ohm resistor to force \nboost off in some cases"
 		(exclude_from_sim no)
-		(at 18.796 130.302 0)
+		(at 18.796 126.746 0)
 		(effects
 			(font
@@
 	)
 	(junction
+		(at 83.82 92.71)
+		(diameter 0)
+		(color 0 0 0 0)
+	)
+	(junction
 		(at 156.21 74.93)
 		(diameter 0)
@@
 	)
 	(junction
+		(at 83.82 83.82)
+		(diameter 0)
+		(color 0 0 0 0)
+	)
+	(junction
 		(at 53.34 97.79)
 		(diameter 0)
@@
 	)
 	(junction
+		(at 83.82 81.28)
+		(diameter 0)
+		(color 0 0 0 0)
+	)
+	(junction
 		(at 57.15 97.79)
 		(diameter 0)
@@
 	)
 	(junction
-		(at 83.82 97.79)
-		(diameter 0)
-		(color 0 0 0 0)
-	)
-	(junction
 		(at 76.2 55.88)
 		(diameter 0)
@@
 	)
 	(junction
-		(at 83.82 83.82)
-		(diameter 0)
-		(color 0 0 0 0)
-	)
-	(junction
 		(at 184.15 97.79)
 		(diameter 0)
@@
 	)
 	(junction
-		(at 91.44 97.79)
-		(diameter 0)
-		(color 0 0 0 0)
-	)
-	(junction
-		(at 83.82 81.28)
-		(diameter 0)
-		(color 0 0 0 0)
-	)
-	(junction
 		(at 217.17 55.88)
 		(diameter 0)
@@
 		(color 0 0 0 0)
 	)
-	(no_connect
-		(at 73.66 107.95)
-	)
 	(wire
 		(pts
@@
 	(wire
 		(pts
-			(xy 114.3 66.04) (xy 114.3 68.58)
+			(xy 83.82 81.28) (xy 83.82 83.82)
 		)
 		(stroke
@@
 	(wire
 		(pts
-			(xy 158.75 62.23) (xy 158.75 55.88)
+			(xy 114.3 66.04) (xy 114.3 68.58)
 		)
 		(stroke
@@
 	(wire
 		(pts
-			(xy 74.93 74.93) (xy 74.93 97.79)
+			(xy 158.75 62.23) (xy 158.75 55.88)
 		)
 		(stroke
@@
 	(wire
 		(pts
-			(xy 83.82 78.74) (xy 83.82 81.28)
+			(xy 74.93 74.93) (xy 74.93 97.79)
 		)
 		(stroke
@@
 	(wire
 		(pts
-			(xy 74.93 97.79) (xy 83.82 97.79)
-		)
-		(stroke
-			(width 0)
-			(type default)
-		)
-	)
-	(wire
-		(pts
 			(xy 76.2 55.88) (xy 95.25 55.88)
 		)
@@
 	(wire
 		(pts
-			(xy 120.65 97.79) (xy 139.7 97.79)
+			(xy 83.82 92.71) (xy 99.06 92.71)
 		)
 		(stroke
@@
 	(wire
 		(pts
-			(xy 83.82 81.28) (xy 83.82 83.82)
+			(xy 120.65 97.79) (xy 139.7 97.79)
 		)
 		(stroke
@@
 	(wire
 		(pts
+			(xy 83.82 78.74) (xy 83.82 81.28)
+		)
+		(stroke
+			(width 0)
+			(type default)
+		)
+	)
+	(wire
+		(pts
 			(xy 158.75 69.85) (xy 158.75 74.93)
 		)
@@
 	(wire
 		(pts
-			(xy 83.82 97.79) (xy 91.44 97.79)
+			(xy 74.93 97.79) (xy 99.06 97.79)
 		)
 		(stroke
@@
 	(wire
 		(pts
-			(xy 99.06 92.71) (xy 99.06 97.79)
-		)
-		(stroke
-			(width 0)
-			(type default)
-		)
-	)
-	(wire
-		(pts
 			(xy 156.21 74.93) (xy 158.75 74.93)
 		)
@@
 	(wire
 		(pts
-			(xy 91.44 97.79) (xy 99.06 97.79)
+			(xy 158.75 55.88) (xy 184.15 55.88)
 		)
 		(stroke
@@
 	(wire
 		(pts
-			(xy 158.75 55.88) (xy 184.15 55.88)
+			(xy 83.82 83.82) (xy 83.82 92.71)
 		)
 		(stroke
@@
 	(wire
 		(pts
-			(xy 83.82 83.82) (xy 83.82 97.79)
+			(xy 83.82 92.71) (xy 83.82 95.25)
 		)
 		(stroke
@@
 	)
 	(image
-		(at 31.75 159.258)
+		(at 31.75 155.702)
 		(scale 0.158454)
 		(data "iVBORw0KGgoAAAANSUhEUgAAA3IAAAGICAYAAAAEQdK3AAAMTmlDQ1BJQ0MgUHJvZmlsZQAASImV"
@@
 		)
 	)
-	(hierarchical_label "GND"
+	(hierarchical_label "AGND"
 		(shape input)
 		(at 99.06 101.6 0)
@@
 		)
 	)
+	(hierarchical_label "PGND"
+		(shape input)
+		(at 83.82 95.25 0)
+		(effects
+			(font
+				(size 1.27 1.27)
+			)
+			(justify left)
+		)
+	)
 	(symbol
 		(lib_id "Device:C")
@@
 			)
 		)
-		(property "Value" "100pF"
+		(property "Value" "0.1nF"
 			(at 123.698 88.9 0)
 			(effects
@@
 			)
 		)
-		(property "Value" "2.55k"
+		(property "Value" "2.21k"
 			(at 130.81 82.042 90)
 			(effects
@@
 			)
 		)
-		(property "P/N" "CRCW06032K55FKEA"
+		(property "P/N" "RT0603BRD072K21L"
 			(at 130.81 77.47 90)
 			(effects
@@
 			)
 		)
-		(property "LCSC P/N" "C844547"
+		(property "LCSC P/N" "C705758"
 			(at 130.81 77.47 90)
 			(effects
@@
 					(unit 1)
 				)
-			)
-		)
-	)
-	(symbol
-		(lib_id "Connector:TestPoint")
-		(at 91.44 97.79 180)
-		(unit 1)
-		(exclude_from_sim no)
-		(in_bom yes)
-		(on_board yes)
-		(dnp no)
-		(fields_autoplaced yes)
-		(property "Reference" "TP3"
-			(at 93.98 99.8219 0)
-			(effects
-				(font
-					(size 1.27 1.27)
-				)
-				(justify right)
-				(hide yes)
-			)
-		)
-		(property "Value" "GND"
-			(at 93.98 102.3619 0)
-			(effects
-				(font
-					(size 1.27 1.27)
-				)
-				(justify right)
-			)
-		)
-		(property "Footprint" ""
-			(at 86.36 97.79 0)
-			(effects
-				(font
-					(size 1.27 1.27)
-				)
-				(hide yes)
-			)
-		)
-		(property "Datasheet" "~"
-			(at 86.36 97.79 0)
-			(effects
-				(font
-					(size 1.27 1.27)
-				)
-				(hide yes)
-			)
-		)
-		(property "Description" "test point"
-			(at 91.44 97.79 0)
-			(effects
-				(font
-					(size 1.27 1.27)
-				)
-				(hide yes)
-			)
-		)
-		(property "LCSC P/N" ""
-			(at 91.44 97.79 0)
-			(effects
-				(font
-					(size 1.27 1.27)
-				)
-				(hide yes)
-			)
-		)
-		(pin "1"
-		)
-		(instances
-			(project "usb_pd_boost"
-				(path "/2b3ef5e9-c974-44d2-8d28-cda88c383d02"
-					(reference "TP3")
-					(unit 1)
-				)
