File: UTSVT_Design_Blocks.kicad_blocks/usb_pd_boost.kicad_block/usb_pd_boost.kicad_sch (KiCad schematic)
At the start: 28 parts, among them IC1 TPS55340PWP

Commit message: reviewed and ready
Parts:
- TP1, TP2, TP4, TP5, TP6, TP7, TP8: footprint (none) -> TestPoint:TestPoint_THTPad_D3.0mm_Drill1.5mm
Other:
- note added: "Ven = 8V Ven = Vin * Rbot/(Rtop+Rbottom) Ratio of Rbottom/(Rtop+Rbottom)=1.08/8≈0.135 Standardized Passives: ratio = 51.1k / (300k + 51.1k) = 0.145 Vin,on = 1.08 / 0.145 ≈ 7.42V Vin,off = 0.92/0.131 = 7V R4 as a DNP 0 ohm resistor to force boost off in some cases"
- note removed: "Ven = 8V Ven = Vin * Rbot/(Rtop+Rbottom) Ratio of Rbottom/(Rtop+Rbottom)=1.08/8≈0.135 Standardized Passives: ratio = 45.3k / (300k + 45.3k) = 45.3k / 300k ≈ 0.131 Vin,on = 1.08 / 0.131 ≈ 8.24V Vin,off = 0.92/0.131 = 7V R4 as a DNP 0 ohm resistor to force boost off in some cases"
Changed lines of the file:
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@@
 		)
 	)
-	(text "Ven = 8V\nVen = Vin * Rbot/(Rtop+Rbottom)\nRatio of Rbottom/(Rtop+Rbottom)=1.08/8≈0.135\n\nStandardized Passives:\nratio = 45.3k / (300k + 45.3k) = 45.3k / 300k ≈ 0.131\n\nVin,on = 1.08 / 0.131 ≈ 8.24V\n\nVin,off = 0.92/0.131 = 7V\n\nR4 as a DNP 0 ohm resistor to force \nboost off in some cases"
+	(text "Ven = 8V\nVen = Vin * Rbot/(Rtop+Rbottom)\nRatio of Rbottom/(Rtop+Rbottom)=1.08/8≈0.135\n\nStandardized Passives:\nratio = 51.1k / (300k + 51.1k) = 0.145\n\nVin,on = 1.08 / 0.145 ≈ 7.42V\n\nVin,off = 0.92/0.131 = 7V\n\nR4 as a DNP 0 ohm resistor to force \nboost off in some cases"
 		(exclude_from_sim no)
 		(at 18.796 126.746 0)
@@
 	)
 	(hierarchical_label "+24V"
-		(shape input)
+		(shape output)
 		(at 237.49 55.88 0)
 		(effects
@@
 			)
 		)
-		(property "Footprint" ""
+		(property "Footprint" "TestPoint:TestPoint_THTPad_D3.0mm_Drill1.5mm"
 			(at 66.04 67.31 0)
 			(effects
@@
 			)
 		)
-		(property "Footprint" ""
+		(property "Footprint" "TestPoint:TestPoint_THTPad_D3.0mm_Drill1.5mm"
 			(at 161.29 74.93 0)
 			(effects
@@
 			)
 		)
-		(property "Footprint" ""
+		(property "Footprint" "TestPoint:TestPoint_THTPad_D3.0mm_Drill1.5mm"
 			(at 110.49 77.47 0)
 			(effects
@@
 			)
 		)
-		(property "Footprint" ""
+		(property "Footprint" "TestPoint:TestPoint_THTPad_D3.0mm_Drill1.5mm"
 			(at 62.23 69.85 0)
 			(effects
@@
 			)
 		)
-		(property "Footprint" ""
+		(property "Footprint" "TestPoint:TestPoint_THTPad_D3.0mm_Drill1.5mm"
 			(at 231.14 55.88 0)
 			(effects
@@
 			)
 		)
-		(property "Footprint" ""
+		(property "Footprint" "TestPoint:TestPoint_THTPad_D3.0mm_Drill1.5mm"
 			(at 40.64 55.88 0)
 			(effects
@@
 			)
 		)
-		(property "Footprint" ""
+		(property "Footprint" "TestPoint:TestPoint_THTPad_D3.0mm_Drill1.5mm"
 			(at 121.92 55.88 0)
 			(effects
