File: 48pinMCU_DesignBlock/48pinMCU_DesignBlock.kicad_sch (KiCad schematic)
At the start: 26 parts, among them SW1 SW_SPDT, Y1 Crystal

Commit message: review lil shah
Parts:
- added C11: 0.1uF, Capacitor_SMD:C_0603_1608Metric_Pad1.08x0.95mm_HandSolder, symbol Device:C
- added C15: 100nF, Capacitor_SMD:C_0603_1608Metric_Pad1.08x0.95mm_HandSolder, symbol Device:C
- added FB1, FB4: FerriteBead, Capacitor_SMD:C_0603_1608Metric_Pad1.08x0.95mm_HandSolder, symbol Device:FerriteBead
- H1, H2, H3, H4: now left out of the parts list
- gave numbers to parts that had none: 2
Connections:
- net PA13 is gone; now on net SWCLK: U1.37 (PA13)
- net PA14 is gone; now on net SWDIO: U1.38 (PA14)
- net +3.3V: now also C11.1, FB4.1; no longer U1.20 (VREF+)
- net GND: now also C11.2, FB1.1; no longer U1.19 (VSSA)
- net GNDA: now also U1.19 (VSSA), C15.2, FB1.2
- net VDDA: now also U1.20 (VREF+), C15.1, FB4.2
- net PA11 renamed USB_DM
- net PA12 renamed USB_DP
Other:
- note added: "Main Flash (user code)"
- note added: "Power Source Filtering/Isolation"
- note added: "Reset BTN + Boot SW"
- note added: "Serial Wire Communication"
- note added: "Sys Memory (bootloader)"
- note added: "VBAT Decoupling Cap"
- note added: "VDDA Seperation"
- note removed: "+24v -> +3.3v Buck (?)"
- note removed: "Boot SW + Reset BTN"
- note removed: "Power Source Filtering"
- note removed: "Serial Wire Flashing - TODO"
- note removed: "USB Flashing (?)"
- moved on the sheet: C1, C10, C12, C13, C14, C2, C3, C4, C5, C6, C7, C8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
