File: UTSVT_Design_Blocks.kicad_blocks/USB_PD.kicad_block/USB_PD.kicad_sch (KiCad schematic)
At the start: 32 parts, among them Q1 SI7997DP-T1-GE3, Q2 Q_Dual_PMOS_G1S2G2D2S1D1, Q3 SI7997DP-T1-GE3, Q4 Q_Dual_PMOS_G1S2G2D2S1D1, U1 CYPD3177-24LQ

Commit message: symbol library yea
Parts:
- removed D3: LED, LED_SMD:LED_0603_1608Metric_Pad1.05x0.95mm_HandSolder, symbol Device:LED
- removed Q1, Q3: SI7997DP-T1-GE3, Components:SI7288DPT1GE3, symbol SI7997DP:SI7997DP-T1-GE3
- removed Q2, Q4: Q_Dual_PMOS_G1S2G2D2S1D1, symbol Transistor_FET:Q_Dual_PMOS_G1S2G2D2S1D1
- removed R10: 4.7k, Resistor_SMD:R_0603_1608Metric_Pad0.98x0.95mm_HandSolder, symbol Device:R_Small
- added C3, C5: 1uF, Capacitor_SMD:C_0603_1608Metric_Pad1.08x0.95mm_HandSolder, symbol Device:C_Small
- added Q1, Q2: SI7997DP-T1-GE3, SI7288DPT1GE3, symbol USB_PD_Symbols:SI7997DP-T1-GE3
- renumbered C2 to C1, C1 to C2, C3 to C4, C4 to C6, C5 to C7, C6 to C8, C7 to C9, D4 to D1, D6 to D2, D2 to D3, D5 to D4, R8 to R10, R4 to R11, R9 to R12, R14 to R13, R15 to R14, R3 to R2, R13 to R3, R11 to R4, R2 to R5, R12 to R6, R5 to R7, R6 to R8, R7 to R9
Connections:
- net 5V_OUT: now also C5.1, Q2.10 (D2), Q2.12 (D2), Q2.5 (D2), Q2.6 (D2)
- net GND: no longer U1.9 (FAULT)
- net VBUS_IN: now also C3.1, Q1.11 (D1), Q1.7 (D1), Q1.8 (D1), Q1.9 (D1), Q2.11 (D1), Q2.7 (D1), Q2.8 (D1), Q2.9 (D1)
- net VBUS_OUT: now also Q1.10 (D2), Q1.12 (D2), Q1.5 (D2), Q1.6 (D2)
- net H_G1: no longer names the net of C2.2, C4.2, D4.2 (A), R11.1, R3.1, R5.1
- net H_G1: now also Q1.2 (G1), Q1.4 (G2)
- net H_S: no longer names the net of D4.1 (K), R11.2
- net H_S: now also Q1.1 (S1), Q1.3 (S2)
- net L_G1: no longer names the net of D3.2 (A), R4.1, R6.1
- net L_G1: now also C3.2, C5.2, Q2.2 (G1), Q2.4 (G2)
- net L_S: no longer names the net of D3.1 (K)
- net L_S: now also Q2.1 (S1), Q2.3 (S2)
- no-connect marks 0 -> 1
Other:
- note added: "D1"
- note added: "D2"
- note added: "Dual Package PMOS VDS: 30V RDS: 5.5mOhm at VGS = -10V Max VGS: +- 20V"
- note added: "G1"
- note added: "G2"
- note added: "Gate is 0V (FET on) or VBUS_IN (FET off)"
- note added: "Gates is 0V (FET on) or floating (FET off)"
- note added: "S"
- note removed: "Gates are driven to 0V (FET on) or VBUS_IN (FET off)"
- note removed: "Power Path PFETs"
- note removed: "Status: ON if good"
- note removed: "VDS: 30V RDS: 5.5mOhm at VGS = -10V Max VGS: +- 20V"
- moved on the sheet: C2, C4, D3, D4, R11, R3, R4, R5, R6
