File: UTSVT_Design_Blocks.kicad_blocks/3V3Buck.kicad_block/3V3Buck.kicad_sch (KiCad schematic)
At the start: 9 parts, among them U1 LMR51635XDDCR

Commit message: buck
Parts:
- removed C5: C_Small, symbol Device:C_Small
- C3: LCSC # C1607 -> (none); LCSC P/N (none) -> C1607; P/N (none) -> 581-0603YC225MAT2A
- C4: footprint Capacitor_SMD:C_0603_1608Metric_Pad1.08x0.95mm_HandSolder -> Resistor_SMD:R_0201_0603Metric_Pad0.64x0.40mm_HandSolder; LCSC # C440198 -> (none); LCSC P/N (none) -> C14663
- C6, C7: footprint Capacitor_SMD:C_1210_3225Metric_Pad1.33x2.70mm_HandSolder -> Capacitor_SMD:C_0805_2012Metric_Pad1.18x1.45mm_HandSolder; LCSC P/N (none) -> C16780; P/N 81-GGM32ED70J476KE2L -> 581-08056D476MAT2A
- L1: footprint Inductor_SMD:L_Sunlord_SWPA4020S -> Inductor_SMD:L_Cenker_CKCS252010; LCSC # C88247 -> (none); LCSC P/N (none) -> C354546; P/N (none) -> 710-78439346056
- R6: value 31.6 -> 31.6k; footprint Resistor_SMD:R_0805_2012Metric_Pad1.20x1.40mm_HandSolder -> Resistor_SMD:R_0201_0603Metric_Pad0.64x0.40mm_HandSolder; LCSC P/N (none) -> C25967; P/N 603-RT0805FRE0731R6L -> 652-CR0603FX-3162ELF
- R7: footprint Capacitor_SMD:C_0402_1005Metric_Pad0.74x0.62mm_HandSolder -> Resistor_SMD:R_0201_0603Metric_Pad0.64x0.40mm_HandSolder; LCSC # C11660 -> (none); LCSC P/N (none) -> C22772; P/N (none) -> 603-RT0603DRE0710K2L
- U1: LCSC P/N (none) -> C42432812; P/N (none) -> 595-LMR51635XDDCR
Connections:
- net V_in renamed V_in_24V
- net V_out renamed V_out_3V3
Other:
- moved on the sheet: C4, C6, C7, L1, R6, R7
