File: UTSVT_Design_Blocks.kicad_blocks/3V3Buck.kicad_block/3V3Buck.kicad_sch (KiCad schematic)
At the start: 12 parts, among them U1 LMR51635XDDCR

Commit message: added all footprints + 3d models to design blocks
Parts:
- U1: footprint breh:DDC0006A-MFG -> UTSVT_ICs:DDC0006A-MFG
- renumbered C3 to C1, C4 to C2, C6 to C3, C7 to C4, R6 to R1, R7 to R2, TP18 to TP?, TP19 to TP?, TP17 to TP?, TP16 to TP?
