File: UTSVT_Design_Blocks.kicad_blocks/48PinMCU.kicad_block/48PinMCU.kicad_sch (KiCad schematic)
At the start: 29 parts, among them J1 Conn_01x04, SW1 SW_SPDT, U1 STM32G431CBT6, Y1 Crystal

Commit message: imma sleep now
Parts:
- C1, C2: LCSC P/N (none) -> C92670
- C10, C11, C14, C4, C5, C6, C7, C8, C9: LCSC P/N (none) -> C14663
- C12, C13, C15: LCSC P/N (none) -> C15849
- C3: LCSC P/N (none) -> C440198
- D16: LCSC P/N (none) -> PESD15VL1BA
- FB1, FB4: LCSC P/N (none) -> C354394
- H1, H2, H3, H4, J1, SW1: LCSC P/N (none) -> -
- R1, R2: LCSC P/N (none) -> C25804
- U1: LCSC P/N (none) -> C529355
- Y1: LCSC P/N (none) -> C144380
