File: UTSVT_Design_Blocks.kicad_blocks/48PinMCU.kicad_block/48PinMCU.kicad_sch (KiCad schematic)
At the start: 29 parts, among them J1 SWD_Header, SW1 SW_SPDT, SW2 Reset, U1 STM32G431CBT6, Y1 Crystal

Commit message: added all footprints + 3d models to design blocks
Parts:
- SW2: footprint UTSVT_Special:BootSW -> UTSVT_Special:TL3365AF180QG
