File: UTSVT_Design_Blocks.kicad_blocks/ESP32.kicad_block/ESP32.kicad_sch (KiCad schematic)
At the start: 21 parts, among them J1 USB_C_Receptacle_USB2.0_16P, SW1 BOOT Switch, SW2 RESET Button, U1 ESP32-C6-MINI-1/U

Commit message: switched to SathSwitch
Parts:
- SW1: P/N JS202011SCQN -> 450406020024
Changed lines of the file:
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@@
 			)
 		)
-		(property "Datasheet" "ckswitches.com/media/1422/js.pdf"
+		(property "Datasheet" "https://www.we-online.com/components/products/datasheet/450406020024.pdf"
 			(at 118.11 41.91 0)
 			(effects
@@
 			)
 		)
-		(property "P/N" "JS202011SCQN"
+		(property "P/N" "450406020024 "
 			(at 118.11 34.29 0)
 			(effects
