File: UTSVT_Design_Blocks.kicad_blocks/ESP32.kicad_block/ESP32.kicad_sch (KiCad schematic)
At the start: 21 parts, among them J1 USB_C_Receptacle_USB2.0_16P, SW1 BOOT Switch, SW2 RESET Button, U1 ESP32-C6-MINI-1

Commit message: oops I forgot a couple things
Parts:
- SW2: footprint utsvt_esp32:TL3365AF180QG -> UTSVT_Special:TL3365AF180QG
Changed lines of the file:
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@@
 			)
 		)
-		(property "Footprint" "utsvt_esp32:TL3365AF180QG"
+		(property "Footprint" "UTSVT_Special:TL3365AF180QG"
 			(at 167.64 27.94 0)
 			(effects
