File: UTSVT_Design_Blocks.kicad_blocks/3.3V Buck.kicad_block/3.3V Buck.kicad_sch (KiCad schematic)
At the start: 8 parts, among them U1 LMR51635XDDCR

Commit message: made changes
Parts:
- C3: footprint Capacitor_SMD:C_0603_1608Metric_Pad1.08x0.95mm_HandSolder -> Capacitor_SMD:C_0805_2012Metric_Pad1.18x1.45mm_HandSolder; LCSC P/N C1607 -> C1771; P/N 581-0603YC225MAT2A -> 963-T21GCB7225MTPA1J
- C6, C7: footprint Capacitor_SMD:C_0805_2012Metric_Pad1.18x1.45mm_HandSolder -> Capacitor_SMD:C_1210_3225Metric_Pad1.33x2.70mm_HandSolder; LCSC P/N C16780 -> C77101; P/N 581-08056D476MAT2A -> 963-MLAST32MAB5476MP
Changed lines of the file:
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@@
 			)
 		)
-		(property "Footprint" "Capacitor_SMD:C_0805_2012Metric_Pad1.18x1.45mm_HandSolder"
+		(property "Footprint" "Capacitor_SMD:C_1210_3225Metric_Pad1.33x2.70mm_HandSolder"
 			(at 166.37 85.09 0)
 			(effects
@@
 			)
 		)
-		(property "P/N" "581-08056D476MAT2A"
+		(property "P/N" "963-MLAST32MAB5476MP"
 			(at 166.37 85.09 0)
 			(effects
@@
 			)
 		)
-		(property "LCSC P/N" "C16780"
+		(property "LCSC P/N" "C77101"
 			(at 166.37 85.09 0)
 			(effects
@@
 			)
 		)
-		(property "Footprint" "Capacitor_SMD:C_0805_2012Metric_Pad1.18x1.45mm_HandSolder"
+		(property "Footprint" "Capacitor_SMD:C_1210_3225Metric_Pad1.33x2.70mm_HandSolder"
 			(at 154.94 85.09 0)
 			(effects
@@
 			)
 		)
-		(property "P/N" "581-08056D476MAT2A"
+		(property "P/N" "963-MLAST32MAB5476MP"
 			(at 154.94 85.09 0)
 			(effects
@@
 			)
 		)
-		(property "LCSC P/N" "C16780"
+		(property "LCSC P/N" "C77101"
 			(at 154.94 85.09 0)
 			(effects
@@
 			)
 		)
-		(property "Footprint" "Capacitor_SMD:C_0603_1608Metric_Pad1.08x0.95mm_HandSolder"
+		(property "Footprint" "Capacitor_SMD:C_0805_2012Metric_Pad1.18x1.45mm_HandSolder"
 			(at 77.47 81.28 0)
 			(effects
@@
 			)
 		)
-		(property "LCSC P/N" "C1607"
+		(property "LCSC P/N" "C1771"
 			(at 77.47 81.28 0)
 			(effects
@@
 			)
 		)
-		(property "P/N" "581-0603YC225MAT2A"
+		(property "P/N" "963-T21GCB7225MTPA1J"
 			(at 77.47 81.28 0)
 			(effects
