File: UTSVT_Design_Blocks.kicad_blocks/5VBuck.kicad_block/5VBuck.kicad_sch (KiCad schematic)
At the start: 12 parts, among them U1 LMR51635XDDCR

Commit message: updated resistor footprint from 0201 to 0603 (#56)
* updated resistor footprint from 0201 to 0603

* updated wrong resistor value
Parts:
- R1, R2: footprint Resistor_SMD:R_0201_0603Metric_Pad0.64x0.40mm_HandSolder -> Resistor_SMD:R_0603_1608Metric
Changed lines of the file:
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@@
 			)
 			(project "5VBuck"
+				(path "/ad6c7df0-eb90-4670-9aa8-3e2007aefc2d/4ce3c563-64ba-4b6e-b334-e3956b5d5a33"
+					(reference "L1")
+					(unit 1)
+				)
 				(path "/ad6c7df0-eb90-4670-9aa8-3e2007aefc2d/c59a1097-f91e-4d56-b57d-869363ca5893"
 					(reference "L1")
@@
 			)
 		)
-		(property "Footprint" "Resistor_SMD:R_0201_0603Metric_Pad0.64x0.40mm_HandSolder"
+		(property "Footprint" "Resistor_SMD:R_0603_1608Metric"
 			(at 167.64 50.8 0)
 			(effects
@@
 			)
 			(project "5VBuck"
+				(path "/ad6c7df0-eb90-4670-9aa8-3e2007aefc2d/4ce3c563-64ba-4b6e-b334-e3956b5d5a33"
+					(reference "R2")
+					(unit 1)
+				)
 				(path "/ad6c7df0-eb90-4670-9aa8-3e2007aefc2d/c59a1097-f91e-4d56-b57d-869363ca5893"
 					(reference "R2")
@@
 			)
 			(project "5VBuck"
+				(path "/ad6c7df0-eb90-4670-9aa8-3e2007aefc2d/4ce3c563-64ba-4b6e-b334-e3956b5d5a33"
+					(reference "C1")
+					(unit 1)
+				)
 				(path "/ad6c7df0-eb90-4670-9aa8-3e2007aefc2d/c59a1097-f91e-4d56-b57d-869363ca5893"
 					(reference "C1")
@@
 		(instances
 			(project "PowerPath"
+				(path "/ad6c7df0-eb90-4670-9aa8-3e2007aefc2d/4ce3c563-64ba-4b6e-b334-e3956b5d5a33"
+					(reference "TP6")
+					(unit 1)
+				)
 				(path "/ad6c7df0-eb90-4670-9aa8-3e2007aefc2d/c59a1097-f91e-4d56-b57d-869363ca5893"
 					(reference "TP6")
@@
 			)
 			(project "5VBuck"
+				(path "/ad6c7df0-eb90-4670-9aa8-3e2007aefc2d/4ce3c563-64ba-4b6e-b334-e3956b5d5a33"
+					(reference "C2")
+					(unit 1)
+				)
 				(path "/ad6c7df0-eb90-4670-9aa8-3e2007aefc2d/c59a1097-f91e-4d56-b57d-869363ca5893"
 					(reference "C2")
@@
 			)
 			(project "5VBuck"
+				(path "/ad6c7df0-eb90-4670-9aa8-3e2007aefc2d/4ce3c563-64ba-4b6e-b334-e3956b5d5a33"
+					(reference "U1")
+					(unit 1)
+				)
 				(path "/ad6c7df0-eb90-4670-9aa8-3e2007aefc2d/c59a1097-f91e-4d56-b57d-869363ca5893"
 					(reference "U1")
@@
 		(instances
 			(project ""
+				(path "/ad6c7df0-eb90-4670-9aa8-3e2007aefc2d/4ce3c563-64ba-4b6e-b334-e3956b5d5a33"
+					(reference "TP5")
+					(unit 1)
+				)
 				(path "/ad6c7df0-eb90-4670-9aa8-3e2007aefc2d/c59a1097-f91e-4d56-b57d-869363ca5893"
 					(reference "TP5")
@@
 			)
 			(project "5VBuck"
+				(path "/ad6c7df0-eb90-4670-9aa8-3e2007aefc2d/4ce3c563-64ba-4b6e-b334-e3956b5d5a33"
+					(reference "#FLG01")
+					(unit 1)
+				)
 				(path "/ad6c7df0-eb90-4670-9aa8-3e2007aefc2d/c59a1097-f91e-4d56-b57d-869363ca5893"
 					(reference "#FLG01")
@@
 		(instances
 			(project "PowerPath"
+				(path "/ad6c7df0-eb90-4670-9aa8-3e2007aefc2d/4ce3c563-64ba-4b6e-b334-e3956b5d5a33"
+					(reference "TP8")
+					(unit 1)
+				)
 				(path "/ad6c7df0-eb90-4670-9aa8-3e2007aefc2d/c59a1097-f91e-4d56-b57d-869363ca5893"
 					(reference "TP8")
@@
 			)
 			(project "5VBuck"
+				(path "/ad6c7df0-eb90-4670-9aa8-3e2007aefc2d/4ce3c563-64ba-4b6e-b334-e3956b5d5a33"
+					(reference "C4")
+					(unit 1)
+				)
 				(path "/ad6c7df0-eb90-4670-9aa8-3e2007aefc2d/c59a1097-f91e-4d56-b57d-869363ca5893"
 					(reference "C4")
@@
 			)
 			(project "5VBuck"
+				(path "/ad6c7df0-eb90-4670-9aa8-3e2007aefc2d/4ce3c563-64ba-4b6e-b334-e3956b5d5a33"
+					(reference "#FLG02")
+					(unit 1)
+				)
 				(path "/ad6c7df0-eb90-4670-9aa8-3e2007aefc2d/c59a1097-f91e-4d56-b57d-869363ca5893"
 					(reference "#FLG02")
@@
 			)
 		)
-		(property "Footprint" "Resistor_SMD:R_0201_0603Metric_Pad0.64x0.40mm_HandSolder"
+		(property "Footprint" "Resistor_SMD:R_0603_1608Metric"
 			(at 167.64 43.18 0)
 			(effects
@@
 			)
 			(project "5VBuck"
+				(path "/ad6c7df0-eb90-4670-9aa8-3e2007aefc2d/4ce3c563-64ba-4b6e-b334-e3956b5d5a33"
+					(reference "R1")
+					(unit 1)
+				)
 				(path "/ad6c7df0-eb90-4670-9aa8-3e2007aefc2d/c59a1097-f91e-4d56-b57d-869363ca5893"
 					(reference "R1")
@@
 			)
 			(project "5VBuck"
+				(path "/ad6c7df0-eb90-4670-9aa8-3e2007aefc2d/4ce3c563-64ba-4b6e-b334-e3956b5d5a33"
+					(reference "C3")
+					(unit 1)
+				)
 				(path "/ad6c7df0-eb90-4670-9aa8-3e2007aefc2d/c59a1097-f91e-4d56-b57d-869363ca5893"
 					(reference "C3")
@@
 		(instances
 			(project "PowerPath"
-				(path "/ad6c7df0-eb90-4670-9aa8-3e2007aefc2d/c59a1097-f91e-4d56-b57d-869363ca5893"
+				(path "/ad6c7df0-eb90-4670-9aa8-3e2007aefc2d/4ce3c563-64ba-4b6e-b334-e3956b5d5a33"
 					(reference "TP7")
+					(unit 1)
+				)
+				(path "/ad6c7df0-eb90-4670-9aa8-3e2007aefc2d/c59a1097-f91e-4d56-b57d-869363ca5893"
+					(reference "TP7")
