File: UTSVT_Design_Blocks.kicad_blocks/5VBuck.kicad_block/5VBuck.kicad_sch (KiCad schematic)
At the start: 12 parts, among them U4 LMR51635XDDCR

Commit message: jk real 48 pin fixes
Parts:
- L1: renamed from L2; LCSC P/N C354639 -> C54563397; P/N CKCS8040-10uH/M -> SRN8040-101M
- renumbered C12 to C1, C13 to C2, C14 to C3, C15 to C4, R32 to R1, R33 to R2, TP15 to TP?, TP13 to TP?, TP16 to TP?, TP14 to TP?, U4 to U1
Changed lines of the file:
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@@
 		(on_board yes)
 		(dnp no)
-		(property "Reference" "L2"
+		(property "Reference" "L1"
 			(at 106.68 48.514 90)
 			(effects
@@
 			)
 		)
-		(property "LCSC P/N" "C354639"
+		(property "LCSC P/N" "C54563397"
 			(at 106.68 46.99 90)
 			(effects
@@
 			)
 		)
-		(property "P/N" "CKCS8040-10uH/M"
+		(property "P/N" "SRN8040-101M"
 			(at 106.68 46.99 90)
 			(effects
@@
 				)
 			)
-			(project "5VBuck"
-				(path "/ad6c7df0-eb90-4670-9aa8-3e2007aefc2d/ae63f0a9-78b8-4efb-b2ee-a2699a24d705"
-					(reference "L2")
-					(unit 1)
-				)
-			)
 		)
 	)
@@
 		(dnp no)
 		(fields_autoplaced yes)
-		(property "Reference" "R33"
+		(property "Reference" "R2"
 			(at 170.18 49.5299 0)
 			(effects
@@
 				)
 			)
-			(project "5VBuck"
-				(path "/ad6c7df0-eb90-4670-9aa8-3e2007aefc2d/ae63f0a9-78b8-4efb-b2ee-a2699a24d705"
-					(reference "R33")
-					(unit 1)
-				)
-			)
 		)
 	)
@@
 		(dnp no)
 		(fields_autoplaced yes)
-		(property "Reference" "C12"
+		(property "Reference" "C1"
 			(at 40.64 45.7262 0)
 			(effects
@@
 				)
 			)
-			(project "5VBuck"
-				(path "/ad6c7df0-eb90-4670-9aa8-3e2007aefc2d/ae63f0a9-78b8-4efb-b2ee-a2699a24d705"
-					(reference "C12")
-					(unit 1)
-				)
-			)
 		)
 	)
@@
 		(on_board yes)
 		(dnp no)
-		(property "Reference" "TP15"
+		(property "Reference" "TP?"
 			(at 184.15 80.5179 0)
 			(effects
@@
 		)
 		(instances
+			(project "5VBuck"
+				(path "/1a7db697-3478-4f8f-a838-af5608c43196"
+					(reference "TP?")
+					(unit 1)
+				)
+			)
 			(project "PowerPath"
 				(path "/ad6c7df0-eb90-4670-9aa8-3e2007aefc2d/ae63f0a9-78b8-4efb-b2ee-a2699a24d705"
@@
 		(on_board yes)
 		(dnp no)
-		(property "Reference" "C13"
+		(property "Reference" "C2"
 			(at 100.838 40.64 0)
 			(effects
@@
 				)
 			)
-			(project "5VBuck"
-				(path "/ad6c7df0-eb90-4670-9aa8-3e2007aefc2d/ae63f0a9-78b8-4efb-b2ee-a2699a24d705"
-					(reference "C13")
-					(unit 1)
-				)
-			)
 		)
 	)
@@
 		(dnp no)
 		(fields_autoplaced yes)
-		(property "Reference" "U4"
+		(property "Reference" "U1"
 			(at 73.66 31.75 0)
 			(effects
@@
 				)
 			)
-			(project "5VBuck"
-				(path "/ad6c7df0-eb90-4670-9aa8-3e2007aefc2d/ae63f0a9-78b8-4efb-b2ee-a2699a24d705"
-					(reference "U4")
-					(unit 1)
-				)
-			)
 		)
 	)
@@
 		(on_board yes)
 		(dnp no)
-		(property "Reference" "TP13"
+		(property "Reference" "TP?"
 			(at 171.45 80.5179 0)
 			(effects
@@
 		)
 		(instances
+			(project "5VBuck"
+				(path "/1a7db697-3478-4f8f-a838-af5608c43196"
+					(reference "TP?")
+					(unit 1)
+				)
+			)
 			(project ""
 				(path "/ad6c7df0-eb90-4670-9aa8-3e2007aefc2d/ae63f0a9-78b8-4efb-b2ee-a2699a24d705"
@@
 		(dnp no)
 		(fields_autoplaced yes)
-		(property "Reference" "#FLG010"
+		(property "Reference" "#FLG01"
 			(at 93.98 40.005 0)
 			(effects
@@
 				)
 			)
-			(project "5VBuck"
-				(path "/ad6c7df0-eb90-4670-9aa8-3e2007aefc2d/ae63f0a9-78b8-4efb-b2ee-a2699a24d705"
-					(reference "#FLG010")
-					(unit 1)
-				)
-			)
 		)
 	)
@@
 		(on_board yes)
 		(dnp no)
-		(property "Reference" "TP16"
+		(property "Reference" "TP?"
 			(at 184.15 93.2179 0)
 			(effects
@@
 		)
 		(instances
+			(project "5VBuck"
+				(path "/1a7db697-3478-4f8f-a838-af5608c43196"
+					(reference "TP?")
+					(unit 1)
+				)
+			)
 			(project "PowerPath"
 				(path "/ad6c7df0-eb90-4670-9aa8-3e2007aefc2d/ae63f0a9-78b8-4efb-b2ee-a2699a24d705"
@@
 		(dnp no)
 		(fields_autoplaced yes)
-		(property "Reference" "C15"
+		(property "Reference" "C4"
 			(at 129.54 49.5362 0)
 			(effects
@@
 				)
 			)
-			(project "5VBuck"
-				(path "/ad6c7df0-eb90-4670-9aa8-3e2007aefc2d/ae63f0a9-78b8-4efb-b2ee-a2699a24d705"
-					(reference "C15")
-					(unit 1)
-				)
-			)
 		)
 	)
@@
 		(on_board yes)
 		(dnp no)
-		(property "Reference" "#FLG011"
+		(property "Reference" "#FLG02"
 			(at 93.98 45.085 0)
 			(effects
@@
 				)
 			)
-			(project "5VBuck"
-				(path "/ad6c7df0-eb90-4670-9aa8-3e2007aefc2d/ae63f0a9-78b8-4efb-b2ee-a2699a24d705"
-					(reference "#FLG011")
-					(unit 1)
-				)
-			)
 		)
 	)
@@
 		(dnp no)
 		(fields_autoplaced yes)
-		(property "Reference" "R32"
+		(property "Reference" "R1"
 			(at 170.18 41.9099 0)
 			(effects
@@
 				)
 			)
-			(project "5VBuck"
-				(path "/ad6c7df0-eb90-4670-9aa8-3e2007aefc2d/ae63f0a9-78b8-4efb-b2ee-a2699a24d705"
-					(reference "R32")
-					(unit 1)
-				)
-			)
 		)
 	)
@@
 		(dnp no)
 		(fields_autoplaced yes)
-		(property "Reference" "C14"
+		(property "Reference" "C3"
 			(at 118.11 49.5362 0)
 			(effects
@@
 				)
 			)
-			(project "5VBuck"
-				(path "/ad6c7df0-eb90-4670-9aa8-3e2007aefc2d/ae63f0a9-78b8-4efb-b2ee-a2699a24d705"
-					(reference "C14")
-					(unit 1)
-				)
-			)
 		)
 	)
@@
 		(on_board yes)
 		(dnp no)
-		(property "Reference" "TP14"
+		(property "Reference" "TP?"
 			(at 171.45 93.2179 0)
 			(effects
@@
 		)
 		(instances
+			(project "5VBuck"
+				(path "/1a7db697-3478-4f8f-a838-af5608c43196"
+					(reference "TP?")
+					(unit 1)
+				)
+			)
 			(project "PowerPath"
 				(path "/ad6c7df0-eb90-4670-9aa8-3e2007aefc2d/ae63f0a9-78b8-4efb-b2ee-a2699a24d705"
@@
 		)
 	)
+	(sheet_instances
+		(path "/"
+			(page "1")
+		)
+	)
+	(embedded_fonts no)
 )

Commit message: added all footprints + 3d models to design blocks
Parts:
- L1: footprint Inductor_SMD:L_TDK_VLP8040 -> UTSVT_Passives:SRN80408R2Y
- U1: footprint utsvt_ics:DDC0006A-MFG -> UTSVT_ICs:DDC0006A-MFG
Changed lines of the file:
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@@
 			)
 		)
-		(property "Footprint" "Inductor_SMD:L_TDK_VLP8040"
+		(property "Footprint" "UTSVT_Passives:SRN80408R2Y"
 			(at 106.68 46.99 0)
 			(effects
@@
 			)
 		)
-		(property "Footprint" "utsvt_ics:DDC0006A-MFG"
+		(property "Footprint" "UTSVT_ICs:DDC0006A-MFG"
 			(at 58.42 41.91 0)
 			(effects

Commit message: oops I forgot a couple things
Parts:
- L1: footprint UTSVT_Passives:SRN80408R2Y -> UTSVT_Passives:SRN8040-101M
Changed lines of the file:
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@@
 			)
 		)
-		(property "Footprint" "UTSVT_Passives:SRN80408R2Y"
+		(property "Footprint" "UTSVT_Passives:SRN8040-101M"
 			(at 106.68 46.99 0)
 			(effects
