File: UTSVT_Design_Blocks.kicad_blocks/100PinMCU.kicad_block/100PinMCU.kicad_sch (KiCad schematic)
At the start: 28 parts, among them J1 SWD_Header_02x02, U2 STM32G491VET6, Y1 Crystal

Commit message: more fixes... imma sleep tho
Parts:
- U2: value STM32G491VET6 -> STM32G491VET6_1; footprint LQFP_491VET6_STM:LQFP_491VET6_STM -> UTSVT_ICs:LQFP_491VET6_STM; symbol 100PinMCU:STM32G491VET6 -> utsvt_ics:STM32G491VET6_1
Changed lines of the file:
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@@
 	)
 	(symbol
-		(lib_id "100PinMCU:STM32G491VET6")
+		(lib_id "utsvt_ics:STM32G491VET6_1")
 		(at 57.785 38.735 0)
 		(unit 1)
@@
 			)
 		)
-		(property "Value" "STM32G491VET6"
+		(property "Value" "STM32G491VET6_1"
 			(at 93.345 31.115 0)
 			(effects
@@
 			)
 		)
-		(property "Footprint" "LQFP_491VET6_STM:LQFP_491VET6_STM"
+		(property "Footprint" "UTSVT_ICs:LQFP_491VET6_STM"
 			(at 57.785 38.735 0)
 			(effects

Commit message: added all footprints + 3d models to design blocks
Parts:
- D2: footprint (none) -> LED_SMD:LED_0201_0603Metric
- FB1, FB2: footprint (none) -> Capacitor_SMD:C_0603_1608Metric_Pad1.08x0.95mm_HandSolder
- J1: footprint 878320406:CONN04_878320406_MOL -> UTSVT_Connectors:SWD_Conn
- R2, R4, R5: footprint (none) -> Resistor_SMD:R_0603_1608Metric_Pad0.98x0.95mm_HandSolder
- Reset1: footprint TL3365AF180QG:TL3365AF180QG -> UTSVT_Special:TL3365AF180QG
- S1: footprint 450406020024:450406020024 -> UTSVT_Special:BootSW
- Y1: footprint Crystal:Crystal_SMD_Abracon_ABM3-2Pin_5.0x3.2mm -> UTSVT_Passives:Crystal_SMD_Abracon_ABM3-2Pin_5.0x3.2mm
Changed lines of the file:
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@@
 			)
 		)
-		(property "Footprint" "Crystal:Crystal_SMD_Abracon_ABM3-2Pin_5.0x3.2mm"
+		(property "Footprint" "UTSVT_Passives:Crystal_SMD_Abracon_ABM3-2Pin_5.0x3.2mm"
 			(at 36.195 59.055 0)
 			(effects
@@
 			)
 		)
-		(property "Footprint" ""
+		(property "Footprint" "Resistor_SMD:R_0603_1608Metric_Pad0.98x0.95mm_HandSolder"
 			(at 233.426 116.459 90)
 			(effects
@@
 			)
 		)
-		(property "Footprint" ""
+		(property "Footprint" "Resistor_SMD:R_0603_1608Metric_Pad0.98x0.95mm_HandSolder"
 			(at 138.684 28.321 90)
 			(effects
@@
 			)
 		)
-		(property "Footprint" ""
+		(property "Footprint" "Resistor_SMD:R_0603_1608Metric_Pad0.98x0.95mm_HandSolder"
 			(at 138.684 30.861 90)
 			(effects
@@
 			)
 		)
-		(property "Footprint" ""
+		(property "Footprint" "Capacitor_SMD:C_0603_1608Metric_Pad1.08x0.95mm_HandSolder"
 			(at 98.425 187.833 90)
 			(effects
@@
 			)
 		)
-		(property "Footprint" ""
+		(property "Footprint" "LED_SMD:LED_0201_0603Metric"
 			(at 232.41 104.775 0)
 			(effects
@@
 			)
 		)
-		(property "Footprint" "878320406:CONN04_878320406_MOL"
+		(property "Footprint" "UTSVT_Connectors:SWD_Conn"
 			(at 156.845 22.225 0)
 			(effects
@@
 			)
 		)
-		(property "Footprint" ""
+		(property "Footprint" "Capacitor_SMD:C_0603_1608Metric_Pad1.08x0.95mm_HandSolder"
 			(at 259.715 57.658 90)
 			(effects
@@
 			)
 		)
-		(property "Footprint" "450406020024:450406020024"
+		(property "Footprint" "UTSVT_Special:BootSW"
 			(at 280.035 4.14 0)
 			(effects
@@
 			)
 		)
-		(property "Footprint" "TL3365AF180QG:TL3365AF180QG"
+		(property "Footprint" "UTSVT_Special:TL3365AF180QG"
 			(at 197.485 115.57 0)
 			(effects
