File: UTSVT_Design_Blocks.kicad_blocks/12VBuck.kicad_block/12VBuck.kicad_sch (KiCad schematic)
At the start: 12 parts, among them U3 LMR51635XDDCR

Commit message: jk real 48 pin fixes
Parts:
- L1: P/N PNLS8040-150M 15UH -> SRN8040-150M
- renumbered C8 to C1, C9 to C2, C10 to C3, C11 to C4, R30 to R1, R31 to R2, U3 to U1
Changed lines of the file:
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@@
 		(dnp no)
 		(fields_autoplaced yes)
-		(property "Reference" "C10"
+		(property "Reference" "C3"
 			(at 172.72 88.9062 0)
 			(effects
@@
 		(dnp no)
 		(fields_autoplaced yes)
-		(property "Reference" "#FLG07"
+		(property "Reference" "#FLG02"
 			(at 149.86 79.375 0)
 			(effects
@@
 		(dnp no)
 		(fields_autoplaced yes)
-		(property "Reference" "C8"
+		(property "Reference" "C1"
 			(at 96.52 85.0962 0)
 			(effects
@@
 		(on_board yes)
 		(dnp no)
-		(property "Reference" "TP9"
+		(property "Reference" "TP?"
 			(at 229.87 123.6979 0)
 			(effects
@@
 				)
 			)
+			(project "12VBuck"
+				(path "/f2a6729b-b8d5-4133-ae64-a5e680928255"
+					(reference "TP?")
+					(unit 1)
+				)
+			)
 		)
 	)
@@
 			)
 		)
-		(property "P/N" "PNLS8040-150M 15UH"
+		(property "P/N" "SRN8040-150M"
 			(at 161.29 86.36 90)
 			(effects
@@
 		(on_board yes)
 		(dnp no)
-		(property "Reference" "TP11"
+		(property "Reference" "TP?"
 			(at 242.57 123.6979 0)
 			(effects
@@
 				)
 			)
+			(project "12VBuck"
+				(path "/f2a6729b-b8d5-4133-ae64-a5e680928255"
+					(reference "TP?")
+					(unit 1)
+				)
+			)
 		)
 	)
@@
 		(on_board yes)
 		(dnp no)
-		(property "Reference" "TP10"
+		(property "Reference" "TP?"
 			(at 229.87 136.3979 0)
 			(effects
@@
 				)
 			)
+			(project "12VBuck"
+				(path "/f2a6729b-b8d5-4133-ae64-a5e680928255"
+					(reference "TP?")
+					(unit 1)
+				)
+			)
 		)
 	)
@@
 		(dnp no)
 		(fields_autoplaced yes)
-		(property "Reference" "U3"
+		(property "Reference" "U1"
 			(at 129.54 71.12 0)
 			(effects
@@
 		(on_board yes)
 		(dnp no)
-		(property "Reference" "TP12"
+		(property "Reference" "TP?"
 			(at 242.57 136.3979 0)
 			(effects
@@
 				)
 			)
+			(project "12VBuck"
+				(path "/f2a6729b-b8d5-4133-ae64-a5e680928255"
+					(reference "TP?")
+					(unit 1)
+				)
+			)
 		)
 	)
@@
 		(dnp no)
 		(fields_autoplaced yes)
-		(property "Reference" "C11"
+		(property "Reference" "C4"
 			(at 184.15 88.9062 0)
 			(effects
@@
 		(dnp no)
 		(fields_autoplaced yes)
-		(property "Reference" "#FLG09"
+		(property "Reference" "#FLG04"
 			(at 181.61 84.455 0)
 			(effects
@@
 		(dnp no)
 		(fields_autoplaced yes)
-		(property "Reference" "#FLG06"
+		(property "Reference" "#FLG01"
 			(at 88.9 79.375 0)
 			(effects
@@
 		(on_board yes)
 		(dnp no)
-		(property "Reference" "C9"
+		(property "Reference" "C2"
 			(at 156.718 80.01 0)
 			(effects
@@
 		(on_board yes)
 		(dnp no)
-		(property "Reference" "#FLG08"
+		(property "Reference" "#FLG03"
 			(at 149.86 84.455 0)
 			(effects
@@
 		(dnp no)
 		(fields_autoplaced yes)
-		(property "Reference" "R30"
+		(property "Reference" "R1"
 			(at 227.33 85.0899 0)
 			(effects
@@
 		(dnp no)
 		(fields_autoplaced yes)
-		(property "Reference" "R31"
+		(property "Reference" "R2"
 			(at 227.33 92.7099 0)
 			(effects
@@
 		)
 	)
+	(sheet_instances
+		(path "/"
+			(page "1")
+		)
+	)
+	(embedded_fonts no)
 )

Commit message: added all footprints + 3d models to design blocks
Parts:
- L1: footprint Inductor_SMD:L_TDK_VLP8040 -> UTSVT_Passives:SRN8040-150M
- U1: footprint utsvt_ics:DDC0006A-MFG -> UTSVT_ICs:DDC0006A-MFG
Changed lines of the file:
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@@
 			)
 		)
-		(property "Footprint" "Inductor_SMD:L_TDK_VLP8040"
+		(property "Footprint" "UTSVT_Passives:SRN8040-150M"
 			(at 161.29 86.36 0)
 			(effects
@@
 			)
 		)
-		(property "Footprint" "utsvt_ics:DDC0006A-MFG"
+		(property "Footprint" "UTSVT_ICs:DDC0006A-MFG"
 			(at 114.3 81.28 0)
 			(effects
