File: LHRS_Design_Blocks.kicad_blocks/5VBuck.kicad_block/5VBuck.kicad_sch (KiCad schematic)
At the start: 12 parts, among them U1 LMR51635XDDCR

Commit message: UTSVT to LHRS
Parts:
- removed TP10: CB, TestPoint:TestPoint_THTPad_D3.0mm_Drill1.5mm, symbol Connector:TestPoint
- removed TP11: FB, TestPoint:TestPoint_THTPad_D3.0mm_Drill1.5mm, symbol Connector:TestPoint
- removed TP12: SW, TestPoint:TestPoint_THTPad_D3.0mm_Drill1.5mm, symbol Connector:TestPoint
- removed TP9: V_in_24V, TestPoint:TestPoint_THTPad_D3.0mm_Drill1.5mm, symbol Connector:TestPoint
- added TP?: FB, TestPoint:TestPoint_THTPad_D3.0mm_Drill1.5mm, symbol Connector:TestPoint
- added TP?: V_in_24V, TestPoint:TestPoint_THTPad_D3.0mm_Drill1.5mm, symbol Connector:TestPoint
- added TP?: SW, TestPoint:TestPoint_THTPad_D3.0mm_Drill1.5mm, symbol Connector:TestPoint
- added TP?: CB, TestPoint:TestPoint_THTPad_D3.0mm_Drill1.5mm, symbol Connector:TestPoint
- L1: value 15u -> 10u; footprint UTSVT_Passives:SRN8040-150M -> LHRS_Passives:SRN8040-101M; LCSC P/N C2849555 -> C54563397; P/N SRN8040-150M -> SRN8040-101M
- R1: value 143k -> 53.6k; LCSC P/N C22877 -> C23074; P/N 0603WAF1433T5E -> 0603WAF5362T5E
- U1: footprint UTSVT_ICs:DDC0006A-MFG -> LHRS_ICs:DDC0006A-MFG
Connections:
- net CB: now also TP?.1
- net FB: now also TP?.1
- net SW: now also TP?.1
- net V_in_24V: now also TP?.1
- net V_out_12V renamed V_out_5V
Other:
- note added: "24V-5V Buck Converter"
- note added: "5V Vout"
- note removed: "12V Vout"
- note removed: "24V-12V Buck Converter"
