File: LHRS_Design_Blocks.kicad_blocks/ESP32.kicad_block/ESP32.kicad_sch (KiCad schematic)
At the start: 21 parts, among them J1 USB_C_Receptacle_USB2.0_16P, SW1 BOOT Switch, SW2 RESET Button, U1 ESP32-C6-MINI-1

Commit message: UTSVT to LHRS
Parts:
- D2: symbol utsvt_ics:SP0503BAH -> lhrs_ics:SP0503BAH
- J1: footprint UTSVT_Connectors:USB_C_Receptacle_GCT_USB4105-xx-A_16P_TopMnt_Horizontal -> LHRS_Connectors:USB_C_Receptacle_GCT_USB4105-xx-A_16P_TopMnt_Horizontal; symbol utsvt_connectors:USB_C_Receptacle_USB2.0_16P -> lhrs_connectors:USB_C_Receptacle_USB2.0_16P
- SW1: footprint UTSVT_Special:BootSW -> LHRS_Special:BootSW
- SW2: footprint UTSVT_Special:TL3365AF180QG -> LHRS_Special:TL3365AF180QG
- U1: footprint UTSVT_Special:ESP32-C6-MINI-1 -> LHRS_Special:ESP32-C6-MINI-1; symbol utsvt_special:ESP32-C6-MINI-1/U -> lhrs_special:ESP32-C6-MINI-1/U
Changed lines of the file:
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@@
 	)
 	(symbol
-		(lib_id "utsvt_special:ESP32-C6-MINI-1/U")
+		(lib_id "lhrs_special:ESP32-C6-MINI-1/U")
 		(at 158.75 78.74 0)
 		(unit 1)
@@
 			)
 		)
-		(property "Footprint" "UTSVT_Special:ESP32-C6-MINI-1"
+		(property "Footprint" "LHRS_Special:ESP32-C6-MINI-1"
 			(at 158.75 78.74 0)
 			(effects
@@
 	)
 	(symbol
-		(lib_id "utsvt_ics:SP0503BAH")
+		(lib_id "lhrs_ics:SP0503BAH")
 		(at 74.93 144.78 90)
 		(unit 1)
@@
 			)
 		)
-		(property "Footprint" "UTSVT_Special:TL3365AF180QG"
+		(property "Footprint" "LHRS_Special:TL3365AF180QG"
 			(at 167.64 27.94 0)
 			(effects
@@
 	)
 	(symbol
-		(lib_id "utsvt_connectors:USB_C_Receptacle_USB2.0_16P")
+		(lib_id "lhrs_connectors:USB_C_Receptacle_USB2.0_16P")
 		(at 31.75 87.63 0)
 		(unit 1)
@@
 			)
 		)
-		(property "Footprint" "UTSVT_Connectors:USB_C_Receptacle_GCT_USB4105-xx-A_16P_TopMnt_Horizontal"
+		(property "Footprint" "LHRS_Connectors:USB_C_Receptacle_GCT_USB4105-xx-A_16P_TopMnt_Horizontal"
 			(at 35.56 87.63 0)
 			(effects
@@
 			)
 		)
-		(property "Footprint" "UTSVT_Special:BootSW"
+		(property "Footprint" "LHRS_Special:BootSW"
 			(at 118.11 34.29 0)
 			(effects
