File: LHRS_Design_Blocks.kicad_blocks/ESP32.kicad_block/ESP32.kicad_sch (KiCad schematic)
At the start: 21 parts, among them J1 USB_C_Receptacle_USB2.0_16P, SW1 BOOT Switch, SW2 RESET Button, U1 ESP32-C6-MINI-1

Commit message: tp symbol + usb fixes
Parts:
- C1, C2: value 10uF -> 10u
- C3, C4: value 0.1uF -> 0.1u
- D2: Mouser Part Number 576-SP0503BAHTG -> (none)
Connections:
- net USB_D+ renamed USB_ESP_D+
- net USB_D- renamed USB_ESP_D-
Other:
- moved on the sheet: D2
