File: LHRS_Design_Blocks.kicad_blocks/Power_Mux.kicad_block/Power_Mux.kicad_sch (KiCad schematic)
At the start: 6 parts, among them U1 TPS2117DRLR

Commit message: UTSVT to LHRS
Parts:
- U1: footprint UTSVT_Power:TPS2117DRLR -> LHRS_Power:TPS2117DRLR
Changed lines of the file:
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@@
 			)
 		)
-		(property "Footprint" "UTSVT_Power:TPS2117DRLR"
+		(property "Footprint" "LHRS_Power:TPS2117DRLR"
 			(at 60.96 62.23 0)
 			(effects
