File: LHRS_Design_Blocks.kicad_blocks/Power_Mux.kicad_block/Power_Mux.kicad_sch (KiCad schematic)
At the start: 6 parts, among them U1 TPS2117DRLR

Commit message: Rev a fixes (#84)
* updated buck block

* tp symbol + usb fixes

* fixes

* updated .gitignore

* updated conns
Parts:
- C1, C2, C3, C4: value 0.1uF -> 0.1u; Mfg MLASH168SB7104KTNA01 -> (none)
- U1: MANUFACTURER Texas Instruments -> (none); MAXIMUM_PACKAGE_HEIGHT 0.6mm -> (none); PARTREV A -> (none); STANDARD IPC-7351B -> (none)
