File: UTSVT_Design_Blocks.kicad_blocks/Contactor.kicad_block/Contactor.kicad_sch (KiCad schematic)
At the start: 15 parts, among them Q1 IRLML0030, Q3 IRLML0030

Commit message: replace good resistors with communist ones
Parts:
- removed R12, R? (x3): 10k, Resistor_SMD:R_0603_1608Metric_Pad0.98x0.95mm_HandSolder, symbol Device:R_US
- removed R15: 4.3k, Resistor_SMD:R_0603_1608Metric_Pad0.98x0.95mm_HandSolder, symbol Device:R_US
- removed R?: 1k, Resistor_SMD:R_0603_1608Metric_Pad0.98x0.95mm_HandSolder, symbol Device:R_US
- added R? (x4): 10k, symbol Device:R
- added R?: 1k, symbol Device:R
- added R?: 4.3k, symbol Device:R
- renumbered C14 to C?, C15 to C?, D32 to D?, D5 to D?, Q1 to Q?, Q3 to Q?, TP4 to TP?, TP7 to TP?
Connections:
- net CONTACTOR+: now also R?.2
- net CONTROL: now also R?.2
- net GND: now also R?.1, R?.1, R?.1
- net SENSE: now also R?.2
- net at D?.2 (A): now also R?.1
- net at J?.3 (Sense-): now also R?.2
- net at C?.2, Q?.1 (G): now also R?.2
- new net: R?.1, R?.1, R?.2

Commit message: fixed footprints + 3d models
Parts:
- D?: footprint CustomKiCad-Library:SODFL5226X100N -> LHRS_Passives:SODFL5226X100N
- J?: footprint UTSVT_Connectors:Molex_Nano-Fit_105309-xx04_1x04_P2.50mm_Vertical -> LHRS_Connectors:Molex_Nano-Fit_105309-xx05_1x04_P2.50mm_Vertical
- R? (x6): footprint (none) -> Resistor_SMD:R_0603_1608Metric_Pad0.98x0.95mm_HandSolder
- TP? (x2): footprint TestPoint:TestPoint_Pad_1.0x1.0mm -> TestPoint:TestPoint_THTPad_D3.0mm_Drill1.5mm
