File: LHRS_Design_Blocks.kicad_blocks/100PinMCU.kicad_block/100PinMCU.kicad_sch (KiCad schematic)
At the start: 33 parts, among them J1 SWD_Header, J2 SWD, SW1 SW_SPDT, U1 STM32G473VETx, Y1 Crystal

Commit message: +3v3 standardized ; orient rgb pins for ezier routing
Connections:
- net 3V3 is gone; now on net +3V3: C10.1, C12.1, C13.1, C3.1, C5.1, C8.1, FB2.1, J1.1 (Pin_1), J2.1 (Pin_1), R1.2, U1.100 (VDD), U1.24 (VDD), U1.49 (VDD), U1.6 (VBAT), U1.64 (VDD), U1.75 (VDD)
- net PA0: now also D2.5; no longer D2.1
- net PA2: now also D2.1; no longer D2.5
- net +3.3V renamed +3V3
Changed lines of the file:
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@@
 		)
 	)
-	(label "PA2"
+	(label "PA0"
 		(at 266.7 129.54 0)
 		(effects
@@
 		)
 	)
-	(label "PA0"
+	(label "PA2"
 		(at 243.84 129.54 0)
 		(effects
@@
 		)
 	)
-	(hierarchical_label "3V3"
+	(hierarchical_label "+3V3"
 		(shape input)
 		(at 219.71 152.4 180)
@@
 		)
 	)
-	(hierarchical_label "3V3"
+	(hierarchical_label "+3V3"
 		(shape input)
 		(at 217.17 134.62 180)
@@
 		)
 	)
-	(hierarchical_label "3V3"
+	(hierarchical_label "+3V3"
 		(shape input)
 		(at 102.87 22.86 0)
@@
 		)
 	)
-	(hierarchical_label "3V3"
+	(hierarchical_label "+3V3"
 		(shape input)
 		(at 248.92 52.07 180)
@@
 		)
 	)
-	(hierarchical_label "+3.3V"
+	(hierarchical_label "+3V3"
 		(shape input)
 		(at 227.33 90.17 180)
@@
 		)
 	)
-	(hierarchical_label "3V3"
+	(hierarchical_label "+3V3"
 		(shape input)
 		(at 196.85 83.82 180)
@@
 		)
 	)
-	(hierarchical_label "3V3"
+	(hierarchical_label "+3V3"
 		(shape input)
 		(at 179.07 21.59 180)
