File: LHRS_Design_Blocks.kicad_blocks/usb_pd_boost.kicad_block/usb_pd_boost.kicad_sch (KiCad schematic)
At the start: 28 parts, among them IC1 TPS55340PWP

Commit message: UTSVT to LHRS
Parts:
- D2: footprint UTSVT_Power:B540C-13-F -> LHRS_Power:B540C-13-F; symbol utsvt_power:B540C-13-F -> lhrs_power:B540C-13-F
- IC1: footprint UTSVT_Power:TPS55340PWP -> LHRS_Power:TPS55340PWP
- L1: footprint UTSVT_Power:SDR1307-100ML -> LHRS_Power:SDR1307-100ML
Changed lines of the file:
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@@
 			)
 		)
-		(property "Footprint" "UTSVT_Power:TPS55340PWP"
+		(property "Footprint" "LHRS_Power:TPS55340PWP"
 			(at 110.49 159.69 0)
 			(effects
@@
 	)
 	(symbol
-		(lib_id "utsvt_power:B540C-13-F")
+		(lib_id "lhrs_power:B540C-13-F")
 		(at 138.43 55.88 180)
 		(unit 1)
@@
 			)
 		)
-		(property "Footprint" "UTSVT_Power:B540C-13-F"
+		(property "Footprint" "LHRS_Power:B540C-13-F"
 			(at 138.43 55.88 0)
 			(effects
@@
 			)
 		)
-		(property "Footprint" "UTSVT_Power:SDR1307-100ML"
+		(property "Footprint" "LHRS_Power:SDR1307-100ML"
 			(at 99.06 55.88 0)
 			(effects

Commit message: fixed res symbols
Parts:
- R1, R2, R3, R4, R5, R6, R7: symbol Device:R_US -> Device:R
