File: LHRS_Design_Blocks.kicad_blocks/usb_pd_boost.kicad_block/usb_pd_boost.kicad_sch (KiCad schematic)
At the start: 28 parts, among them IC1 TPS55340PWP

Commit message: 12vbuck (#73)
* 12vbuck

* adress reviews

* new passives

---------

Co-authored-by: Abby Parsons <abigailparsons@utexas,edu>
Parts:
- R1: value 187k -> 88.7k
Connections:
- net +24V renamed +12V
Other:
- note added: "9V: IOUT_MAX = 9*(5.25-0.994/2)*0.9/24 IOUT_MAX ≈ 3.20A (IC Limit) IOUT (90% efficient) = 3A ?? 5V: IOUT_MAX ≈ 1.78A (IC Limit) Real (90% efficient) = 2.25A ?? IOUT = 54W / 24V ?? IOUT ≈ 2.25A ?? 95% → 57W out → 24V @ 2.38A ??"
- note added: "Vin(min) = 5V or 9V Vout = 12V L = 10uH fSW = 600kHZ nest = 90% = 0.9 ILIM = 5.25A (data sheet pg 16)"
- note added: "Vout = 1.229V * (R1/R2 + 1) Vout = 1.229V * (Rsh/Rsl + 1) Vout = 1.229V * (88.7k/10k + 1) Vout = 12.13023 volts"
- note added: "ΔIL = 9*0.6625/(10µH*600kHz) ΔIL = 5.9625 / 6 ΔIL ≈ 0.994A (9V) ΔIL ≈ 0.552A (5V)"
- note removed: "9V: IOUT_MAX = 9*(5.25-0.994/2)*0.9/24 IOUT_MAX ≈ 1.60A (IC Limit) IOUT (90% efficient) = 1A 20V: IOUT_MAX ≈ 3.62A (IC Limit) Real (90% efficient) = 2.25A IOUT = 54W / 24V IOUT ≈ 2.25A 95% → 57W out → 24V @ 2.38A"
- note removed: "Vin(min) = 9V or 20V Vout = 24V L = 10uH fSW = 600kHZ nest = 90% = 0.9 ILIM = 5.25A (data sheet pg 16)"
- note removed: "Vout = 1.229V * (R1/R2 + 1) Vout = 1.229V * (Rsh/Rsl + 1) Vout = 1.229V * (187k/10k + 1) Vout = 24.2113 volts"
- note removed: "ΔIL = 9*0.6625/(10µH*600kHz) ΔIL = 5.9625 / 6 ΔIL ≈ 0.994A (9V) ΔIL ≈ 0.833A (20V)"
Changed lines of the file:
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@@
 		)
 	)
-	(text "ΔIL = 9*0.6625/(10µH*600kHz)\nΔIL = 5.9625 / 6\nΔIL ≈ 0.994A (9V)\nΔIL ≈ 0.833A (20V)"
+	(text "ΔIL = 9*0.6625/(10µH*600kHz)\nΔIL = 5.9625 / 6\nΔIL ≈ 0.994A (9V)\nΔIL ≈ 0.552A (5V)"
 		(exclude_from_sim no)
 		(at 102.87 167.894 0)
@@
 		)
 	)
-	(text "9V:\nIOUT_MAX = 9*(5.25-0.994/2)*0.9/24\nIOUT_MAX ≈ 1.60A (IC Limit)\nIOUT (90% efficient) = 1A\n\n20V:\nIOUT_MAX ≈ 3.62A (IC Limit)\nReal (90% efficient) = 2.25A\nIOUT = 54W / 24V\nIOUT ≈ 2.25A\n95% → 57W out → 24V @ 2.38A"
+	(text "9V:\nIOUT_MAX = 9*(5.25-0.994/2)*0.9/24\nIOUT_MAX ≈ 3.20A (IC Limit)\nIOUT (90% efficient) = 3A ??\n\n5V:\nIOUT_MAX ≈ 1.78A (IC Limit)\nReal (90% efficient) = 2.25A ??\nIOUT = 54W / 24V ??\nIOUT ≈ 2.25A ??\n95% → 57W out → 24V @ 2.38A ??"
 		(exclude_from_sim no)
 		(at 81.534 182.626 0)
@@
 		)
 	)
-	(text "Vin(min) = 9V or 20V\nVout = 24V\nL = 10uH\nfSW = 600kHZ\nnest = 90% = 0.9\nILIM = 5.25A (data sheet pg 16)\n"
+	(text "Vin(min) = 5V or 9V\nVout = 12V\nL = 10uH\nfSW = 600kHZ\nnest = 90% = 0.9\nILIM = 5.25A (data sheet pg 16)\n"
 		(exclude_from_sim no)
 		(at 98.806 147.574 0)
@@
 		)
 	)
-	(text "Vout = 1.229V * (R1/R2 + 1)\nVout = 1.229V * (Rsh/Rsl + 1)\nVout = 1.229V * (187k/10k + 1)\nVout = 24.2113 volts"
+	(text "Vout = 1.229V * (R1/R2 + 1)\nVout = 1.229V * (Rsh/Rsl + 1)\nVout = 1.229V * (88.7k/10k + 1)\nVout = 12.13023 volts"
 		(exclude_from_sim no)
 		(at 81.534 127.254 0)
@@
 		)
 	)
-	(hierarchical_label "+24V"
+	(hierarchical_label "+12V"
 		(shape output)
 		(at 237.49 55.88 0)
@@
 			)
 		)
-		(property "Value" "187k"
+		(property "Value" "88.7k"
 			(at 161.29 67.3099 0)
 			(show_name no)

Commit message: much math
Parts:
- C4: value 0.1uF -> 0.22uF; LCSC P/N C6666325 -> (none); P/N MLASH168SB7104KTNA01 -> CC0603MRY5V7BB224
- C5: LCSC P/N C14665 -> (none)
- R1: P/N CRCW0603187KFKEA -> RC0402FR-0788K7L
- R2: LCSC P/N C843841 -> (none); P/N CRCW060310K0FKEI -> CRCW060310K0FKEI
- R3: value 2.21k -> 1.3k
- R6: value 301k -> 162k; LCSC P/N C273742 -> (none); P/N RC0603FR-07301KL -> CRCW0402162KFKEDHP
Other:
- note added: "- 5V-9V to 12.00V @ 1A-2.25A - Internal 5-A, 40-V low-side MOSFET switch"
- note added: "5V: IOUT_MAX = 5*(5.25-0.521/2)*0.9/12 IOUT_MAX ≈ 1.78A (IC Limit) Real (90% efficient) = 1.602A 9V: IOUT_MAX = 9*(5.25-0.488/2)*0.9/12 IOUT_MAX ≈ 3.38A (IC Limit) IOUT (90% efficient) = 3.042A IOUT = 41W / 12V IOUT ≈ 3.42A 95% → 41W out → 12V @ 3.24A"
- note added: "C1-2 = Vin bypass caps"
- note added: "Cout >= 0.625 * 1 / 600k * 0.1 Cout >= 10.42uF"
- note added: "Dmax = 0.625 IOUT = 1A fSW = 600kHz COUT_nominal = 3×4.7µF + 2×1µF = 16.1µF Vripple = Dmax*Iout/fsw*Cout Vripple ≈ 64.7 mV"
- note added: "R1 = 88.7k R2 = 10k fBW ~= fSW/10 to fSW/20 fSW = 600k, fBW = 6.2kHZ Gea = 440 µA/V R3 = 1 / (0.00044 × 0.101 × 10^(Kps/20)) R3 ~= 1.3k"
- note added: "R3 = 1.3k fBW ~= fSW/10 to fSW/20 fSW = 600k, fBW = 6.2kHZ C4 = 0.22uF"
- note added: "R7/R6+R7 = 4.5 <- turn on V R7 = 51.1k, R6 = 162k"
- note added: "Resr = 8.2mΩ Cout = ~16.1uF R3 = 1.3k C5 = 102pF ~= 100pF"
- note added: "Rfreq = 57500 * fsw(kHz)^-1.03 Rfreq = 57000 * (600)^-1.03 Rfreq = 79.1k -> Round to standard value Rfreq = 78.7k"
- note added: "Rout = 12/1.78 = 6.74 1-D = 5/12 = 0.4167 fRHPZ = 6.74 * (0.4167)^2 / 2pi * 10uH fRHPZ = 18.63kHz fBW = 18.63kHz / 3 = 6.21kHz"
- note added: "Vin = 5V: Dmax = 1 - (Vin*efficiency/Vout) Dmax = 1 - ((5*0.9)/12) Dmax = 0.625 Vin = 9V: Dmax = 1 - (Vin*efficiency/Vout) Dmax = 1 - ((9*0.9)/12) Dmax = 0.325"
- note added: "ΔIL = 5*0.625/(10µH*600kHz) ΔIL ≈ 0.521A (5V) ΔIL = 9*0.325 /(10µH*600kHz) ΔIL ≈ 0.488A (9V)"
- note added: "ΔIL = VIN × D / (L × fSW) ΔIL = 5 × 0.625 / (10µH × 600kHz) ΔIL ≈ 0.521A (worst case) ICIN,rms = ΔIL / √12 ICIN,rms = 0.521 / 3.464 ICIN,rms ≈ 0.150A Allowing 50mV ripple CIN ≥ 0.521 / (4 × 600k × 0.05) CIN ≥ 4.34µF effective"
- note removed: "- 8V-20V to 24.00V @ 1A-2.25A - Internal 5-A, 40-V low-side MOSFET switch"
- note removed: "9V: IOUT_MAX = 9*(5.25-0.994/2)*0.9/24 IOUT_MAX ≈ 3.20A (IC Limit) IOUT (90% efficient) = 3A ?? 5V: IOUT_MAX ≈ 1.78A (IC Limit) Real (90% efficient) = 2.25A ?? IOUT = 54W / 24V ?? IOUT ≈ 2.25A ?? 95% → 57W out → 24V @ 2.38A ??"
- note removed: "C7 = Vin bypass caps"
- note removed: "Dmax = 0.6625 IOUT = 1A fSW = 600kHz COUT_nominal = 3×4.7µF + 2×1µF = 16.1µF Vripple = Dmax*Iout/fsw*Cout Vripple ≈ 68.6 mV"
- note removed: "R1 = 187k R2 = 10k fBW ~= fSW/10 to fSW/20 fSW = 600k, fBW = 6.2kHZ Gea = 440 µA/V R3 = 1 / (0.00044 × 0.0508 × 10^(Kps/20)) R3 ~= 2.2k --> 2.49k, common passives"
- note removed: "R3 = 2.2k fBW ~= fSW/10 to fSW/20 fSW = 600k, fBW = 6.2kHZ C4 = 0.1uF"
- note removed: "Resr = 13.7mΩ Cout = ~16.1uF R3 = 2.2k C5 = 104pF ~= 100pF"
- note removed: "Rfreq = 57500 * fsw(kHz)^-1.03 Rfreq = 57000 * (600)^-1.03 Rfreq = 78.4k"
- note removed: "Vin = 9V Dmax = 1 - (Vin*efficiency/Vout) Dmax = 1 - ((9*0.9)/24) Dmax = 0.6625 Vin = 20V D = 1 - (VIN × η / VOUT) D = 1 - (20 × 0.9 / 24) D = 1 - 0.75 D = 0.25"
- note removed: "ΔIL = 9*0.6625/(10µH*600kHz) ΔIL = 5.9625 / 6 ΔIL ≈ 0.994A (9V) ΔIL ≈ 0.552A (5V)"
- note removed: "ΔIL = VIN × D / (L × fSW) ΔIL = 9 × 0.6625 / (10µH × 600kHz) ΔIL ≈ 0.994A ICIN,rms = ΔIL / √12 ICIN,rms = 0.994 / 3.464 ICIN,rms ≈ 0.287A Allowing 50mV ripple CIN ≥ 0.994 / (4 × 600k × 0.05) CIN ≥ 8.3µF effective"
