File: LHRS_Design_Blocks.kicad_blocks/usb_pd_boost.kicad_block/usb_pd_boost.kicad_sch (KiCad schematic)
At the start: 28 parts, among them IC1 TPS55340PWP

Commit message: Rev a fixes (#84)
* updated buck block

* tp symbol + usb fixes

* fixes

* updated .gitignore

* updated conns
Parts:
- removed TP2: EN, TestPoint:TestPoint_THTPad_D3.0mm_Drill1.5mm, symbol Connector:TestPoint
- removed TP5: SW, TestPoint:TestPoint_THTPad_D3.0mm_Drill1.5mm, symbol Connector:TestPoint
- removed TP6: FB, TestPoint:TestPoint_THTPad_D3.0mm_Drill1.5mm, symbol Connector:TestPoint
- removed TP7: SS, TestPoint:TestPoint_THTPad_D3.0mm_Drill1.5mm, symbol Connector:TestPoint
- removed TP8: COMP, TestPoint:TestPoint_THTPad_D3.0mm_Drill1.5mm, symbol Connector:TestPoint
- C1, C2: value 10uF -> 10u
- C10, C11: value 1uF -> 1u
- C3, C4: value 0.1uF -> 0.1u
- C5: value 0.1nF -> 0.1n
- C6: value 0.047uF -> 0.047u
- C7, C8, C9: value 4.7uF -> 4.7u
- D2: Height 2.5 -> (none); LCSC P/N (none) -> C908244; Manufacturer_Name Diodes Incorporated -> (none); Manufacturer_Part_Number B540C-13-F -> (none); Mouser Part Number 621-B540C-F -> (none); Mouser Price/Stockl https://www.mouser.co.uk/ProductDetail/Diodes-Incorporated/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 -> (none); P/N (none) -> B540C-13-F
- IC1: Height 1.2 -> (none); Manufacturer_Name Texas Instruments -> (none); Manufacturer_Part_Number TPS55340PWP -> (none); Mouser Part Number 595-TPS55340PWP -> (none); Mouser Price/Stock https://www.mouser.co.uk/ProductDetail/Texas-Instruments/TP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 -> (none)
