File: LHRS_Design_Blocks.kicad_blocks/48PinMCU.kicad_block/48PinMCU.kicad_sch (KiCad schematic)
At the start: 30 parts, among them J1 SWD_Header, SW1 Reset, SW2 SW_SPDT, Y1 Crystal

Commit message: fixed leds + datasheets
Parts:
- D2: footprint LED_SMD:LED_0201_0603Metric -> LED_SMD:LED_0603_1608Metric_Pad1.05x0.95mm_HandSolder; LSCS P/N (none) -> C125103; P/N XL-1608UBC-06A -> LTST-C193TBKT-5A
Changed lines of the file:
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@@
 			)
 		)
-		(property "Footprint" "LED_SMD:LED_0201_0603Metric"
+		(property "Footprint" "LED_SMD:LED_0603_1608Metric_Pad1.05x0.95mm_HandSolder"
 			(at 259.842 107.442 0)
 			(hide yes)
@@
 			)
 		)
-		(property "P/N" "XL-1608UBC-06A"
+		(property "P/N" "LTST-C193TBKT-5A"
 			(at 259.842 107.442 90)
 			(hide yes)
@@
 			)
 		)
-		(property "LSCS P/N" ""
+		(property "LSCS P/N" "C125103"
 			(at 259.842 107.442 90)
 			(hide yes)
