File: LHRS_Design_Blocks.kicad_blocks/48PinMCU.kicad_block/48PinMCU.kicad_sch (KiCad schematic)
At the start: 34 parts, among them J1 SWD_Header, J2 SWD, SW1 Reset, SW2 SW_SPDT, U1 STM32G473CETx, Y1 Crystal

Commit message: change mouser p/n for 1uF to be right
Parts:
- C11, C9: Mouser Part Number MLASH168SB7104KTNA01 -> CL10A105KB8NNNC; P/N MLASU168SB5105KTNA01 -> CL10A105KB8NNNC
Changed lines of the file:
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@@
 			)
 		)
-		(property "Mouser Part Number" "MLASH168SB7104KTNA01"
+		(property "Mouser Part Number" "CL10A105KB8NNNC"
 			(at 201.422 58.674 0)
 			(hide yes)
@@
 			)
 		)
-		(property "P/N" "MLASU168SB5105KTNA01"
+		(property "P/N" "CL10A105KB8NNNC"
 			(at 201.422 58.674 0)
 			(hide yes)
@@
 			)
 		)
-		(property "Mouser Part Number" "MLASH168SB7104KTNA01"
+		(property "Mouser Part Number" "CL10A105KB8NNNC"
 			(at 216.662 58.674 0)
 			(hide yes)
@@
 			)
 		)
-		(property "P/N" "MLASU168SB5105KTNA01"
+		(property "P/N" "CL10A105KB8NNNC"
 			(at 216.662 58.674 0)
 			(hide yes)
