File: LHRS_Design_Blocks.kicad_blocks/48PinMCU.kicad_block/48PinMCU.kicad_sch (KiCad schematic)
At the start: 34 parts, among them J1 SWD_Header, J2 SWD, SW1 Reset, SW2 SW_SPDT, U1 STM32G473CETx, Y1 Crystal

Commit message: Rev a fixes (#84)
* updated buck block

* tp symbol + usb fixes

* fixes

* updated .gitignore

* updated conns
Parts:
- C10, C11, C12, C13, C14, C3, C5, C6, C7, C8, C9: Mouser Part Number MLASH168SB7104KTNA01 -> (none)
- C4: Mouser Part Number 08055D475KAT4A -> (none)
- D1: MANUFACTURER Everlight -> (none)
- D2: Color Blue -> (none); Mouser P/N 771-PESD15VL1BA-T/R -> (none)
- J1: LSCS P/N C17492485 -> (none)
- R2, R7: Mouser Part Number CRCW060310K0FKEI -> (none)
- SW1: Mouser Part Number 612-TL3365AF180QG -> (none)
