File: LHRS_Design_Blocks.kicad_blocks/12VBuck.kicad_block/12VBuck.kicad_sch (KiCad schematic)
At the start: 12 parts, among them U1 LMR51635XDDCR

Commit message: UTSVT to LHRS
Parts:
- removed TP?: FB, TestPoint:TestPoint_THTPad_D3.0mm_Drill1.5mm, symbol Connector:TestPoint
- removed TP?: V_in_24V, TestPoint:TestPoint_THTPad_D3.0mm_Drill1.5mm, symbol Connector:TestPoint
- removed TP?: SW, TestPoint:TestPoint_THTPad_D3.0mm_Drill1.5mm, symbol Connector:TestPoint
- removed TP?: CB, TestPoint:TestPoint_THTPad_D3.0mm_Drill1.5mm, symbol Connector:TestPoint
- added TP10: CB, TestPoint:TestPoint_THTPad_D3.0mm_Drill1.5mm, symbol Connector:TestPoint
- added TP11: FB, TestPoint:TestPoint_THTPad_D3.0mm_Drill1.5mm, symbol Connector:TestPoint
- added TP12: SW, TestPoint:TestPoint_THTPad_D3.0mm_Drill1.5mm, symbol Connector:TestPoint
- added TP9: V_in_24V, TestPoint:TestPoint_THTPad_D3.0mm_Drill1.5mm, symbol Connector:TestPoint
- L1: value 10u -> 15u; footprint UTSVT_Passives:SRN8040-101M -> LHRS_Passives:SRN8040-150M; LCSC P/N C54563397 -> C2849555; P/N SRN8040-101M -> SRN8040-150M
- R1: value 53.6k -> 143k; LCSC P/N C23074 -> C22877; P/N 0603WAF5362T5E -> 0603WAF1433T5E
- U1: footprint UTSVT_ICs:DDC0006A-MFG -> LHRS_ICs:DDC0006A-MFG
Connections:
- net CB: now also TP10.1
- net FB: now also TP11.1
- net SW: now also TP12.1
- net V_in_24V: now also TP9.1
- net V_out_5V renamed V_out_12V
Other:
- note added: "12V Vout"
- note added: "24V-12V Buck Converter"
- note removed: "24V-5V Buck Converter"
- note removed: "5V Vout"

Commit message: 12vbuck
Parts:
- C3, C4: value 47u -> 33u
- L1: value 15u -> 10u
- R1: value 143k -> 53.6k
Connections:
- net V_in_24V renamed V_in_12V
- net V_out_12V renamed V_out_5V
Other:
- note added: "12V-5V Buck Converter"
- note added: "Vout 5"
- note removed: "24V-12V Buck Converter"

Commit message: adress reviews
Parts:
- TP9: value V_in_24V -> V_in_12V
Changed lines of the file:
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@@
 	)
 	(hierarchical_label "GND"
-		(shape input)
+		(shape bidirectional)
 		(at 181.61 95.25 180)
 		(effects
@@
 	)
 	(hierarchical_label "GND"
-		(shape input)
+		(shape bidirectional)
 		(at 170.18 95.25 180)
 		(effects
@@
 	)
 	(hierarchical_label "GND"
-		(shape input)
+		(shape bidirectional)
 		(at 93.98 91.44 180)
 		(effects
@@
 	)
 	(hierarchical_label "GND"
-		(shape input)
+		(shape bidirectional)
 		(at 224.79 97.79 180)
 		(effects
@@
 	)
 	(hierarchical_label "GND"
-		(shape input)
+		(shape bidirectional)
 		(at 147.32 96.52 0)
 		(effects
@@
 			)
 		)
-		(property "Value" "V_in_24V"
+		(property "Value" "V_in_12V"
 			(at 222.25 122.428 0)
 			(show_name no)
@@
 			)
 		)
-		(property "Datasheet" "kicad-embed://lmr51635.pdf"
+		(property "Datasheet" "https://www.ti.com/lit/ds/symlink/lmr51635.pdf?ts=1788472542955&ref_url=https%253A%252F%252Fwww.ti.com%252Fproduct%252FLMR51635%252Fpart-details%252FLMR51635XFDDCR"
 			(at 114.3 81.28 0)
 			(hide yes)

Commit message: new passives
Parts:
- removed C3: 33u, Capacitor_SMD:C_1210_3225Metric_Pad1.33x2.70mm_HandSolder, symbol Device:C_Small
- added C5: 100n, Capacitor_SMD:C_0805_2012Metric_Pad1.18x1.45mm_HandSolder, symbol Device:C_Small
- C1: value 2.2u -> 4.7u; LCSC P/N C1771 -> (none); P/N CL21F225ZAFNNNE -> MSASL168SB5475KTNA01
- C2: LCSC P/N C14663 -> (none)
- C4: value 33u -> 47u; LCSC P/N C77101 -> (none); P/N GRM32ER61C476KE15L -> ZRB18AC80E476ME01L
- L1: value 10u -> 8.2u; LCSC P/N C2849555 -> (none); P/N SRN8040-150M -> 74439369082
- R1: value 53.6k -> 100k; LCSC P/N C22877 -> (none); P/N 0603WAF1433T5E -> AE1206BR-07100KL
- R2: value 10.2k -> 19.1k; LCSC P/N C22772 -> (none); P/N 0603WAF1022T5E -> ERA-2ARB1912X
Connections:
- net GND: now also C5.2
- net V_in_12V: now also C5.1

Commit message: updated footprints, p/n, and checked for stocks for every passive
Parts:
- C10: renamed from C4; LCSC P/N (none) -> C6870970; P/N ZRB18AC80E476ME01L -> C1210C476M9PACTU
- C11: renamed from C1; LCSC P/N (none) -> C6962403; P/N MSASL168SB5475KTNA01 -> 08055D475KAT4A
- C12: renamed from C2; LCSC P/N (none) -> C6666325
- C5: footprint Capacitor_SMD:C_0805_2012Metric_Pad1.18x1.45mm_HandSolder -> Capacitor_SMD:C_0603_1608Metric_Pad1.08x0.95mm_HandSolder; LCSC P/N (none) -> C6666325
- L3: renamed from L1; footprint LHRS_Passives:SRN8040-150M -> LHRS_Passives:74439369082
- R1: LCSC P/N (none) -> C25803; P/N AE1206BR-07100KL -> CRCW0603100KFKEE
- R4: renamed from R2; LCSC P/N (none) -> C844132; P/N ERA-2ARB1912X -> CRCW060319K1FKEAHP
- renumbered U1 to U3
Changed lines of the file:
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@@
 		)
 		(instances
+			(project "12-5vBuck"
+				(path "/0fbc6656-132d-42e4-bdc9-f0a11468b104/973e334b-57f3-4378-b197-420dc86c33e2"
+					(reference "#FLG02")
+					(unit 1)
+				)
+			)
 			(project "PS-Buck"
 				(path "/331f457b-ed4e-4d4a-ad6d-c8acb2febfed/9243f342-8d42-4433-b049-031be1288812"
@@
 		(dnp no)
 		(fields_autoplaced yes)
-		(property "Reference" "C1"
+		(property "Reference" "C11"
 			(at 96.52 85.0962 0)
 			(show_name no)
@@
 			)
 		)
-		(property "LCSC P/N" ""
+		(property "LCSC P/N" "C6962403"
 			(at 93.98 86.36 0)
 			(hide yes)
@@
 			)
 		)
-		(property "P/N" "MSASL168SB5475KTNA01"
+		(property "P/N" "08055D475KAT4A"
 			(at 93.98 86.36 0)
 			(hide yes)
@@
 		)
 		(instances
+			(project "12-5vBuck"
+				(path "/0fbc6656-132d-42e4-bdc9-f0a11468b104/973e334b-57f3-4378-b197-420dc86c33e2"
+					(reference "C11")
+					(unit 1)
+				)
+			)
 			(project "PS-Buck"
 				(path "/331f457b-ed4e-4d4a-ad6d-c8acb2febfed/9243f342-8d42-4433-b049-031be1288812"
@@
 		(in_pos_files yes)
 		(dnp no)
-		(property "Reference" "TP?"
+		(property "Reference" "TP9"
 			(at 229.87 123.6979 0)
 			(hide yes)
@@
 		)
 		(instances
+			(project "12-5vBuck"
+				(path "/0fbc6656-132d-42e4-bdc9-f0a11468b104/973e334b-57f3-4378-b197-420dc86c33e2"
+					(reference "TP9")
+					(unit 1)
+				)
+			)
 			(project "PowerPath"
 				(path "/ad6c7df0-eb90-4670-9aa8-3e2007aefc2d/41c72b07-cf60-4ca9-96a7-6ae96aaa0c90"
@@
 		(in_pos_files yes)
 		(dnp no)
-		(property "Reference" "L1"
+		(property "Reference" "L3"
 			(at 161.29 87.884 90)
 			(show_name no)
@@
 			)
 		)
-		(property "Footprint" "LHRS_Passives:SRN8040-150M"
+		(property "Footprint" "LHRS_Passives:74439369082"
 			(at 161.29 86.36 0)
 			(hide yes)
@@
 		)
 		(instances
+			(project "12-5vBuck"
+				(path "/0fbc6656-132d-42e4-bdc9-f0a11468b104/973e334b-57f3-4378-b197-420dc86c33e2"
+					(reference "L3")
+					(unit 1)
+				)
+			)
 			(project "PS-Buck"
 				(path "/331f457b-ed4e-4d4a-ad6d-c8acb2febfed/9243f342-8d42-4433-b049-031be1288812"
@@
 		(in_pos_files yes)
 		(dnp no)
-		(property "Reference" "TP?"
+		(property "Reference" "TP11"
 			(at 242.57 123.6979 0)
 			(hide yes)
@@
 		)
 		(instances
+			(project "12-5vBuck"
+				(path "/0fbc6656-132d-42e4-bdc9-f0a11468b104/973e334b-57f3-4378-b197-420dc86c33e2"
+					(reference "TP11")
+					(unit 1)
+				)
+			)
 			(project "PowerPath"
 				(path "/ad6c7df0-eb90-4670-9aa8-3e2007aefc2d/41c72b07-cf60-4ca9-96a7-6ae96aaa0c90"
@@
 		(in_pos_files yes)
 		(dnp no)
-		(property "Reference" "TP?"
+		(property "Reference" "TP10"
 			(at 229.87 136.3979 0)
 			(hide yes)
@@
 		)
 		(instances
+			(project "12-5vBuck"
+				(path "/0fbc6656-132d-42e4-bdc9-f0a11468b104/973e334b-57f3-4378-b197-420dc86c33e2"
+					(reference "TP10")
+					(unit 1)
+				)
+			)
 			(project "PowerPath"
 				(path "/ad6c7df0-eb90-4670-9aa8-3e2007aefc2d/41c72b07-cf60-4ca9-96a7-6ae96aaa0c90"
@@
 		(dnp no)
 		(fields_autoplaced yes)
-		(property "Reference" "U1"
+		(property "Reference" "U3"
 			(at 129.54 71.12 0)
 			(show_name no)
@@
 		)
 		(instances
+			(project "12-5vBuck"
+				(path "/0fbc6656-132d-42e4-bdc9-f0a11468b104/973e334b-57f3-4378-b197-420dc86c33e2"
+					(reference "U3")
+					(unit 1)
+				)
+			)
 			(project "PS-Buck"
 				(path "/331f457b-ed4e-4d4a-ad6d-c8acb2febfed/9243f342-8d42-4433-b049-031be1288812"
@@
 		(in_pos_files yes)
 		(dnp no)
-		(property "Reference" "TP?"
+		(property "Reference" "TP12"
 			(at 242.57 136.3979 0)
 			(hide yes)
@@
 		)
 		(instances
+			(project "12-5vBuck"
+				(path "/0fbc6656-132d-42e4-bdc9-f0a11468b104/973e334b-57f3-4378-b197-420dc86c33e2"
+					(reference "TP12")
+					(unit 1)
+				)
+			)
 			(project "PowerPath"
 				(path "/ad6c7df0-eb90-4670-9aa8-3e2007aefc2d/41c72b07-cf60-4ca9-96a7-6ae96aaa0c90"
@@
 		(dnp no)
 		(fields_autoplaced yes)
-		(property "Reference" "C4"
+		(property "Reference" "C10"
 			(at 184.15 88.9062 0)
 			(show_name no)
@@
 			)
 		)
-		(property "P/N" "ZRB18AC80E476ME01L"
+		(property "P/N" "C1210C476M9PACTU"
 			(at 181.61 90.17 0)
 			(hide yes)
@@
 			)
 		)
-		(property "LCSC P/N" ""
+		(property "LCSC P/N" "C6870970"
 			(at 181.61 90.17 0)
 			(hide yes)
@@
 		)
 		(instances
+			(project "12-5vBuck"
+				(path "/0fbc6656-132d-42e4-bdc9-f0a11468b104/973e334b-57f3-4378-b197-420dc86c33e2"
+					(reference "C10")
+					(unit 1)
+				)
+			)
 			(project "PS-Buck"
 				(path "/331f457b-ed4e-4d4a-ad6d-c8acb2febfed/9243f342-8d42-4433-b049-031be1288812"
@@
 		)
 		(instances
+			(project "12-5vBuck"
+				(path "/0fbc6656-132d-42e4-bdc9-f0a11468b104/973e334b-57f3-4378-b197-420dc86c33e2"
+					(reference "#FLG04")
+					(unit 1)
+				)
+			)
 			(project "PS-Buck"
 				(path "/331f457b-ed4e-4d4a-ad6d-c8acb2febfed/9243f342-8d42-4433-b049-031be1288812"
@@
 		)
 		(instances
+			(project "12-5vBuck"
+				(path "/0fbc6656-132d-42e4-bdc9-f0a11468b104/973e334b-57f3-4378-b197-420dc86c33e2"
+					(reference "#FLG01")
+					(unit 1)
+				)
+			)
 			(project "PS-Buck"
 				(path "/331f457b-ed4e-4d4a-ad6d-c8acb2febfed/9243f342-8d42-4433-b049-031be1288812"
@@
 		(in_pos_files yes)
 		(dnp no)
-		(property "Reference" "C2"
+		(property "Reference" "C12"
 			(at 156.718 80.01 0)
 			(show_name no)
@@
 			)
 		)
-		(property "LCSC P/N" ""
+		(property "LCSC P/N" "C6666325"
 			(at 153.67 83.82 0)
 			(hide yes)
@@
 		)
 		(instances
+			(project "12-5vBuck"
+				(path "/0fbc6656-132d-42e4-bdc9-f0a11468b104/973e334b-57f3-4378-b197-420dc86c33e2"
+					(reference "C12")
+					(unit 1)
+				)
+			)
 			(project "PS-Buck"
 				(path "/331f457b-ed4e-4d4a-ad6d-c8acb2febfed/9243f342-8d42-4433-b049-031be1288812"
@@
 		)
 		(instances
+			(project "12-5vBuck"
+				(path "/0fbc6656-132d-42e4-bdc9-f0a11468b104/973e334b-57f3-4378-b197-420dc86c33e2"
+					(reference "#FLG03")
+					(unit 1)
+				)
+			)
 			(project "PS-Buck"
 				(path "/331f457b-ed4e-4d4a-ad6d-c8acb2febfed/9243f342-8d42-4433-b049-031be1288812"
@@
 			)
 		)
-		(property "P/N" "AE1206BR-07100KL"
+		(property "P/N" "CRCW0603100KFKEE"
 			(at 224.79 86.36 0)
 			(hide yes)
@@
 			)
 		)
-		(property "LCSC P/N" ""
+		(property "LCSC P/N" "C25803"
 			(at 224.79 86.36 0)
 			(hide yes)
@@
 		)
 		(instances
+			(project "12-5vBuck"
+				(path "/0fbc6656-132d-42e4-bdc9-f0a11468b104/973e334b-57f3-4378-b197-420dc86c33e2"
+					(reference "R1")
+					(unit 1)
+				)
+			)
 			(project "PS-Buck"
 				(path "/331f457b-ed4e-4d4a-ad6d-c8acb2febfed/9243f342-8d42-4433-b049-031be1288812"
@@
 			)
 		)
-		(property "Footprint" "Capacitor_SMD:C_0805_2012Metric_Pad1.18x1.45mm_HandSolder"
+		(property "Footprint" "Capacitor_SMD:C_0603_1608Metric_Pad1.08x0.95mm_HandSolder"
 			(at 102.87 88.9 0)
 			(hide yes)
@@
 			)
 		)
-		(property "LCSC P/N" ""
+		(property "LCSC P/N" "C6666325"
 			(at 102.87 88.9 0)
 			(hide yes)
@@
 		)
 		(instances
+			(project "12-5vBuck"
+				(path "/0fbc6656-132d-42e4-bdc9-f0a11468b104/973e334b-57f3-4378-b197-420dc86c33e2"
+					(reference "C5")
+					(unit 1)
+				)
+			)
 			(project "12VBuck"
 				(path "/f2a6729b-b8d5-4133-ae64-a5e680928255"
@@
 		(dnp no)
 		(fields_autoplaced yes)
-		(property "Reference" "R2"
+		(property "Reference" "R4"
 			(at 227.33 92.7099 0)
 			(show_name no)
@@
 			)
 		)
-		(property "LCSC P/N" ""
+		(property "LCSC P/N" "C844132"
 			(at 224.79 93.98 0)
 			(hide yes)
@@
 			)
 		)
-		(property "P/N" "ERA-2ARB1912X"
+		(property "P/N" "CRCW060319K1FKEAHP"
 			(at 224.79 93.98 0)
 			(hide yes)
@@
 		)
 		(instances
+			(project "12-5vBuck"
+				(path "/0fbc6656-132d-42e4-bdc9-f0a11468b104/973e334b-57f3-4378-b197-420dc86c33e2"
+					(reference "R4")
+					(unit 1)
+				)
+			)
 			(project "PS-Buck"
 				(path "/331f457b-ed4e-4d4a-ad6d-c8acb2febfed/9243f342-8d42-4433-b049-031be1288812"
@@
 		)
 	)
-	(sheet_instances
-		(path "/"
-			(page "1")
-		)
-	)
-	(embedded_fonts no)
 )

Commit message: updated caps, added new pn
Parts:
- removed C10: 47u, Capacitor_SMD:C_1210_3225Metric_Pad1.33x2.70mm_HandSolder, symbol Device:C_Small
- added C4, C5: 22u, Capacitor_SMD:C_1210_3225Metric_Pad1.33x2.70mm_HandSolder, symbol Device:C
- added C6: 3.3u, Capacitor_SMD:C_0805_2012Metric_Pad1.18x1.45mm_HandSolder, symbol Device:C
- renumbered C11 to C1, C5 to C2, C12 to C3, L3 to L1, R4 to R2, TP9 to TP1, TP10 to TP2, TP11 to TP3, TP12 to TP4, U3 to U1
Connections:
- net GND: now also C4.2, C5.2, C6.2
- net V_out_5V: now also C4.1, C5.1, C6.1

Commit message: 12vbuck
Parts:
- removed C4: 22u, Capacitor_SMD:C_1210_3225Metric_Pad1.33x2.70mm_HandSolder, symbol Device:C
- added #FLG01: PWR_FLAG, symbol Device:C
- added C3: 33u, Capacitor_SMD:C_1210_3225Metric_Pad1.33x2.70mm_HandSolder, symbol Device:C_Small
- L1: value 8.2u -> 10u
- R1: value 100k -> 53.6k
Connections:
- net GND: now also #FLG01.2
- net V_out_5V: now also #FLG01.1
Changed lines of the file:
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@@
+	)
+	(symbol
+		(lib_id "Device:C_Small")
+		(at 170.18 90.17 0)
+		(unit 1)
+		(body_style 1)
+		(exclude_from_sim no)
+		(in_bom yes)
+		(on_board yes)
+		(in_pos_files yes)
+		(dnp no)
+		(fields_autoplaced yes)
+		(property "Reference" "C3"
+			(at 172.72 88.9062 0)
+			(show_name no)
+			(do_not_autoplace no)
+			(effects
+				(font
+					(size 1.27 1.27)
+				)
+				(justify left)
+			)
+		)
+		(property "Value" "33u"
+			(at 172.72 91.4462 0)
+			(show_name no)
+			(do_not_autoplace no)
+			(effects
+				(font
+					(size 1.27 1.27)
+				)
+				(justify left)
+			)
+		)
+		(property "Footprint" "Capacitor_SMD:C_1210_3225Metric_Pad1.33x2.70mm_HandSolder"
+			(at 170.18 90.17 0)
+			(hide yes)
+			(show_name no)
+			(do_not_autoplace no)
+			(effects
+				(font
+					(size 1.27 1.27)
+				)
+			)
+		)
+		(property "Datasheet" ""
+			(at 170.18 90.17 0)
+			(hide yes)
+			(show_name no)
+			(do_not_autoplace no)
+			(effects
+				(font
+					(size 1.27 1.27)
+				)
+			)
+		)
+		(property "Description" "Unpolarized capacitor, small symbol"
+			(at 170.18 90.17 0)
+			(hide yes)
+			(show_name no)
+			(do_not_autoplace no)
+			(effects
+				(font
+					(size 1.27 1.27)
+				)
+			)
+		)
+		(property "P/N" "GRM32ER61C476KE15L"
+			(at 170.18 90.17 0)
+			(hide yes)
+			(show_name no)
+			(do_not_autoplace no)
+			(effects
+				(font
+					(size 1.27 1.27)
+				)
+			)
+		)
+		(property "LCSC P/N" "C77101"
+			(at 170.18 90.17 0)
+			(hide yes)
+			(show_name no)
+			(do_not_autoplace no)
+			(effects
+				(font
+					(size 1.27 1.27)
+				)
+			)
+		)
+		(pin "1"
+		)
+		(pin "2"
+		)
+		(instances
+			(project "PS-Buck"
+				(path "/331f457b-ed4e-4d4a-ad6d-c8acb2febfed/9243f342-8d42-4433-b049-031be1288812"
+					(reference "C9")
+					(unit 1)
+				)
+			)
+			(project "PS-Buck"
+				(path "/ad6c7df0-eb90-4670-9aa8-3e2007aefc2d/41c72b07-cf60-4ca9-96a7-6ae96aaa0c90"
+					(reference "C10")
+					(unit 1)
+				)
+			)
+			(project "12VBuck"
+				(path "/f2a6729b-b8d5-4133-ae64-a5e680928255"
+					(reference "C3")
+					(unit 1)
+				)
+			)
+		)
 	)
 	(symbol
@@
 			)
 		)
-		(property "Value" "8.2u"
+		(property "Value" "10u"
 			(at 161.29 89.916 90)
 			(show_name no)
@@
 		(dnp no)
 		(fields_autoplaced yes)
-		(property "Reference" "#FLG04"
-			(at 179.07 84.455 0)
-			(hide yes)
-			(show_name no)
-			(do_not_autoplace no)
-			(effects
-				(font
-					(size 1.27 1.27)
-				)
-			)
-		)
-		(property "Value" "PWR_FLAG"
-			(at 179.07 81.28 0)
-			(show_name no)
-			(do_not_autoplace no)
-			(effects
-				(font
-					(size 1.27 1.27)
-				)
-			)
-		)
-		(property "Footprint" ""
-			(at 179.07 86.36 0)
+		(property "Reference" "C4"
+			(at 184.15 88.9062 0)
+			(show_name no)
+			(do_not_autoplace no)
+			(effects
+				(font
+					(size 1.27 1.27)
+				)
+			)
+		)
+		(property "Value" "33u"
+			(at 184.15 91.4462 0)
+			(show_name no)
+			(do_not_autoplace no)
+			(effects
+				(font
+					(size 1.27 1.27)
+				)
+			)
+		)
+		(property "Footprint" "Capacitor_SMD:C_1210_3225Metric_Pad1.33x2.70mm_HandSolder"
+			(at 181.61 90.17 0)
 			(hide yes)
 			(show_name no)
@@
 		)
 		(property "Datasheet" ""
-			(at 179.07 86.36 0)
-			(hide yes)
-			(show_name no)
-			(do_not_autoplace no)
-			(effects
-				(font
-					(size 1.27 1.27)
-				)
-			)
-		)
-		(property "Description" "Special symbol for telling ERC where power comes from"
-			(at 179.07 86.36 0)
+			(at 181.61 90.17 0)
+			(hide yes)
+			(show_name no)
+			(do_not_autoplace no)
+			(effects
+				(font
+					(size 1.27 1.27)
+				)
+			)
+		)
+		(property "Description" "Unpolarized capacitor, small symbol"
+			(at 181.61 90.17 0)
+			(hide yes)
+			(show_name no)
+			(do_not_autoplace no)
+			(effects
+				(font
+					(size 1.27 1.27)
+				)
+			)
+		)
+		(property "P/N" "GRM32ER61C476KE15L"
+			(at 181.61 90.17 0)
+			(hide yes)
+			(show_name no)
+			(do_not_autoplace no)
+			(effects
+				(font
+					(size 1.27 1.27)
+				)
+			)
+		)
+		(property "LCSC P/N" "C77101"
+			(at 181.61 90.17 0)
 			(hide yes)
 			(show_name no)
@@
 		(dnp no)
 		(fields_autoplaced yes)
-		(property "Reference" "#FLG01"
-			(at 88.9 79.375 0)
+		(property "Reference" "#FLG04"
+			(at 181.61 84.455 0)
 			(hide yes)
 			(show_name no)
@@
 		)
 		(property "Value" "PWR_FLAG"
-			(at 88.9 76.2 0)
+			(at 181.61 81.28 0)
 			(show_name no)
 			(do_not_autoplace no)
@@
 		)
 		(property "Footprint" ""
-			(at 88.9 81.28 0)
+			(at 181.61 86.36 0)
 			(hide yes)
 			(show_name no)
@@
 		)
 		(property "Datasheet" ""
-			(at 88.9 81.28 0)
+			(at 181.61 86.36 0)
 			(hide yes)
 			(show_name no)
@@
 		)
 		(property "Description" "Special symbol for telling ERC where power comes from"
-			(at 88.9 81.28 0)
+			(at 181.61 86.36 0)
 			(hide yes)
 			(show_name no)
@@
 		(in_pos_files yes)
 		(dnp no)
-		(property "Reference" "C4"
-			(at 164.084 93.98 0)
-			(show_name no)
-			(do_not_autoplace no)
-			(effects
-				(font
-					(size 1.27 1.27)
-				)
-				(justify left)
-			)
-		)
-		(property "Value" "22u"
-			(at 164.084 96.52 0)
-			(show_name no)
-			(do_not_autoplace no)
-			(effects
-				(font
-					(size 1.27 1.27)
-				)
-				(justify left)
-			)
-		)
-		(property "Footprint" "Capacitor_SMD:C_1210_3225Metric_Pad1.33x2.70mm_HandSolder"
-			(at 171.1452 99.06 0)
+		(fields_autoplaced yes)
+		(property "Reference" "#FLG01"
+			(at 88.9 79.375 0)
+			(hide yes)
+			(show_name no)
+			(do_not_autoplace no)
+			(effects
+				(font
+					(size 1.27 1.27)
+				)
+			)
+		)
+		(property "Value" "PWR_FLAG"
+			(at 88.9 76.2 0)
+			(show_name no)
+			(do_not_autoplace no)
+			(effects
+				(font
+					(size 1.27 1.27)
+				)
+				(justify left)
+			)
+		)
+		(property "Footprint" ""
+			(at 88.9 81.28 0)
 			(hide yes)
 			(show_name no)
@@
 		)
 		(property "Datasheet" ""
-			(at 170.18 95.25 0)
-			(hide yes)
-			(show_name no)
-			(do_not_autoplace no)
-			(effects
-				(font
-					(size 1.27 1.27)
-				)
-			)
-		)
-		(property "Description" "Unpolarized capacitor"
-			(at 170.18 95.25 0)
-			(hide yes)
-			(show_name no)
-			(do_not_autoplace no)
-			(effects
-				(font
-					(size 1.27 1.27)
-				)
-			)
-		)
-		(property "P/N" "GMK325BJ226MM-P"
-			(at 170.18 95.25 0)
-			(hide yes)
-			(show_name no)
-			(do_not_autoplace no)
-			(effects
-				(font
-					(size 1.27 1.27)
-				)
-			)
-		)
-		(property "LCSC P/N" "C778721"
-			(at 170.18 95.25 0)
+			(at 88.9 81.28 0)
+			(hide yes)
+			(show_name no)
+			(do_not_autoplace no)
+			(effects
+				(font
+					(size 1.27 1.27)
+				)
+			)
+		)
+		(property "Description" "Special symbol for telling ERC where power comes from"
+			(at 88.9 81.28 0)
 			(hide yes)
 			(show_name no)
@@
 			)
 		)
-		(property "Value" "100k"
+		(property "Value" "53.6k"
 			(at 227.33 87.6299 0)
 			(show_name no)

Commit message: adress reviews
Connections:
- net GND: no longer #FLG01.2, C2.2, C5.2, C6.2
- new net: #FLG01.2, C5.2, C6.2
Changed lines of the file:
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@@
 	(hierarchical_label "GND"
 		(shape bidirectional)
-		(at 179.07 102.87 180)
+		(at 181.61 95.25 180)
 		(effects
 			(font
@@
 	(hierarchical_label "GND"
 		(shape bidirectional)
-		(at 102.87 93.98 180)
+		(at 170.18 95.25 180)
 		(effects
 			(font
