File: LHRS_Design_Blocks.kicad_blocks/12VBuck.kicad_block/12VBuck.kicad_sch (KiCad schematic)
At the start: 15 parts, among them U1 LMR51635XDDCR

Commit message: new passives
Parts:
- removed C3: 33u, Capacitor_SMD:C_1210_3225Metric_Pad1.33x2.70mm_HandSolder, symbol Device:C_Small
- C1: LCSC P/N C6962403 -> (none); P/N 08055D475KAT4A -> MSASL168SB5475KTNA01
- C3: LCSC P/N C6666325 -> (none)
- C5: renamed from C2; footprint Capacitor_SMD:C_0603_1608Metric_Pad1.08x0.95mm_HandSolder -> Capacitor_SMD:C_0805_2012Metric_Pad1.18x1.45mm_HandSolder; LCSC P/N C6666325 -> (none)
- L1: value 10u -> 8.2u
- R1: value 53.6k -> 100k; LCSC P/N C25803 -> (none); P/N CRCW0603100KFKEE -> AE1206BR-07100KL
- R2: LCSC P/N C844132 -> (none); P/N CRCW060319K1FKEAHP -> ERA-2ARB1912X
Connections:
- net GND: now also C5.2
- net V_out_5V: no longer #FLG01.1, C5.1, C6.1, L1.2
- net at C5.2, C6.2: no longer #FLG01.2
- new net: C5.1, L1.2
Changed lines of the file:
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@@
 		(color 0 0 0 0)
 	)
-	(junction
-		(at 179.07 99.06)
-		(diameter 0)
-		(color 0 0 0 0)
-	)
 	(wire
 		(pts
@@
 	(wire
 		(pts
-			(xy 170.18 91.44) (xy 179.07 91.44)
-		)
-		(stroke
-			(width 0)
-			(type default)
-		)
-	)
-	(wire
-		(pts
 			(xy 93.98 81.28) (xy 93.98 83.82)
 		)
@@
 	(wire
 		(pts
-			(xy 170.18 99.06) (xy 179.07 99.06)
+			(xy 227.33 130.81) (xy 227.33 128.27)
 		)
 		(stroke
@@
 	(wire
 		(pts
-			(xy 179.07 91.44) (xy 186.69 91.44)
+			(xy 219.71 90.17) (xy 224.79 90.17)
 		)
 		(stroke
@@
 	(wire
 		(pts
-			(xy 227.33 130.81) (xy 227.33 128.27)
+			(xy 93.98 81.28) (xy 102.87 81.28)
 		)
 		(stroke
@@
 	(wire
 		(pts
-			(xy 219.71 90.17) (xy 224.79 90.17)
+			(xy 224.79 90.17) (xy 224.79 91.44)
 		)
 		(stroke
@@
 	(wire
 		(pts
-			(xy 224.79 90.17) (xy 224.79 91.44)
-		)
-		(stroke
-			(width 0)
-			(type default)
-		)
-	)
-	(wire
-		(pts
-			(xy 179.07 86.36) (xy 187.96 86.36)
+			(xy 102.87 81.28) (xy 102.87 86.36)
 		)
 		(stroke
@@
 	(wire
 		(pts
-			(xy 163.83 86.36) (xy 179.07 86.36)
+			(xy 163.83 86.36) (xy 181.61 86.36)
 		)
 		(stroke
@@
 	(hierarchical_label "GND"
 		(shape bidirectional)
-		(at 170.18 95.25 180)
+		(at 102.87 93.98 180)
 		(effects
 			(font
@@
 	)
 	(symbol
-		(lib_id "Device:C_Small")
-		(at 170.18 90.17 0)
-		(unit 1)
-		(body_style 1)
-		(exclude_from_sim no)
-		(in_bom yes)
-		(on_board yes)
-		(in_pos_files yes)
-		(dnp no)
-		(fields_autoplaced yes)
-		(property "Reference" "C3"
-			(at 172.72 88.9062 0)
-			(show_name no)
-			(do_not_autoplace no)
-			(effects
-				(font
-					(size 1.27 1.27)
-				)
-				(justify left)
-			)
-		)
-		(property "Value" "33u"
-			(at 172.72 91.4462 0)
-			(show_name no)
-			(do_not_autoplace no)
-			(effects
-				(font
-					(size 1.27 1.27)
-				)
-				(justify left)
-			)
-		)
-		(property "Footprint" "Capacitor_SMD:C_1210_3225Metric_Pad1.33x2.70mm_HandSolder"
-			(at 170.18 90.17 0)
-			(hide yes)
-			(show_name no)
-			(do_not_autoplace no)
-			(effects
-				(font
-					(size 1.27 1.27)
-				)
-			)
-		)
-		(property "Datasheet" ""
-			(at 170.18 90.17 0)
-			(hide yes)
-			(show_name no)
-			(do_not_autoplace no)
-			(effects
-				(font
-					(size 1.27 1.27)
-				)
-			)
-		)
-		(property "Description" "Unpolarized capacitor, small symbol"
-			(at 170.18 90.17 0)
-			(hide yes)
-			(show_name no)
-			(do_not_autoplace no)
-			(effects
-				(font
-					(size 1.27 1.27)
-				)
-			)
-		)
-		(property "P/N" "GRM32ER61C476KE15L"
-			(at 170.18 90.17 0)
-			(hide yes)
-			(show_name no)
-			(do_not_autoplace no)
-			(effects
-				(font
-					(size 1.27 1.27)
-				)
-			)
-		)
-		(property "LCSC P/N" "C77101"
-			(at 170.18 90.17 0)
-			(hide yes)
-			(show_name no)
-			(do_not_autoplace no)
-			(effects
-				(font
-					(size 1.27 1.27)
-				)
-			)
-		)
-		(pin "1"
-		)
-		(pin "2"
-		)
-		(instances
-			(project "PS-Buck"
-				(path "/331f457b-ed4e-4d4a-ad6d-c8acb2febfed/9243f342-8d42-4433-b049-031be1288812"
-					(reference "C9")
-					(unit 1)
-				)
-			)
-			(project "PS-Buck"
-				(path "/ad6c7df0-eb90-4670-9aa8-3e2007aefc2d/41c72b07-cf60-4ca9-96a7-6ae96aaa0c90"
-					(reference "C10")
-					(unit 1)
-				)
-			)
-			(project "12VBuck"
-				(path "/f2a6729b-b8d5-4133-ae64-a5e680928255"
-					(reference "C3")
-					(unit 1)
-				)
-			)
-		)
-	)
-	(symbol
 		(lib_id "power:PWR_FLAG")
 		(at 149.86 81.28 0)
@@
 			)
 		)
-		(property "LCSC P/N" "C6962403"
+		(property "LCSC P/N" ""
 			(at 93.98 86.36 0)
 			(hide yes)
@@
 			)
 		)
-		(property "P/N" "08055D475KAT4A"
+		(property "P/N" "MSASL168SB5475KTNA01"
 			(at 93.98 86.36 0)
 			(hide yes)
@@
 			)
 		)
-		(property "Value" "10u"
+		(property "Value" "8.2u"
 			(at 161.29 89.916 90)
 			(show_name no)
@@
 			)
 		)
-		(property "Value" "33u"
+		(property "Value" "47u"
 			(at 184.15 91.4462 0)
 			(show_name no)
@@
 			)
 		)
-		(property "P/N" "GRM32ER61C476KE15L"
+		(property "P/N" "ZRB18AC80E476ME01L"
 			(at 181.61 90.17 0)
 			(hide yes)
@@
 			)
 		)
-		(property "LCSC P/N" "C77101"
+		(property "LCSC P/N" ""
 			(at 181.61 90.17 0)
 			(hide yes)
@@
 			)
 		)
-		(property "LCSC P/N" "C6666325"
+		(property "LCSC P/N" ""
 			(at 153.67 83.82 0)
 			(hide yes)
@@
 			)
 		)
-		(property "Value" "53.6k"
+		(property "Value" "100k"
 			(at 227.33 87.6299 0)
 			(show_name no)
@@
 			)
 		)
-		(property "P/N" "CRCW0603100KFKEE"
+		(property "P/N" "AE1206BR-07100KL"
 			(at 224.79 86.36 0)
 			(hide yes)
@@
 			)
 		)
-		(property "LCSC P/N" "C25803"
+		(property "LCSC P/N" ""
 			(at 224.79 86.36 0)
 			(hide yes)
@@
 		(dnp no)
 		(fields_autoplaced yes)
-		(property "Reference" "C2"
+		(property "Reference" "C5"
 			(at 105.41 87.6362 0)
 			(show_name no)
@@
 			)
 		)
-		(property "Footprint" "Capacitor_SMD:C_0603_1608Metric_Pad1.08x0.95mm_HandSolder"
+		(property "Footprint" "Capacitor_SMD:C_0805_2012Metric_Pad1.18x1.45mm_HandSolder"
 			(at 102.87 88.9 0)
 			(hide yes)
@@
 			)
 		)
-		(property "LCSC P/N" "C6666325"
+		(property "LCSC P/N" ""
 			(at 102.87 88.9 0)
 			(hide yes)
@@
 		)
 		(instances
-			(project "12-5vBuck"
-				(path "/0fbc6656-132d-42e4-bdc9-f0a11468b104/973e334b-57f3-4378-b197-420dc86c33e2"
-					(reference "C2")
-					(unit 1)
-				)
-			)
 			(project "12VBuck"
 				(path "/f2a6729b-b8d5-4133-ae64-a5e680928255"
@@
 			)
 		)
-		(property "LCSC P/N" "C844132"
+		(property "LCSC P/N" ""
 			(at 224.79 93.98 0)
 			(hide yes)
@@
 			)
 		)
-		(property "P/N" "CRCW060319K1FKEAHP"
+		(property "P/N" "ERA-2ARB1912X"
 			(at 224.79 93.98 0)
 			(hide yes)

Commit message: updated footprints, p/n, and checked for stocks for every passive
Parts:
- removed C5: 22u, Capacitor_SMD:C_1210_3225Metric_Pad1.33x2.70mm_HandSolder, symbol Device:C
- C11: renamed from C1; LCSC P/N (none) -> C6962403; P/N MSASL168SB5475KTNA01 -> 08055D475KAT4A
- C12: renamed from C3; LCSC P/N (none) -> C6666325
- C5: footprint Capacitor_SMD:C_0805_2012Metric_Pad1.18x1.45mm_HandSolder -> Capacitor_SMD:C_0603_1608Metric_Pad1.08x0.95mm_HandSolder; LCSC P/N (none) -> C6666325
- R1: LCSC P/N (none) -> C25803; P/N AE1206BR-07100KL -> CRCW0603100KFKEE
- R4: renamed from R2; LCSC P/N (none) -> C844132; P/N ERA-2ARB1912X -> CRCW060319K1FKEAHP
- renumbered L1 to L3, TP2 to TP10, TP3 to TP11, TP4 to TP12, TP1 to TP9, U1 to U3
Changed lines of the file:
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@@
 		(dnp no)
 		(fields_autoplaced yes)
-		(property "Reference" "C1"
+		(property "Reference" "C11"
 			(at 96.52 85.0962 0)
 			(show_name no)
@@
 			)
 		)
-		(property "LCSC P/N" ""
+		(property "LCSC P/N" "C6962403"
 			(at 93.98 86.36 0)
 			(hide yes)
@@
 			)
 		)
-		(property "P/N" "MSASL168SB5475KTNA01"
+		(property "P/N" "08055D475KAT4A"
 			(at 93.98 86.36 0)
 			(hide yes)
@@
 			(project "12-5vBuck"
 				(path "/0fbc6656-132d-42e4-bdc9-f0a11468b104/973e334b-57f3-4378-b197-420dc86c33e2"
-					(reference "C1")
+					(reference "C11")
 					(unit 1)
 				)
@@
 		(in_pos_files yes)
 		(dnp no)
-		(property "Reference" "TP1"
+		(property "Reference" "TP9"
 			(at 229.87 123.6979 0)
 			(hide yes)
@@
 			(project "12-5vBuck"
 				(path "/0fbc6656-132d-42e4-bdc9-f0a11468b104/973e334b-57f3-4378-b197-420dc86c33e2"
-					(reference "TP1")
+					(reference "TP9")
 					(unit 1)
 				)
@@
 		(in_pos_files yes)
 		(dnp no)
-		(property "Reference" "L1"
+		(property "Reference" "L3"
 			(at 161.29 87.884 90)
 			(show_name no)
@@
 			(project "12-5vBuck"
 				(path "/0fbc6656-132d-42e4-bdc9-f0a11468b104/973e334b-57f3-4378-b197-420dc86c33e2"
-					(reference "L1")
+					(reference "L3")
 					(unit 1)
 				)
@@
 		(in_pos_files yes)
 		(dnp no)
-		(property "Reference" "TP3"
+		(property "Reference" "TP11"
 			(at 242.57 123.6979 0)
 			(hide yes)
@@
 			(project "12-5vBuck"
 				(path "/0fbc6656-132d-42e4-bdc9-f0a11468b104/973e334b-57f3-4378-b197-420dc86c33e2"
-					(reference "TP3")
+					(reference "TP11")
 					(unit 1)
 				)
@@
 		(in_pos_files yes)
 		(dnp no)
-		(property "Reference" "TP2"
+		(property "Reference" "TP10"
 			(at 229.87 136.3979 0)
 			(hide yes)
@@
 			(project "12-5vBuck"
 				(path "/0fbc6656-132d-42e4-bdc9-f0a11468b104/973e334b-57f3-4378-b197-420dc86c33e2"
-					(reference "TP2")
+					(reference "TP10")
 					(unit 1)
 				)
@@
 		(dnp no)
 		(fields_autoplaced yes)
-		(property "Reference" "U1"
+		(property "Reference" "U3"
 			(at 129.54 71.12 0)
 			(show_name no)
@@
 			(project "12-5vBuck"
 				(path "/0fbc6656-132d-42e4-bdc9-f0a11468b104/973e334b-57f3-4378-b197-420dc86c33e2"
-					(reference "U1")
+					(reference "U3")
 					(unit 1)
 				)
@@
 		(in_pos_files yes)
 		(dnp no)
-		(property "Reference" "TP4"
+		(property "Reference" "TP12"
 			(at 242.57 136.3979 0)
 			(hide yes)
@@
 			(project "12-5vBuck"
 				(path "/0fbc6656-132d-42e4-bdc9-f0a11468b104/973e334b-57f3-4378-b197-420dc86c33e2"
-					(reference "TP4")
+					(reference "TP12")
 					(unit 1)
 				)
@@
 		(dnp no)
 		(fields_autoplaced yes)
-		(property "Reference" "C4"
+		(property "Reference" "C10"
 			(at 184.15 88.9062 0)
 			(show_name no)
@@
 			)
 		)
-		(property "P/N" "ZRB18AC80E476ME01L"
+		(property "P/N" "C1210C476M9PACTU"
 			(at 181.61 90.17 0)
 			(hide yes)
@@
 			)
 		)
-		(property "LCSC P/N" ""
+		(property "LCSC P/N" "C6870970"
 			(at 181.61 90.17 0)
 			(hide yes)
@@
 		)
 		(pin "1"
+		)
+		(pin "2"
 		)
 		(instances
 			(project "12-5vBuck"
 				(path "/0fbc6656-132d-42e4-bdc9-f0a11468b104/973e334b-57f3-4378-b197-420dc86c33e2"
-					(reference "#FLG04")
+					(reference "C10")
 					(unit 1)
 				)
@@
 			(project "12-5vBuck"
 				(path "/0fbc6656-132d-42e4-bdc9-f0a11468b104/973e334b-57f3-4378-b197-420dc86c33e2"
-					(reference "#FLG01")
+					(reference "#FLG04")
 					(unit 1)
 				)
@@
 			(project "12-5vBuck"
 				(path "/0fbc6656-132d-42e4-bdc9-f0a11468b104/973e334b-57f3-4378-b197-420dc86c33e2"
-					(reference "C4")
+					(reference "#FLG01")
+					(unit 1)
+				)
+			)
+			(project "PS-Buck"
+				(path "/331f457b-ed4e-4d4a-ad6d-c8acb2febfed/9243f342-8d42-4433-b049-031be1288812"
+					(reference "#FLG011")
 					(unit 1)
 				)
@@
 		(in_pos_files yes)
 		(dnp no)
-		(property "Reference" "C3"
+		(property "Reference" "C12"
 			(at 156.718 80.01 0)
 			(show_name no)
@@
 			)
 		)
-		(property "LCSC P/N" ""
+		(property "LCSC P/N" "C6666325"
 			(at 153.67 83.82 0)
 			(hide yes)
@@
 			(project "12-5vBuck"
 				(path "/0fbc6656-132d-42e4-bdc9-f0a11468b104/973e334b-57f3-4378-b197-420dc86c33e2"
-					(reference "C3")
+					(reference "C12")
 					(unit 1)
 				)
@@
 			)
 		)
-		(property "P/N" "AE1206BR-07100KL"
+		(property "P/N" "CRCW0603100KFKEE"
 			(at 224.79 86.36 0)
 			(hide yes)
@@
 			)
 		)
-		(property "LCSC P/N" ""
+		(property "LCSC P/N" "C25803"
 			(at 224.79 86.36 0)
 			(hide yes)
@@
 			)
 		)
-		(property "Footprint" "Capacitor_SMD:C_0805_2012Metric_Pad1.18x1.45mm_HandSolder"
+		(property "Footprint" "Capacitor_SMD:C_0603_1608Metric_Pad1.08x0.95mm_HandSolder"
 			(at 102.87 88.9 0)
 			(hide yes)
@@
 			)
 		)
-		(property "LCSC P/N" ""
+		(property "LCSC P/N" "C6666325"
 			(at 102.87 88.9 0)
 			(hide yes)
@@
 		)
 		(instances
+			(project "12-5vBuck"
+				(path "/0fbc6656-132d-42e4-bdc9-f0a11468b104/973e334b-57f3-4378-b197-420dc86c33e2"
+					(reference "C5")
+					(unit 1)
+				)
+			)
 			(project "12VBuck"
 				(path "/f2a6729b-b8d5-4133-ae64-a5e680928255"
@@
 		(dnp no)
 		(fields_autoplaced yes)
-		(property "Reference" "R2"
+		(property "Reference" "R4"
 			(at 227.33 92.7099 0)
 			(show_name no)
@@
 			)
 		)
-		(property "LCSC P/N" ""
+		(property "LCSC P/N" "C844132"
 			(at 224.79 93.98 0)
 			(hide yes)
@@
 			)
 		)
-		(property "P/N" "ERA-2ARB1912X"
+		(property "P/N" "CRCW060319K1FKEAHP"
 			(at 224.79 93.98 0)
 			(hide yes)
@@
 			(project "12-5vBuck"
 				(path "/0fbc6656-132d-42e4-bdc9-f0a11468b104/973e334b-57f3-4378-b197-420dc86c33e2"
-					(reference "R2")
+					(reference "R4")
 					(unit 1)
 				)
@@
 					(unit 1)
 				)
-			)
-		)
-	)
-	(symbol
-		(lib_id "Device:C")
-		(at 179.07 95.25 0)
-		(unit 1)
-		(body_style 1)
-		(exclude_from_sim no)
-		(in_bom yes)
-		(on_board yes)
-		(in_pos_files yes)
-		(dnp no)
-		(property "Reference" "C5"
-			(at 173.482 94.234 0)
-			(show_name no)
-			(do_not_autoplace no)
-			(effects
-				(font
-					(size 1.27 1.27)
-				)
-				(justify left)
-			)
-		)
-		(property "Value" "22u"
-			(at 173.482 96.774 0)
-			(show_name no)
-			(do_not_autoplace no)
-			(effects
-				(font
-					(size 1.27 1.27)
-				)
-				(justify left)
-			)
-		)
-		(property "Footprint" "Capacitor_SMD:C_1210_3225Metric_Pad1.33x2.70mm_HandSolder"
-			(at 180.0352 99.06 0)
-			(hide yes)
-			(show_name no)
-			(do_not_autoplace no)
-			(effects
-				(font
-					(size 1.27 1.27)
-				)
-			)
-		)
-		(property "Datasheet" ""
-			(at 179.07 95.25 0)
-			(hide yes)
-			(show_name no)
-			(do_not_autoplace no)
-			(effects
-				(font
-					(size 1.27 1.27)
-				)
-			)
-		)
-		(property "Description" "Unpolarized capacitor"
-			(at 179.07 95.25 0)
-			(hide yes)
-			(show_name no)
-			(do_not_autoplace no)
-			(effects
-				(font
-					(size 1.27 1.27)
-				)
-			)
-		)
-		(property "P/N" "GMK325BJ226MM-P"
-			(at 179.07 95.25 0)
-			(hide yes)
-			(show_name no)
-			(do_not_autoplace no)
-			(effects
-				(font
-					(size 1.27 1.27)
-				)
-			)
-		)
-		(property "LCSC P/N" "C778721"
-			(at 179.07 95.25 0)
-			(hide yes)
-			(show_name no)
-			(do_not_autoplace no)
-			(effects
-				(font
-					(size 1.27 1.27)
-				)
-			)
-		)
-		(pin "2"
-		)
-		(pin "1"
-		)
-		(instances
-			(project "12-5vBuck"
-				(path "/0fbc6656-132d-42e4-bdc9-f0a11468b104/973e334b-57f3-4378-b197-420dc86c33e2"
-					(reference "C5")
-					(unit 1)
-				)

Commit message: Embedded data sheets in symbol, fixed 12V Buck Design Block schematic issues caused by merge, made edits to 12V Buck Boost Design Block
Parts:
- removed #FLG01: PWR_FLAG, symbol Device:C
- removed U3: LMR51635XDDCR, LHRS_ICs:DDC0006A-MFG, symbol 2026-04-25_18-34-12:LMR51635XDDCR
- added C4, C5: 22u, Capacitor_SMD:C_1210_3225Metric_Pad1.33x2.70mm_HandSolder, symbol Device:C
- added U1: LMR51635XDDCR, DDC0006A-MFG, symbol lhrs_power:LMR51635XDDCR
- renumbered C11 to C1, C12 to C2, L3 to L1, R4 to R2, TP9 to TP1, TP10 to TP2, TP11 to TP3, TP12 to TP4
Connections:
- net CB: now also U1.6 (CB)
- net FB: now also U1.1 (FB)
- net GND: now also C6.2, C4.2, C5.2, U1.4 (GND)
- net SW: now also U1.5 (SW)
- net V_in_12V: now also U1.2 (EN), U1.3 (VIN)
- net V_out_5V: now also C6.1, L1.2, C4.1, C5.1

Commit message: Rev a fixes (#84)
* updated buck block

* tp symbol + usb fixes

* fixes

* updated .gitignore

* updated conns
Parts:
- removed TP1: V_in_12V, TestPoint:TestPoint_THTPad_D3.0mm_Drill1.5mm, symbol Connector:TestPoint
- removed TP2: CB, TestPoint:TestPoint_THTPad_D3.0mm_Drill1.5mm, symbol Connector:TestPoint
- removed TP3: FB, TestPoint:TestPoint_THTPad_D3.0mm_Drill1.5mm, symbol Connector:TestPoint
- removed TP4: SW, TestPoint:TestPoint_THTPad_D3.0mm_Drill1.5mm, symbol Connector:TestPoint
- L1: footprint LHRS_Passives:74439369082 -> LHRS_Power:XAL5050822MEC; LCSC P/N (none) -> C5309356; P/N 74439369082 -> XAL5050-822MEC
- U1: LCSC P/N (none) -> C42432812; P/N (none) -> LMR51635XDDCR
Other:
- note added: "Vin: 4.6V to 60V"
- note removed: "Test Points"
