File: LHRS_Design_Blocks.kicad_blocks/PowerProtection.kicad_block/PowerProtection.kicad_sch (KiCad schematic)
At the start: 18 parts, among them IC1 LM74502DDFR, Q1 PSMN012-100YS, Q2 PSMN012-100YS

Commit message: updated library parts + new 15V TVS diode
Parts:
- removed D2: SMBJ30CD, UTSVT_Power:SMBJ30CD, symbol Device:D_Zener
- added D2: SMBJ15CA, Diode_SMD:D_SMB, symbol PP:SMBJ15CA
- D1: footprint UTSVT_Passives:SODFL5026X125N -> LHRS_Passives:SODFL5026X125N
- IC1: footprint UTSVT_Power:LM74502DDFR -> LHRS_Power:LM74502DDFR
- R5: value 9.53k -> 7.32k
- R6: value 100k -> 15.8k
- R7: value 13.7k -> 100k
Connections:
- net GND: now also D2.1 (A1)
- net Vin: now also D2.2 (A2)
Other:
- note added: "Output of Python Calulations for Resistor Values"
- note removed: "1.235 is Enable/UVLO falling threshold on data sheet worst case(may want to change to average)"
- note removed: "Overvoltage Protection: 14.37V Vovr = (R2 * Vov)/(R1 + R2) Vov = Vovr * (R1 + R2) / R2 14.37 = 1.25 * (100k + 9.53k) / 100k 133uA loss"
- moved on the sheet: C6, C7, R4, R5, R6, R7

Commit message: updated libraries + changed resistor orientaiton
Parts:
- D2: symbol PP:SMBJ15CA -> lhrs_power:SMBJ15CA
- Q1, Q2: footprint UTSVT_Power:PSMN012-100YS -> Package_TO_SOT_SMD:LFPAK56; symbol utsvt_power:PSMN012-100YS -> lhrs_power:PSMN012-100YS
Connections:
- net EN/UVLO: now also R6.2, R7.2; no longer R6.1, R7.1
- net GND: now also R6.1; no longer R7.2
- net Vin: now also R7.1; no longer R6.2
Other:
- moved on the sheet: Q2
Changed lines of the file:
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@@
 	(wire
 		(pts
-			(xy 87.63 41.91) (xy 83.82 41.91)
+			(xy 83.82 41.91) (xy 87.63 41.91)
 		)
 		(stroke
@@
 	(wire
 		(pts
-			(xy 87.63 46.99) (xy 83.82 46.99)
-		)
-		(stroke
-			(width 0)
-			(type default)
-		)
-	)
-	(wire
-		(pts
 			(xy 25.4 44.45) (xy 34.29 44.45)
 		)
@@
 	(wire
 		(pts
+			(xy 83.82 46.99) (xy 87.63 46.99)
+		)
+		(stroke
+			(width 0)
+			(type default)
+		)
+	)
+	(wire
+		(pts
 			(xy 134.62 81.28) (xy 134.62 82.55)
 		)
@@
 	)
 	(symbol
-		(lib_id "PP:SMBJ15CA")
+		(lib_id "lhrs_power:SMBJ15CA")
 		(at 26.67 50.8 90)
 		(unit 1)
@@
 	(symbol
 		(lib_id "Device:R_US")
-		(at 139.7 90.17 0)
+		(at 139.7 90.17 180)
 		(unit 1)
 		(body_style 1)
@@
 		(in_pos_files yes)
 		(dnp no)
-		(property "Reference" "R7"
-			(at 142.24 90.17 90)
+		(property "Reference" "R6"
+			(at 141.986 90.17 90)
 			(show_name no)
 			(do_not_autoplace no)
@@
 			)
 		)
-		(property "Value" "100k"
-			(at 137.414 90.17 90)
+		(property "Value" "15.8k"
+			(at 136.906 90.424 90)
 			(show_name no)
 			(do_not_autoplace no)
@@
 		)
 		(property "Footprint" "Resistor_SMD:R_0603_1608Metric_Pad0.98x0.95mm_HandSolder"
-			(at 140.716 90.424 90)
+			(at 138.684 89.916 90)
 			(hide yes)
 			(show_name no)
@@
 			)
 		)
-		(property "P/N" "CRCW060310K0FKEI"
-			(at 139.7 90.17 0)
+		(property "P/N" "CRCW0603137KFKEA"
+			(at 139.7 90.17 90)
 			(hide yes)
 			(show_name no)
@@
 			)
 		)
-		(property "LCSC P/N" "C25804"
-			(at 139.7 90.17 0)
+		(property "LCSC P/N" "C2090646"
+			(at 139.7 90.17 90)
 			(hide yes)
 			(show_name no)
@@
 			(project "PowerProtection"
 				(path "/a968d2b9-0c0e-491c-a5a4-aacd8448ff64"
-					(reference "R7")
+					(reference "R6")
 					(unit 1)
 				)
@@
 	(symbol
 		(lib_id "Device:R_US")
-		(at 134.62 77.47 180)
-		(unit 1)
-		(body_style 1)
-		(exclude_from_sim no)
-		(in_bom yes)
-		(on_board yes)
-		(in_pos_files yes)
-		(dnp no)
-		(property "Reference" "R6"
-			(at 136.906 77.47 90)
-			(show_name no)
-			(do_not_autoplace no)
-			(effects
-				(font
-					(size 1.27 1.27)
-				)
-			)
-		)
-		(property "Value" "15.8k"
-			(at 131.826 77.724 90)
-			(show_name no)
-			(do_not_autoplace no)
-			(effects
-				(font
-					(size 1.27 1.27)
-				)
-			)
-		)
-		(property "Footprint" "Resistor_SMD:R_0603_1608Metric_Pad0.98x0.95mm_HandSolder"
-			(at 133.604 77.216 90)
-			(hide yes)
-			(show_name no)
-			(do_not_autoplace no)
-			(effects
-				(font
-					(size 1.27 1.27)
-				)
-			)
-		)
-		(property "Datasheet" ""
-			(at 134.62 77.47 0)
-			(hide yes)
-			(show_name no)
-			(do_not_autoplace no)
-			(effects
-				(font
-					(size 1.27 1.27)
-				)
-			)
-		)
-		(property "Description" "Resistor, US symbol"
-			(at 134.62 77.47 0)
-			(hide yes)
-			(show_name no)
-			(do_not_autoplace no)
-			(effects
-				(font
-					(size 1.27 1.27)
-				)
-			)
-		)
-		(property "P/N" "CRCW0603137KFKEA"
-			(at 134.62 77.47 90)
-			(hide yes)
-			(show_name no)
-			(do_not_autoplace no)
-			(effects
-				(font
-					(size 1.27 1.27)
-				)
-			)
-		)
-		(property "LCSC P/N" "C2090646"
-			(at 134.62 77.47 90)
-			(hide yes)
-			(show_name no)
-			(do_not_autoplace no)
-			(effects
-				(font
-					(size 1.27 1.27)
-				)
-			)
-		)
-		(pin "1"
-		)
-		(pin "2"
-		)
-		(instances
-			(project "PowerProtection"
-				(path "/a968d2b9-0c0e-491c-a5a4-aacd8448ff64"
-					(reference "R6")
-					(unit 1)
-				)
-			)
-		)
-	)
-	(symbol
-		(lib_id "Device:R_US")
 		(at 67.31 57.15 90)
 		(unit 1)
@@
 	)
 	(symbol
-		(lib_id "utsvt_power:PSMN012-100YS")
-		(at 59.69 38.1 90)
+		(lib_id "lhrs_power:PSMN012-100YS")
+		(at 55.88 46.99 90)
 		(unit 1)
 		(body_style 1)
@@
 		(dnp no)
 		(property "Reference" "Q1"
-			(at 51.816 38.608 90)
+			(at 52.578 38.862 90)
 			(show_name no)
 			(do_not_autoplace no)
@@
 		)
 		(property "Value" "PSMN012-100YS"
-			(at 50.8 40.894 90)
+			(at 51.054 41.148 90)
 			(show_name no)
 			(do_not_autoplace no)
@@
 			)
 		)
-		(property "Footprint" "UTSVT_Power:PSMN012-100YS"
+		(property "Footprint" "Package_TO_SOT_SMD:LFPAK56"
 			(at 53.34 41.91 0)
 			(hide yes)
@@
 		)
 		(property "P/N" "PSMN012-100YSFX"
-			(at 55.88 46.99 90)
+			(at 55.88 46.99 0)
 			(hide yes)
 			(show_name no)
@@
 		)
 		(property "LCSC P/N" "C20443035"
-			(at 55.88 46.99 90)
+			(at 55.88 46.99 0)
 			(hide yes)
 			(show_name no)
@@
 	)
 	(symbol
-		(lib_name "PSMN012-100YS_1")
-		(lib_id "utsvt_power:PSMN012-100YS")
-		(at 96.52 36.83 90)
+		(lib_id "lhrs_power:PSMN012-100YS")
+		(at 93.98 46.99 270)
+		(mirror x)
 		(unit 1)
 		(body_style 1)
@@
 		(dnp no)
 		(property "Reference" "Q2"
-			(at 98.298 39.116 90)
+			(at 100.584 38.608 90)
 			(show_name no)
 			(do_not_autoplace no)
@@
 		)
 		(property "Value" "PSMN012-100YS"
-			(at 99.06 41.402 90)
+			(at 99.06 40.894 90)
 			(show_name no)
 			(do_not_autoplace no)
@@
 			)
 		)
-		(property "Footprint" "UTSVT_Power:PSMN012-100YS"
-			(at 90.17 40.64 0)
+		(property "Footprint" "Package_TO_SOT_SMD:LFPAK56"
+			(at 96.52 41.91 0)
 			(hide yes)
 			(show_name no)
@@
 		)
 		(property "Datasheet" "kicad-embed://PSMN012-100YS.pdf"
-			(at 105.41 45.72 0)
+			(at 81.28 46.99 0)
 			(hide yes)
 			(show_name no)
@@
 		)
 		(property "Description" "N-MOSFET transistor, drain/source/gate"
-			(at 92.71 45.72 0)
+			(at 93.98 46.99 0)
 			(hide yes)
 			(show_name no)
@@
 		)
 		(property "Sim.Device" "NMOS"
-			(at 109.855 45.72 0)
+			(at 76.835 46.99 0)
 			(hide yes)
 			(show_name no)
@@
 		)
 		(property "Sim.Type" "VDMOS"
-			(at 111.76 45.72 0)
+			(at 74.93 46.99 0)
 			(hide yes)
 			(show_name no)
@@
 		)
 		(property "Sim.Pins" "1=D 2=G 3=S"
-			(at 107.95 45.72 0)
+			(at 78.74 46.99 0)
 			(hide yes)
 			(show_name no)
@@
 		)
 		(property "P/N" "PSMN012-100YSFX"
-			(at 92.71 45.72 90)
+			(at 93.98 46.99 0)
 			(hide yes)
 			(show_name no)
@@
 		)
 		(property "LCSC P/N" "C20443035"
-			(at 92.71 45.72 90)
+			(at 93.98 46.99 0)
 			(hide yes)
 			(show_name no)
@@
 					(unit 1)
 				)
+			)
+		)
+	)
+	(symbol
+		(lib_id "Device:R_US")
+		(at 134.62 77.47 0)
+		(unit 1)
+		(body_style 1)
+		(exclude_from_sim no)
+		(in_bom yes)
+		(on_board yes)
+		(in_pos_files yes)
+		(dnp no)
+		(property "Reference" "R7"
+			(at 137.16 77.47 90)
+			(show_name no)
+			(do_not_autoplace no)
+			(effects
+				(font
+					(size 1.27 1.27)
+				)
+			)
+		)
+		(property "Value" "100k"
+			(at 132.334 77.47 90)
+			(show_name no)
+			(do_not_autoplace no)
+			(effects
+				(font
+					(size 1.27 1.27)
+				)
+			)
+		)
+		(property "Footprint" "Resistor_SMD:R_0603_1608Metric_Pad0.98x0.95mm_HandSolder"
+			(at 135.636 77.724 90)
+			(hide yes)
+			(show_name no)
+			(do_not_autoplace no)
+			(effects
+				(font
+					(size 1.27 1.27)
+				)
+			)
+		)
+		(property "Datasheet" ""
+			(at 134.62 77.47 0)
+			(hide yes)
+			(show_name no)
+			(do_not_autoplace no)
+			(effects
+				(font
+					(size 1.27 1.27)
+				)
+			)
+		)
+		(property "Description" "Resistor, US symbol"
+			(at 134.62 77.47 0)
+			(hide yes)
+			(show_name no)
+			(do_not_autoplace no)
+			(effects
+				(font
+					(size 1.27 1.27)
+				)
+			)
+		)
+		(property "P/N" "CRCW060310K0FKEI"
+			(at 134.62 77.47 0)
+			(hide yes)
+			(show_name no)
+			(do_not_autoplace no)
+			(effects
+				(font
+					(size 1.27 1.27)
+				)
+			)
+		)
+		(property "LCSC P/N" "C25804"
+			(at 134.62 77.47 0)
+			(hide yes)
+			(show_name no)
+			(do_not_autoplace no)
+			(effects
+				(font
+					(size 1.27 1.27)
+				)
+			)
+		)
+		(pin "1"
+		)
+		(pin "2"
+		)
+		(instances
+			(project "PowerProtection"
+				(path "/a968d2b9-0c0e-491c-a5a4-aacd8448ff64"
+					(reference "R7")
+					(unit 1)
+				)

Commit message: changed linbrary linking
Parts:
- IC1: symbol UTSVT_ICs:LM74502HDDFR -> lhrs_power:LM74502HDDFR
