File: LHRS_Design_Blocks.kicad_blocks/PowerProtection.kicad_block/PowerProtection.kicad_sch (KiCad schematic)
At the start: 18 parts, among them IC1 LM74502DDFR, Q1 PSMN012-100YS, Q2 PSMN012-100YS

Commit message: updated to match standard parts list
Parts:
- C1: LCSC P/N C14663 -> C1591; P/N MLASH168SB7104KTNA01 -> CL10B104KB8NNNC
- C2: LCSC P/N C15849 -> C559769; P/N MLASU168SB5105KTNA01 -> CC0603KRX7R9BB105
- C3: LCSC P/N C344195 -> C107083; Mouser Part Number 963-MSASU168SB7224KT -> CC0603KRX7R9BB224
- C4: LCSC P/N C57112 -> C100042; P/N MSASH168SB5103KTNA01 -> CC0603KRX7R9BB103
- C5: P/N GRM21BR61H106KE43K -> GRM21BR61H106KE43L
- C6, C7: LCSC P/N (none) -> C1591; P/N (none) -> CL10B104KB8NNNC
- R1: Mouser Part Number 71-CRCW060310K0FKEI -> 0603WAF1002T5E
- R4, R7: P/N CRCW0603100KFKEE -> 0603WAF1003T5E
Connections:
- net EN/UVLO: now also C7.1; no longer C6.2
- net GND: now also C6.2, C7.2; no longer C6.1, C7.1
- net OV: now also C6.1; no longer C7.2
Changed lines of the file:
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@@
-	)
-	(symbol
-		(lib_id "Device:C")
-		(at 129.54 90.17 180)
-		(unit 1)
-		(body_style 1)
-		(exclude_from_sim no)
-		(in_bom yes)
-		(on_board yes)
-		(in_pos_files yes)
-		(dnp no)
-		(property "Reference" "C6"
-			(at 125.984 89.154 90)
-			(show_name no)
-			(do_not_autoplace no)
-			(effects
-				(font
-					(size 1.27 1.27)
-				)
-				(justify left)
-			)
-		)
-		(property "Value" "0.1u"
-			(at 132.842 88.392 90)
-			(show_name no)
-			(do_not_autoplace no)
-			(effects
-				(font
-					(size 1.27 1.27)
-				)
-				(justify left)
-			)
-		)
-		(property "Footprint" "Capacitor_SMD:C_0603_1608Metric_Pad1.08x0.95mm_HandSolder"
-			(at 128.5748 86.36 0)
-			(hide yes)
-			(show_name no)
-			(do_not_autoplace no)
-			(effects
-				(font
-					(size 1.27 1.27)
-				)
-			)
-		)
-		(property "Datasheet" ""
-			(at 129.54 90.17 0)
-			(hide yes)
-			(show_name no)
-			(do_not_autoplace no)
-			(effects
-				(font
-					(size 1.27 1.27)
-				)
-			)
-		)
-		(property "Description" "Unpolarized capacitor"
-			(at 129.54 90.17 0)
-			(hide yes)
-			(show_name no)
-			(do_not_autoplace no)
-			(effects
-				(font
-					(size 1.27 1.27)
-				)
-			)
-		)
-		(pin "2"
-		)
-		(pin "1"
-		)
-		(instances
-			(project "PowerProtection"
-				(path "/a968d2b9-0c0e-491c-a5a4-aacd8448ff64"
-					(reference "C6")
-					(unit 1)
-				)
-			)
-		)
 	)
 	(symbol
@@
 			)
 		)
-		(property "Mouser Part Number" "963-MSASU168SB7224KT"
+		(property "Mouser Part Number" "CC0603KRX7R9BB224"
 			(at 54.61 81.28 0)
 			(hide yes)
@@
 			)
 		)
-		(property "LCSC P/N" "C344195"
+		(property "LCSC P/N" "C107083"
 			(at 54.61 81.28 0)
 			(hide yes)
@@
 			)
 		)
-		(property "Mouser Part Number" "71-CRCW060310K0FKEI"
+		(property "Mouser Part Number" "0603WAF1002T5E"
 			(at 43.18 62.23 0)
 			(hide yes)
@@
 			)
 		)
-		(property "P/N" "MLASH168SB7104KTNA01"
+		(property "P/N" "CL10B104KB8NNNC"
 			(at 34.29 50.8 0)
 			(hide yes)
@@
 			)
 		)
-		(property "LCSC P/N" "C14663"
+		(property "LCSC P/N" "C1591"
 			(at 34.29 50.8 0)
 			(hide yes)
@@
 	)
 	(symbol
-		(lib_id "Device:C")
-		(at 110.49 90.17 180)
-		(unit 1)
-		(body_style 1)
-		(exclude_from_sim no)
-		(in_bom yes)
-		(on_board yes)
-		(in_pos_files yes)
-		(dnp no)
-		(property "Reference" "C7"
-			(at 107.188 88.9 90)
-			(show_name no)
-			(do_not_autoplace no)
-			(effects
-				(font
-					(size 1.27 1.27)
-				)
-				(justify left)
-			)
-		)
-		(property "Value" "0.1u"
-			(at 114.046 88.392 90)
-			(show_name no)
-			(do_not_autoplace no)
-			(effects
-				(font
-					(size 1.27 1.27)
-				)
-				(justify left)
-			)
-		)
-		(property "Footprint" "Capacitor_SMD:C_0603_1608Metric_Pad1.08x0.95mm_HandSolder"
-			(at 109.5248 86.36 0)
-			(hide yes)
-			(show_name no)
-			(do_not_autoplace no)
-			(effects
-				(font
-					(size 1.27 1.27)
-				)
-			)
-		)
-		(property "Datasheet" ""
-			(at 110.49 90.17 0)
-			(hide yes)
-			(show_name no)
-			(do_not_autoplace no)
-			(effects
-				(font
-					(size 1.27 1.27)
-				)
-			)
-		)
-		(property "Description" "Unpolarized capacitor"
-			(at 110.49 90.17 0)
-			(hide yes)
-			(show_name no)
-			(do_not_autoplace no)
-			(effects
-				(font
-					(size 1.27 1.27)
-				)
-			)
-		)
-		(pin "2"
-		)
-		(pin "1"
-		)
-		(instances
-			(project "PowerProtection"
-				(path "/a968d2b9-0c0e-491c-a5a4-aacd8448ff64"
-					(reference "C7")
-					(unit 1)
-				)
-			)
-		)
-	)
-	(symbol
 		(lib_id "lhrs_power:LM74502HDDFR")
 		(at 58.42 77.47 0)
@@
 	)
 	(symbol
+		(lib_id "Device:C")
+		(at 110.49 90.17 0)
+		(unit 1)
+		(body_style 1)
+		(exclude_from_sim no)
+		(in_bom yes)
+		(on_board yes)
+		(in_pos_files yes)
+		(dnp no)
+		(property "Reference" "C6"
+			(at 113.284 89.154 0)
+			(show_name no)
+			(do_not_autoplace no)
+			(effects
+				(font
+					(size 1.27 1.27)
+				)
+				(justify left)
+			)
+		)
+		(property "Value" "0.1u"
+			(at 113.03 91.44 0)
+			(show_name no)
+			(do_not_autoplace no)
+			(effects
+				(font
+					(size 1.27 1.27)
+				)
+				(justify left)
+			)
+		)
+		(property "Footprint" "Capacitor_SMD:C_0603_1608Metric_Pad1.08x0.95mm_HandSolder"
+			(at 111.4552 93.98 0)
+			(hide yes)
+			(show_name no)
+			(do_not_autoplace no)
+			(effects
+				(font
+					(size 1.27 1.27)
+				)
+			)
+		)
+		(property "Datasheet" ""
+			(at 110.49 90.17 0)
+			(hide yes)
+			(show_name no)
+			(do_not_autoplace no)
+			(effects
+				(font
+					(size 1.27 1.27)
+				)
+			)
+		)
+		(property "Description" "Unpolarized capacitor"
+			(at 110.49 90.17 0)
+			(hide yes)
+			(show_name no)
+			(do_not_autoplace no)
+			(effects
+				(font
+					(size 1.27 1.27)
+				)
+			)
+		)
+		(property "P/N" "CL10B104KB8NNNC"
+			(at 110.49 90.17 0)
+			(hide yes)
+			(show_name no)
+			(do_not_autoplace no)
+			(effects
+				(font
+					(size 1.27 1.27)
+				)
+			)
+		)
+		(property "LCSC P/N" "C1591"
+			(at 110.49 90.17 0)
+			(hide yes)
+			(show_name no)
+			(do_not_autoplace no)
+			(effects
+				(font
+					(size 1.27 1.27)
+				)
+			)
+		)
+		(pin "1"
+		)
+		(pin "2"
+		)
+		(instances
+			(project "PowerProtection"
+				(path "/a968d2b9-0c0e-491c-a5a4-aacd8448ff64"
+					(reference "C6")
+					(unit 1)
+				)
+			)
+		)
+	)
+	(symbol
 		(lib_id "ECE319H:C")
 		(at 60.96 63.5 0)
@@
 			)
 		)
-		(property "P/N" "MSASH168SB5103KTNA01"
+		(property "P/N" "CC0603KRX7R9BB103"
 			(at 60.96 63.5 0)
 			(hide yes)
@@
 			)
 		)
-		(property "LCSC P/N" "C57112 "
+		(property "LCSC P/N" "C100042"
 			(at 60.96 63.5 0)
 			(hide yes)
@@
 			)
 		)
-		(property "P/N" "GRM21BR61H106KE43K"
+		(property "P/N" "GRM21BR61H106KE43L"
 			(at 109.22 53.975 0)
 			(hide yes)
@@
 			)
 		)
-		(property "P/N" "MLASU168SB5105KTNA01"
+		(property "P/N" "CC0603KRX7R9BB105"
 			(at 32.385 86.36 0)
 			(hide yes)
@@
 			)
 		)
-		(property "LCSC P/N" "C15849"
+		(property "LCSC P/N" "C559769"
 			(at 35.56 83.82 0)
 			(hide yes)
@@
 				(path "/a968d2b9-0c0e-491c-a5a4-aacd8448ff64"
 					(reference "C2")
+					(unit 1)
+				)
+			)
+		)
+	)
+	(symbol
+		(lib_id "Device:C")
+		(at 129.54 90.17 0)
+		(unit 1)
+		(body_style 1)
+		(exclude_from_sim no)
+		(in_bom yes)
+		(on_board yes)
+		(in_pos_files yes)
+		(dnp no)
+		(property "Reference" "C7"
+			(at 132.08 88.9 0)
+			(show_name no)
+			(do_not_autoplace no)
+			(effects
+				(font
+					(size 1.27 1.27)
+				)
+				(justify left)
+			)
+		)
+		(property "Value" "0.1u"
+			(at 131.826 91.44 0)
+			(show_name no)
+			(do_not_autoplace no)
+			(effects
+				(font
+					(size 1.27 1.27)
+				)
+				(justify left)
+			)
+		)
+		(property "Footprint" "Capacitor_SMD:C_0603_1608Metric_Pad1.08x0.95mm_HandSolder"
+			(at 130.5052 93.98 0)
+			(hide yes)
+			(show_name no)
+			(do_not_autoplace no)
+			(effects
+				(font
+					(size 1.27 1.27)
+				)
+			)
+		)
+		(property "Datasheet" ""
+			(at 129.54 90.17 0)
+			(hide yes)
+			(show_name no)
+			(do_not_autoplace no)
+			(effects
+				(font
+					(size 1.27 1.27)
+				)
+			)
+		)
+		(property "Description" "Unpolarized capacitor"
+			(at 129.54 90.17 0)
+			(hide yes)
+			(show_name no)
+			(do_not_autoplace no)
+			(effects
+				(font
+					(size 1.27 1.27)
+				)
+			)
+		)
+		(property "P/N" "CL10B104KB8NNNC"
+			(at 129.54 90.17 0)
+			(hide yes)
+			(show_name no)
+			(do_not_autoplace no)
+			(effects
+				(font
+					(size 1.27 1.27)
+				)
+			)
+		)
+		(property "LCSC P/N" "C1591"
+			(at 129.54 90.17 0)
+			(hide yes)
+			(show_name no)
+			(do_not_autoplace no)
+			(effects
+				(font
+					(size 1.27 1.27)
+				)
+			)
+		)
+		(pin "1"
+		)
+		(pin "2"
+		)
+		(instances
+			(project "PowerProtection"
+				(path "/a968d2b9-0c0e-491c-a5a4-aacd8448ff64"
+					(reference "C7")
 					(unit 1)
 				)
@@
 			)
 		)
-		(property "P/N" "CRCW0603100KFKEE"
+		(property "P/N" "0603WAF1003T5E"
 			(at 115.57 77.47 0)
 			(hide yes)
@@
 			)
 		)
-		(property "P/N" "CRCW0603100KFKEE"
+		(property "P/N" "0603WAF1003T5E"
 			(at 134.62 77.47 0)
 			(hide yes)

Commit message: finalize P/N selection
Parts:
- C3: Mouser Part Number CC0603KRX7R9BB224 -> (none); P/N MSASU168SB7224KTNB25 -> CC0603KRX7R9BB224
- D1: LCSC P/N (none) -> C183490; P/N (none) -> SMAF4758A
- R1: Mouser Part Number 0603WAF1002T5E -> (none); P/N CRCW060310K0FKEI -> 0603WAF1002T5E
Changed lines of the file:
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@@
+			)
+		)
+		(property "P/N" "SMAF4758A"
+			(at 43.18 83.82 0)
+			(hide yes)
+			(show_name no)
+			(do_not_autoplace no)
+			(effects
+				(font
+					(size 1.27 1.27)
+				)
+			)
+		)
+		(property "LCSC P/N" "C183490"
+			(at 43.18 83.82 0)
+			(hide yes)
+			(show_name no)
+			(do_not_autoplace no)
+			(effects
+				(font
+					(size 1.27 1.27)
+				)
 			)
 		)
@@
 			)
 		)
-		(property "P/N" "MSASU168SB7224KTNB25"
-			(at 54.61 81.28 0)
-			(hide yes)
-			(show_name no)
-			(do_not_autoplace no)
-			(effects
-				(font
-					(size 1.27 1.27)
-				)
-			)
-		)
-		(property "Mouser Part Number" "CC0603KRX7R9BB224"
+		(property "P/N" "CC0603KRX7R9BB224"
 			(at 54.61 81.28 0)
 			(hide yes)
@@
 			)
 		)
-		(property "P/N" "CRCW060310K0FKEI"
+		(property "P/N" "0603WAF1002T5E"
 			(at 43.18 62.23 0)
 			(hide yes)
-			(show_name no)
-			(do_not_autoplace no)
-			(effects
-				(font
-					(size 1.27 1.27)
-				)
-			)
-		)
-		(property "Mouser Part Number" "0603WAF1002T5E"
-			(at 43.18 62.23 0)
-			(hide yes)
