File: LHRS_Design_Blocks.kicad_blocks/USB-C Connector.kicad_block/USB-C Connector.kicad_sch (KiCad schematic)
At the start: 6 parts, among them J1 USB_C_Receptacle_USB2.0_16P

Commit message: bidirectional, updated comments
Other:
- note added: "If using USB-C PD, remove CC1 and CC2 pull down resistor, if not using USB-C PD, keep them"
- note removed: "Pulldowns for 5V USB-C PD"
- moved on the sheet: D2, R1, R2
