File: LHRS_Design_Blocks.kicad_blocks/Power_Mux_12V.kicad_block/Power_Mux_12V.kicad_sch (KiCad schematic)
At the start: 11 parts

Commit message: fixed some erc issues
Parts:
- C90: renamed from C?; footprint (none) -> Capacitor_SMD:C_0603_1608Metric_Pad1.08x0.95mm_HandSolder
- R122, R123, R124, R125, R126, R127, R128, R129, R130: renamed from R?; footprint (none) -> Resistor_SMD:R_0603_1608Metric_Pad0.98x0.95mm_HandSolder
- U17: renamed from U?; footprint LHRS_Power:IC_TPS2121RUXR -> LHRS_ICs:TPS2121RUXR
Connections:
- net PR1 is gone; now on net PRI: U17.6 (PR1)
Changed lines of the file:
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@@
 	(wire
 		(pts
+			(xy 149.86 67.31) (xy 149.86 69.85)
+		)
+		(stroke
+			(width 0)
+			(type default)
+		)
+	)
+	(wire
+		(pts
 			(xy 112.395 77.47) (xy 117.475 77.47)
 		)
@@
 	(wire
 		(pts
+			(xy 142.875 67.31) (xy 149.86 67.31)
+		)
+		(stroke
+			(width 0)
+			(type default)
+		)
+	)
+	(wire
+		(pts
 			(xy 53.34 52.705) (xy 53.34 55.245)
 		)
@@
 		)
 	)
-	(label "PR1"
+	(label "PRI"
 		(at 112.395 67.31 0)
 		(effects
@@
 	(hierarchical_label "GND"
 		(shape input)
-		(at 142.875 67.31 270)
+		(at 149.86 69.85 270)
 		(effects
 			(font
@@
 		(dnp no)
 		(fields_autoplaced yes)
-		(property "Reference" "R?"
+		(property "Reference" "R126"
 			(at 55.88 45.7199 0)
 			(show_name no)
@@
 			)
 		)
-		(property "Footprint" ""
+		(property "Footprint" "Resistor_SMD:R_0603_1608Metric_Pad0.98x0.95mm_HandSolder"
 			(at 53.34 46.99 0)
 			(hide yes)
@@
 		(instances
 			(project "PS-BPSLeader"
-				(path "/d4a4ed4f-0983-4aef-b212-0e3284ab3963/69244dac-f10b-499c-a2b2-3cdf1370aa1f/1a445fba-997a-4276-b1d7-6bccd354442b"
-					(reference "R?")
+				(path "/d4a4ed4f-0983-4aef-b212-0e3284ab3963/69244dac-f10b-499c-a2b2-3cdf1370aa1f/0f3e3992-4755-4e76-a363-7a4e463e2a3d"
+					(reference "R126")
 					(unit 1)
 				)
@@
 		(dnp no)
 		(fields_autoplaced yes)
-		(property "Reference" "R?"
+		(property "Reference" "R125"
 			(at 41.91 56.5149 0)
 			(show_name no)
@@
 			)
 		)
-		(property "Footprint" ""
+		(property "Footprint" "Resistor_SMD:R_0603_1608Metric_Pad0.98x0.95mm_HandSolder"
 			(at 39.37 57.785 0)
 			(hide yes)
@@
 		(instances
 			(project "PS-BPSLeader"
-				(path "/d4a4ed4f-0983-4aef-b212-0e3284ab3963/69244dac-f10b-499c-a2b2-3cdf1370aa1f/1a445fba-997a-4276-b1d7-6bccd354442b"
-					(reference "R?")
+				(path "/d4a4ed4f-0983-4aef-b212-0e3284ab3963/69244dac-f10b-499c-a2b2-3cdf1370aa1f/0f3e3992-4755-4e76-a363-7a4e463e2a3d"
+					(reference "R125")
 					(unit 1)
 				)
@@
 		(dnp no)
 		(fields_autoplaced yes)
-		(property "Reference" "R?"
+		(property "Reference" "R123"
 			(at 29.21 56.5149 0)
 			(show_name no)
@@
 			)
 		)
-		(property "Footprint" ""
+		(property "Footprint" "Resistor_SMD:R_0603_1608Metric_Pad0.98x0.95mm_HandSolder"
 			(at 26.67 57.785 0)
 			(hide yes)
@@
 		(instances
 			(project "PS-BPSLeader"
-				(path "/d4a4ed4f-0983-4aef-b212-0e3284ab3963/69244dac-f10b-499c-a2b2-3cdf1370aa1f/1a445fba-997a-4276-b1d7-6bccd354442b"
-					(reference "R?")
+				(path "/d4a4ed4f-0983-4aef-b212-0e3284ab3963/69244dac-f10b-499c-a2b2-3cdf1370aa1f/0f3e3992-4755-4e76-a363-7a4e463e2a3d"
+					(reference "R123")
 					(unit 1)
 				)
@@
 		(dnp no)
 		(fields_autoplaced yes)
-		(property "Reference" "R?"
+		(property "Reference" "R122"
 			(at 29.21 45.7199 0)
 			(show_name no)
@@
 			)
 		)
-		(property "Footprint" ""
+		(property "Footprint" "Resistor_SMD:R_0603_1608Metric_Pad0.98x0.95mm_HandSolder"
 			(at 26.67 46.99 0)
 			(hide yes)
@@
 		(instances
 			(project "PS-BPSLeader"
-				(path "/d4a4ed4f-0983-4aef-b212-0e3284ab3963/69244dac-f10b-499c-a2b2-3cdf1370aa1f/1a445fba-997a-4276-b1d7-6bccd354442b"
-					(reference "R?")
+				(path "/d4a4ed4f-0983-4aef-b212-0e3284ab3963/69244dac-f10b-499c-a2b2-3cdf1370aa1f/0f3e3992-4755-4e76-a363-7a4e463e2a3d"
+					(reference "R122")
 					(unit 1)
 				)
@@
 		(dnp no)
 		(fields_autoplaced yes)
-		(property "Reference" "R?"
+		(property "Reference" "R124"
 			(at 41.91 45.7199 0)
 			(show_name no)
@@
 			)
 		)
-		(property "Footprint" ""
+		(property "Footprint" "Resistor_SMD:R_0603_1608Metric_Pad0.98x0.95mm_HandSolder"
 			(at 39.37 46.99 0)
 			(hide yes)
@@
 		(instances
 			(project "PS-BPSLeader"
-				(path "/d4a4ed4f-0983-4aef-b212-0e3284ab3963/69244dac-f10b-499c-a2b2-3cdf1370aa1f/1a445fba-997a-4276-b1d7-6bccd354442b"
-					(reference "R?")
+				(path "/d4a4ed4f-0983-4aef-b212-0e3284ab3963/69244dac-f10b-499c-a2b2-3cdf1370aa1f/0f3e3992-4755-4e76-a363-7a4e463e2a3d"
+					(reference "R124")
 					(unit 1)
 				)
@@
 		(dnp no)
 		(fields_autoplaced yes)
-		(property "Reference" "R?"
+		(property "Reference" "R130"
 			(at 113.665 94.6149 0)
 			(show_name no)
@@
 			)
 		)
-		(property "Footprint" ""
+		(property "Footprint" "Resistor_SMD:R_0603_1608Metric_Pad0.98x0.95mm_HandSolder"
 			(at 111.76 95.885 0)
 			(hide yes)
@@
 		(instances
 			(project "PS-BPSLeader"
-				(path "/d4a4ed4f-0983-4aef-b212-0e3284ab3963/69244dac-f10b-499c-a2b2-3cdf1370aa1f/1a445fba-997a-4276-b1d7-6bccd354442b"
-					(reference "R?")
+				(path "/d4a4ed4f-0983-4aef-b212-0e3284ab3963/69244dac-f10b-499c-a2b2-3cdf1370aa1f/0f3e3992-4755-4e76-a363-7a4e463e2a3d"
+					(reference "R130")
 					(unit 1)
 				)
@@
 		(dnp no)
 		(fields_autoplaced yes)
-		(property "Reference" "U?"
+		(property "Reference" "U17"
 			(at 130.175 54.61 0)
 			(show_name no)
@@
 			)
 		)
-		(property "Footprint" "LHRS_Power:IC_TPS2121RUXR"
+		(property "Footprint" "LHRS_ICs:TPS2121RUXR"
 			(at 130.175 80.01 0)
 			(hide yes)
@@
 		(instances
 			(project "PS-BPSLeader"
-				(path "/d4a4ed4f-0983-4aef-b212-0e3284ab3963/69244dac-f10b-499c-a2b2-3cdf1370aa1f/1a445fba-997a-4276-b1d7-6bccd354442b"
-					(reference "U?")
+				(path "/d4a4ed4f-0983-4aef-b212-0e3284ab3963/69244dac-f10b-499c-a2b2-3cdf1370aa1f/0f3e3992-4755-4e76-a363-7a4e463e2a3d"
+					(reference "U17")
 					(unit 1)
 				)
@@
 		(dnp no)
 		(fields_autoplaced yes)
-		(property "Reference" "R?"
+		(property "Reference" "R128"
 			(at 68.58 45.7199 0)
 			(show_name no)
@@
 			)
 		)
-		(property "Footprint" ""
+		(property "Footprint" "Resistor_SMD:R_0603_1608Metric_Pad0.98x0.95mm_HandSolder"
 			(at 66.675 46.99 0)
 			(hide yes)
@@
 		(instances
 			(project "PS-BPSLeader"
-				(path "/d4a4ed4f-0983-4aef-b212-0e3284ab3963/69244dac-f10b-499c-a2b2-3cdf1370aa1f/1a445fba-997a-4276-b1d7-6bccd354442b"
-					(reference "R?")
+				(path "/d4a4ed4f-0983-4aef-b212-0e3284ab3963/69244dac-f10b-499c-a2b2-3cdf1370aa1f/0f3e3992-4755-4e76-a363-7a4e463e2a3d"
+					(reference "R128")
 					(unit 1)
 				)
@@
 		(dnp no)
 		(fields_autoplaced yes)
-		(property "Reference" "C?"
+		(property "Reference" "C90"
 			(at 102.87 94.6212 0)
 			(show_name no)
@@
 			)
 		)
-		(property "Footprint" ""
+		(property "Footprint" "Capacitor_SMD:C_0603_1608Metric_Pad1.08x0.95mm_HandSolder"
 			(at 105.41 95.885 0)
 			(hide yes)
@@
 		(instances
 			(project "PS-BPSLeader"
-				(path "/d4a4ed4f-0983-4aef-b212-0e3284ab3963/69244dac-f10b-499c-a2b2-3cdf1370aa1f/1a445fba-997a-4276-b1d7-6bccd354442b"
-					(reference "C?")
+				(path "/d4a4ed4f-0983-4aef-b212-0e3284ab3963/69244dac-f10b-499c-a2b2-3cdf1370aa1f/0f3e3992-4755-4e76-a363-7a4e463e2a3d"
+					(reference "C90")
 					(unit 1)
 				)
@@
 		(dnp no)
 		(fields_autoplaced yes)
-		(property "Reference" "R?"
+		(property "Reference" "R127"
 			(at 55.88 56.5149 0)
 			(show_name no)
@@
 			)
 		)
-		(property "Footprint" ""
+		(property "Footprint" "Resistor_SMD:R_0603_1608Metric_Pad0.98x0.95mm_HandSolder"
 			(at 53.34 57.785 0)
 			(hide yes)
@@
 		(instances
 			(project "PS-BPSLeader"
-				(path "/d4a4ed4f-0983-4aef-b212-0e3284ab3963/69244dac-f10b-499c-a2b2-3cdf1370aa1f/1a445fba-997a-4276-b1d7-6bccd354442b"
-					(reference "R?")
+				(path "/d4a4ed4f-0983-4aef-b212-0e3284ab3963/69244dac-f10b-499c-a2b2-3cdf1370aa1f/0f3e3992-4755-4e76-a363-7a4e463e2a3d"
+					(reference "R127")
 					(unit 1)
 				)
@@
 		(dnp no)
 		(fields_autoplaced yes)
-		(property "Reference" "R?"
+		(property "Reference" "R129"
 			(at 69.215 56.5149 0)
 			(show_name no)
@@
 			)
 		)
-		(property "Footprint" ""
+		(property "Footprint" "Resistor_SMD:R_0603_1608Metric_Pad0.98x0.95mm_HandSolder"
 			(at 66.675 57.785 0)
 			(hide yes)
@@
 		(instances
 			(project "PS-BPSLeader"
-				(path "/d4a4ed4f-0983-4aef-b212-0e3284ab3963/69244dac-f10b-499c-a2b2-3cdf1370aa1f/1a445fba-997a-4276-b1d7-6bccd354442b"
-					(reference "R?")
+				(path "/d4a4ed4f-0983-4aef-b212-0e3284ab3963/69244dac-f10b-499c-a2b2-3cdf1370aa1f/0f3e3992-4755-4e76-a363-7a4e463e2a3d"
+					(reference "R129")
 					(unit 1)
 				)

Commit message: Fixed 12V Buck Boost Capacitors having the wrong P/N and footprint. Found P/N and LCSC P/N for 12V Power Mux. 5k resistors have been changed to 5.1k to use the standard parts list.
Parts:
- C90: LCSC P/N (none) -> C15849; P/N (none) -> CC0603KRX7R9BB105
- R122, R124, R128: LCSC P/N (none) -> C20015033; P/N (none) -> ERA-3AED5762V
- R123, R125, R127, R129: value 5k -> 5.1k; LCSC P/N (none) -> C23186; P/N (none) -> CRCW06035K10FKEC
- R126: LCSC P/N (none) -> C4018536; P/N (none) -> RQ73C1J26K1BTD
- R130: LCSC P/N (none) -> C203418; P/N (none) -> CR0603-FX-2212ELF
- U17: Availability In Stock -> (none); Check_prices https://www.snapeda.com/parts/TPS2121RUXR/Texas+Instruments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 -> (none); MANUFACTURER TEXAS INSTRUMENTS -> (none); MF Texas Instruments -> (none); MP TPS2121RUXR -> (none); Package VQFN-HR-12 Texas Instruments -> (none); Price None -> (none); Purchase-URL https://www.snapeda.com/api/url_track_click_mouser/?unipart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 -> (none); STANDARD Manufacturer Recommendations -> (none); SnapEDA_Link https://www.snapeda.com/parts/TPS2121RUXR/Texas+Instruments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 -> (none)
