File: LHRS_Design_Blocks.kicad_blocks/Contactor.kicad_block/Contactor.kicad_sch (KiCad schematic)
At the start: 15 parts

Commit message: Contactor economizer (#75)
All design blocks should be good. P/N, symbols, datasheets, etc. should be good.

* fixed merge conflicts from local files not updating for some reason

* gitignore stuff

* fixed merge conflicts and added 12V power mux

* added power mux design block

* added bq chip symbol

* fixed merge of lhrs_power symbols

* added footprints for economizer, mux, and bms transceiver

* fixed some erc issues

* First draft of 12V Buck-boost design block has been created

* 12vbuck

* adress reviews

* new passives

* updated footprints, p/n, and checked for stocks for every passive

* removed temp folder

* added transformer footprint

* added 3d model for transformer, changed silkscreen for SOT23_NXP

* Removed KiCad project files

* Embedded contactor economizer datasheet and fixed symbols for LM74502DDFR and LM7450HDDFR

* added datasheet to drv110

* Embedded data sheets in symbol, fixed 12V Buck Design Block schematic issues caused by merge, made edits to 12V Buck Boost Design Block

* Fixed 12V Buck Boost Capacitors having the wrong P/N and footprint. Found P/N and LCSC P/N for 12V Power Mux. 5k resistors have been changed to 5.1k to use the standard parts list.

---------

Co-authored-by: Gavin Wang <gavinwang07@gmail.com>
Co-authored-by: Abby Parsons <abigailparsons@utexas,edu>
Co-authored-by: Shuopu Wang <shuopuwang027@gmail.com>
Parts:
- removed C?: 1u, Capacitor_SMD:C_0603_1608Metric_Pad1.08x0.95mm_HandSolder, symbol Device:C
- removed C?: 0.1u, Capacitor_SMD:C_0603_1608Metric_Pad1.08x0.95mm_HandSolder, symbol Device:C
- removed D?: Contact, LED_SMD:LED_0603_1608Metric, symbol Device:LED
- removed D?: VSSAF522-M3/H, LHRS_Passives:SODFL5226X100N, symbol Diode:C3D25170H
- removed J?: ContactorConnector, LHRS_Connectors:Molex_Nano-Fit_105309-xx04_1x04_P2.50mm_Vertical, symbol LHRS_Connectors:ContactorConnector
- removed Q? (x2): IRLML0030, Package_TO_SOT_SMD:SOT-23, symbol Transistor_FET:IRLML0030
- removed R? (x4): 10k, Resistor_SMD:R_0603_1608Metric_Pad0.98x0.95mm_HandSolder, symbol Device:R
- removed R?: 1k, Resistor_SMD:R_0603_1608Metric_Pad0.98x0.95mm_HandSolder, symbol Device:R
- removed R?: 4.3k, Resistor_SMD:R_0603_1608Metric_Pad0.98x0.95mm_HandSolder, symbol Device:R
- removed TP?: ctrl, TestPoint:TestPoint_THTPad_D3.0mm_Drill1.5mm, symbol Connector:TestPoint
- removed TP?: Sense, TestPoint:TestPoint_THTPad_D3.0mm_Drill1.5mm, symbol Connector:TestPoint
- added C1: 0.1n, Capacitor_SMD:C_0603_1608Metric_Pad1.08x0.95mm_HandSolder, symbol Device:C_Small
- added C?: 0.1u, Capacitor_SMD:C_0603_1608Metric_Pad1.08x0.95mm_HandSolder, symbol Device:C
- added C? (x2): 4.7u, Capacitor_SMD:C_0805_2012Metric_Pad1.18x1.45mm_HandSolder, symbol Device:C
- added C?: 1u, Capacitor_SMD:C_0603_1608Metric_Pad1.08x0.95mm_HandSolder, symbol Device:C_Small
- added C?: 1u, Capacitor_SMD:C_0603_1608Metric_Pad1.08x0.95mm_HandSolder, symbol Device:C
- added D1, D?: VSSAF522-M3/H, LHRS_Passives:SODFL5226X100N, symbol Diode:C3D25170H
- added D?: Contact, LED_SMD:LED_0603_1608Metric_Pad1.05x0.95mm_HandSolder, symbol Device:LED
- added J?: Contactor Connector, LHRS_Connectors:Molex_Nano-Fit_105309-xx04_1x04_P2.50mm_Vertical, symbol lhrs_connectors:ContactorConnector
- added Q? (x2): IRLML0030, Package_TO_SOT_SMD:SOT-23, symbol Transistor_FET:IRLML0030
- added R1, R?: 1k, Resistor_SMD:R_0603_1608Metric_Pad0.98x0.95mm_HandSolder, symbol Device:R
- added R62, R? (x2): 10k, Resistor_SMD:R_0603_1608Metric_Pad0.98x0.95mm_HandSolder, symbol Device:R
- added R?: 4.3k, Resistor_SMD:R_0603_1608Metric_Pad0.98x0.95mm_HandSolder, symbol Device:R
- added R?: 66.67k, Resistor_SMD:R_0603_1608Metric_Pad0.98x0.95mm_HandSolder, symbol Device:R
- added R?: 120k, Resistor_SMD:R_0603_1608Metric_Pad0.98x0.95mm_HandSolder, symbol Device:R
- added R?: 1, Resistor_SMD:R_0603_1608Metric_Pad0.98x0.95mm_HandSolder, symbol Device:R
- added R?: 0, Resistor_SMD:R_0603_1608Metric_Pad0.98x0.95mm_HandSolder, symbol Device:R
- added TP?: ctrl, TestPoint:TestPoint_THTPad_D3.0mm_Drill1.5mm, symbol Connector:TestPoint
- added TP?: Sense, TestPoint:TestPoint_THTPad_D3.0mm_Drill1.5mm, symbol Connector:TestPoint
- added U?: DRV110APWR, LHRS_ICs:PW14_TEX, symbol lhrs_ics:DRV110APWR
Connections:
- net CONTACTOR+: now also C?.1, D?.1 (K), J?.1 (Con+(12V)), J?.4 (Sense+(12V)), R?.2, R?.2
- net CONTROL: now also U?.13 (EN)
- net GND: now also C1.2, C?.1, C?.1, C?.2, C?.2, C?.2, D1.2 (A), R?.1, R?.1, R?.1, R?.1, R?.1, U?.8 (GND)
- net HV_CONTROL: now also D?.1 (K), D?.2 (A), J?.2 (Con-), Q?.3 (D)
- net SENSE: now also C?.2, Q?.2 (S), R?.2, TP?.1
- new net: J?.3 (Sense-), R?.1
- new net: Q?.1 (G), TP?.1, U?.11 (OUT)
- new net: D?.2 (A), R?.1
- new net: C?.2, Q?.1 (G), R?.2
- new net: C?.1, U?.2 (KEEP)
- new net: R?.2, U?.3 (PEAK)
- new net: R?.2, U?.4 (HOLD)
- new net: R?.2, U?.5 (OSC)
- new net: C?.1, D1.1 (K), R?.1, U?.7 (VIN)
- new net: Q?.2 (S), R1.2, R?.2
- new net 3V3: Q?.3 (D), R62.2
- new net Econ_Sense: C1.1, R1.1, U?.9 (SENSE)
- new net Status: R62.1, U?.12 (STATUS)
Other:
- note added: "Ckeep=1u -> Tkeep=100ms"
- note added: "Currently just datasheet typical application values. Need to calculate values based on peak and hold current for contactor."
- note added: "R_hold = 66.67k"
- note added: "Vgs = 12V"
- note removed: "Vgs ~= 1/2*Vin = 12V"
