File: LHRS_Design_Blocks.kicad_blocks/Contactor.kicad_block/Contactor.kicad_sch (KiCad schematic)
At the start: 15 parts

Commit message: fixed merge conflicts from local files not updating for some reason
Connections:
- net +24V: no longer J?.1 (Con+(24V))
- net CONTACTOR+: no longer D?.1 (K), R?.2
- net GND: no longer C?.1
- net HV_CONTROL: no longer J?.2 (Con-)
- net CONTROL: no longer names the net of Q?.1 (G), R?.2, TP?.1
- new net: D?.1 (K), R?.2
Changed lines of the file:
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@@
 	(wire
 		(pts
-			(xy 226.06 87.63) (xy 241.3 87.63)
+			(xy 230.505 52.07) (xy 248.285 52.07)
 		)
 		(stroke
@@
 		(pts
 			(xy 227.33 93.98) (xy 227.33 91.44)
-		)
-		(stroke
-			(width 0)
-			(type default)
-		)
-	)
-	(wire
-		(pts
-			(xy 237.49 78.74) (xy 237.49 83.82)
 		)
 		(stroke
@@
 	)
 	(label "HV_CONTROL"
-		(at 226.06 87.63 0)
+		(at 230.505 52.07 0)
 		(effects
 			(font
@@
 		)
 	)
-	(hierarchical_label "GND"
-		(shape bidirectional)
-		(at 184.15 109.22 270)
-		(effects
-			(font
-				(size 1.27 1.27)
-			)
-			(justify right)
-		)
-	)
-	(hierarchical_label "CONTROL"
-		(shape input)
-		(at 68.58 101.6 180)
-		(effects
-			(font
-				(size 1.27 1.27)
-			)
-			(justify right)
-		)
-	)
 	(hierarchical_label "CONTACTOR+"
 		(shape input)
-		(at 96.52 72.39 90)
-		(effects
-			(font
-				(size 1.27 1.27)
-			)
-			(justify left)
+		(at 245.11 59.69 180)
+		(effects
+			(font
+				(size 1.27 1.27)
+			)
+			(justify right)
+		)
+	)
+	(hierarchical_label "GND"
+		(shape input)
+		(at 45.085 73.025 270)
+		(effects
+			(font
+				(size 1.27 1.27)
+			)
+			(justify right)
+		)
+	)
+	(hierarchical_label "GND"
+		(shape input)
+		(at 114.935 118.11 270)
+		(effects
+			(font
+				(size 1.27 1.27)
+			)
+			(justify right)
+		)
+	)
+	(hierarchical_label "GND"
+		(shape input)
+		(at 65.405 118.057 270)
+		(effects
+			(font
+				(size 1.27 1.27)
+			)
+			(justify right)
+		)
+	)
+	(hierarchical_label "GND"
+		(shape input)
+		(at 200.025 73.66 270)
+		(effects
+			(font
+				(size 1.27 1.27)
+			)
+			(justify right)
+		)
+	)
+	(hierarchical_label "CONTACTOR+"
+		(shape input)
+		(at 244.475 48.26 180)
+		(effects
+			(font
+				(size 1.27 1.27)
+			)
+			(justify right)
 		)
 	)
@@
 		(effects
 			(font
+				(size 1.27 1.27)
+			)
+			(justify right)
+		)
+	)
+	(hierarchical_label "GND"
+		(shape input)
+		(at 142.24 114.935 270)
+		(effects
+			(font
+				(size 1.27 1.27)
+			)
+			(justify right)
+		)
+	)
+	(hierarchical_label "CONTACTOR+"
+		(shape input)
+		(at 39.37 54.61 180)
+		(effects
+			(font
+				(size 1.27 1.27)
+			)
+			(justify right)
+		)
+	)
+	(hierarchical_label "GND"
+		(shape input)
+		(at 88.9 74.93 270)
+		(effects
+			(font
+				(size 1.27 1.27)
+			)
+			(justify right)
+		)
+	)
+	(hierarchical_label "GND"
+		(shape input)
+		(at 49.53 112.395 270)
+		(effects
+			(font

Commit message: fixed merge conflicts and added 12V power mux
Parts:
- removed J?: ContactorConnector, LHRS_Connectors:Molex_Nano-Fit_105309-xx04_1x04_P2.50mm_Vertical, symbol LHRS_Connectors:ContactorConnector
- removed Q?: IRLML0030, Package_TO_SOT_SMD:SOT-23, symbol Transistor_FET:IRLML0030
- removed R? (x3): 10k, Resistor_SMD:R_0603_1608Metric_Pad0.98x0.95mm_HandSolder, symbol Device:R
- removed TP?: ctrl, TestPoint:TestPoint_THTPad_D3.0mm_Drill1.5mm, symbol Connector:TestPoint
- added C1: 0.1n, symbol Device:C_Small
- added C? (x2): 4.7u, symbol Device:C
- added C?: 1u, symbol Device:C_Small
- added D1: VSSAF522-M3/H, LHRS_Passives:SODFL5226X100N, symbol Diode:C3D25170H
- added J?: Contactor Connector, LHRS_Connectors:Molex_Nano-Fit_105309-xx04_1x04_P2.50mm_Vertical, symbol lhrs_connectors:ContactorConnector
- added Q?: IRLML0030, Package_TO_SOT_SMD:SOT-23, symbol Transistor_FET:IRLML0030
- added R1, R?: 1k, Resistor_SMD:R_0603_1608Metric_Pad0.98x0.95mm_HandSolder, symbol Device:R
- added R?: 120k, Resistor_SMD:R_0603_1608Metric_Pad0.98x0.95mm_HandSolder, symbol Device:R
- added R?: 0, Resistor_SMD:R_0603_1608Metric_Pad0.98x0.95mm_HandSolder, symbol Device:R
- added R?: 66.67k, Resistor_SMD:R_0603_1608Metric_Pad0.98x0.95mm_HandSolder, symbol Device:R
- added R?: 1, Resistor_SMD:R_0603_1608Metric_Pad0.98x0.95mm_HandSolder, symbol Device:R
- added TP?: ctrl, TestPoint:TestPoint_THTPad_D3.0mm_Drill1.5mm, symbol Connector:TestPoint
- added U?: DRV110APWR, PW14_TEX, symbol lhrs_ics:DRV110APWR
- R?: value 1k -> 10k
Connections:
- net CONTACTOR+: now also D?.1 (K), R?.2, C?.1, J?.1 (Con+(12V)), J?.4 (Sense+(12V)), R?.2
- net GND: now also C?.1, C1.2, C?.2, C?.2, C?.2, D1.2 (A), R?.1, R?.1, R?.1, R?.1, U?.8 (GND)
- net HV_CONTROL: now also J?.2 (Con-), Q?.3 (D)
- net at R?.1: now also J?.3 (Sense-)
- net 3.3V renamed 3V3
- new net: R?.2, U?.3 (PEAK)
- new net: R?.2, U?.5 (OSC)
- new net: C?.1, D1.1 (K), R?.1, U?.7 (VIN)
- new net: Q?.1 (G), TP?.1, U?.11 (OUT)
- new net: C?.1, U?.2 (KEEP)
- new net: R?.2, U?.4 (HOLD)
- new net: Q?.2 (S), R1.2, R?.2
- new net CONTROL: U?.13 (EN)
- new net Sense: C1.1, R1.1, U?.9 (SENSE)
- new net Status: U?.12 (STATUS)
Other:
- note added: "Ckeep=1u -> Tkeep=100ms"
- note added: "Currently just datasheet typical application values. Need to calculate values based on peak and hold current for contactor."
- note added: "R_hold = 66.67k"
- note added: "Vgs = 12V"
- note removed: "Vgs ~= 1/2*Vin = 12V"
- moved on the sheet: C?, D?, Q?, R?, TP?

Commit message: added footprints for economizer, mux, and bms transceiver
Parts:
- removed C?: 4.7u, symbol Device:C
- removed D?: VSSAF522-M3/H, LHRS_Passives:SODFL5226X100N, symbol Diode:C3D25170H
- removed Q?: IRLML0030, Package_TO_SOT_SMD:SOT-23, symbol Transistor_FET:IRLML0030
- removed R?: 120k, Resistor_SMD:R_0603_1608Metric_Pad0.98x0.95mm_HandSolder, symbol Device:R
- removed R?: 10k, Resistor_SMD:R_0603_1608Metric_Pad0.98x0.95mm_HandSolder, symbol Device:R
- removed R?: 4.3k, Resistor_SMD:R_0603_1608Metric_Pad0.98x0.95mm_HandSolder, symbol Device:R
- removed TP?: ctrl, TestPoint:TestPoint_THTPad_D3.0mm_Drill1.5mm, symbol Connector:TestPoint
- added C?: 4.7u, symbol Device:C
- added D?: VSSAF522-M3/H, LHRS_Passives:SODFL5226X100N, symbol Diode:C3D25170H
- added Q?: IRLML0030, Package_TO_SOT_SMD:SOT-23, symbol Transistor_FET:IRLML0030
- added R? (x2): 10k, Resistor_SMD:R_0603_1608Metric_Pad0.98x0.95mm_HandSolder, symbol Device:R
- added R?: 120k, Resistor_SMD:R_0603_1608Metric_Pad0.98x0.95mm_HandSolder, symbol Device:R
- added R?: 4.3k, Resistor_SMD:R_0603_1608Metric_Pad0.98x0.95mm_HandSolder, symbol Device:R
- added TP?: ctrl, TestPoint:TestPoint_THTPad_D3.0mm_Drill1.5mm, symbol Connector:TestPoint
Connections:
- net 3V3: now also R?.2
- net CONTACTOR+: now also D?.1 (K), R?.2
- net GND: now also C?.2, R?.1, R?.1
- net HV_CONTROL: now also D?.2 (A), Q?.3 (D)
- net SENSE: now also R?.2
- net Status: now also R?.1
- net at D?.2 (A): now also R?.1
- net at U?.3 (PEAK): now also R?.2
- net at D1.1 (K), R?.1, U?.7 (VIN): now also C?.1
- net at U?.11 (OUT): now also Q?.1 (G), TP?.1
- net at R1.2, R?.2: now also Q?.2 (S)
Other:
- moved on the sheet: C1, C?, D1, D?, J?, Q?, R1, R?, TP?, U?

Commit message: fixed some erc issues
Parts:
- removed C1: 0.1n, symbol Device:C_Small
- removed C? (x2): 4.7u, symbol Device:C
- removed C?: 1u, Capacitor_SMD:C_0603_1608Metric_Pad1.08x0.95mm_HandSolder, symbol Device:C
- removed C?: 0.1u, Capacitor_SMD:C_0603_1608Metric_Pad1.08x0.95mm_HandSolder, symbol Device:C
- removed C?: 1u, symbol Device:C_Small
- removed D1, D?: VSSAF522-M3/H, LHRS_Passives:SODFL5226X100N, symbol Diode:C3D25170H
- removed D?: Contact, LED_SMD:LED_0603_1608Metric, symbol Device:LED
- removed J?: Contactor Connector, LHRS_Connectors:Molex_Nano-Fit_105309-xx04_1x04_P2.50mm_Vertical, symbol lhrs_connectors:ContactorConnector
- removed Q? (x2): IRLML0030, Package_TO_SOT_SMD:SOT-23, symbol Transistor_FET:IRLML0030
- removed R1, R?: 1k, Resistor_SMD:R_0603_1608Metric_Pad0.98x0.95mm_HandSolder, symbol Device:R
- removed R? (x3): 10k, Resistor_SMD:R_0603_1608Metric_Pad0.98x0.95mm_HandSolder, symbol Device:R
- removed R?: 0, Resistor_SMD:R_0603_1608Metric_Pad0.98x0.95mm_HandSolder, symbol Device:R
- removed R?: 120k, Resistor_SMD:R_0603_1608Metric_Pad0.98x0.95mm_HandSolder, symbol Device:R
- removed R?: 66.67k, Resistor_SMD:R_0603_1608Metric_Pad0.98x0.95mm_HandSolder, symbol Device:R
- removed R?: 4.3k, Resistor_SMD:R_0603_1608Metric_Pad0.98x0.95mm_HandSolder, symbol Device:R
- removed R?: 1, Resistor_SMD:R_0603_1608Metric_Pad0.98x0.95mm_HandSolder, symbol Device:R
- removed TP?: ctrl, TestPoint:TestPoint_THTPad_D3.0mm_Drill1.5mm, symbol Connector:TestPoint
- removed TP?: Sense, TestPoint:TestPoint_THTPad_D3.0mm_Drill1.5mm, symbol Connector:TestPoint
- removed U?: DRV110APWR, PW14_TEX, symbol lhrs_ics:DRV110APWR
- added C34, C36: 4.7u, Capacitor_SMD:C_0805_2012Metric_Pad1.18x1.45mm_HandSolder, symbol Device:C
- added C35: 1u, Capacitor_SMD:C_0603_1608Metric_Pad1.08x0.95mm_HandSolder, symbol Device:C_Small
- added C37: 0.1n, Capacitor_SMD:C_0603_1608Metric_Pad1.08x0.95mm_HandSolder, symbol Device:C_Small
- added C38: 1u, Capacitor_SMD:C_0603_1608Metric_Pad1.08x0.95mm_HandSolder, symbol Device:C
- added C39: 0.1u, Capacitor_SMD:C_0603_1608Metric_Pad1.08x0.95mm_HandSolder, symbol Device:C
- added D13, D15: VSSAF522-M3/H, LHRS_Passives:SODFL5226X100N, symbol Diode:C3D25170H
- added D14: Contact, LED_SMD:LED_0603_1608Metric_Pad1.05x0.95mm_HandSolder, symbol Device:LED
- added J16: Contactor Connector, LHRS_Connectors:Molex_Nano-Fit_105309-xx04_1x04_P2.50mm_Vertical, symbol lhrs_connectors:ContactorConnector
- added Q6, Q7: IRLML0030, Package_TO_SOT_SMD:SOT-23, symbol Transistor_FET:IRLML0030
- added R58: 66.67k, Resistor_SMD:R_0603_1608Metric_Pad0.98x0.95mm_HandSolder, symbol Device:R
- added R59: 0, Resistor_SMD:R_0603_1608Metric_Pad0.98x0.95mm_HandSolder, symbol Device:R
- added R60, R65: 1k, Resistor_SMD:R_0603_1608Metric_Pad0.98x0.95mm_HandSolder, symbol Device:R
- added R61: 120k, Resistor_SMD:R_0603_1608Metric_Pad0.98x0.95mm_HandSolder, symbol Device:R
- added R62, R66, R67: 10k, Resistor_SMD:R_0603_1608Metric_Pad0.98x0.95mm_HandSolder, symbol Device:R
- added R63: 4.3k, Resistor_SMD:R_0603_1608Metric_Pad0.98x0.95mm_HandSolder, symbol Device:R
- added R64: 1, Resistor_SMD:R_0603_1608Metric_Pad0.98x0.95mm_HandSolder, symbol Device:R
- added TP7: ctrl, TestPoint:TestPoint_THTPad_D3.0mm_Drill1.5mm, symbol Connector:TestPoint
- added TP8: Sense, TestPoint:TestPoint_THTPad_D3.0mm_Drill1.5mm, symbol Connector:TestPoint
- added U7: DRV110APWR, LHRS_ICs:PW14_TEX, symbol lhrs_ics:DRV110APWR
Connections:
- net 3V3: now also Q7.3 (D), R62.2
- net CONTACTOR+: now also C34.1, D15.1 (K), J16.1 (Con+(12V)), J16.4 (Sense+(12V)), R60.2, R63.2
- net CONTROL: now also U7.13 (EN)
- net GND: now also C34.2, C35.2, C36.2, C37.2, C38.1, C39.1, D13.2 (A), R58.1, R59.1, R61.1, R64.1, R66.1, U7.8 (GND)
- net HV_CONTROL: now also D14.1 (K), D15.2 (A), J16.2 (Con-), Q6.3 (D)
- net SENSE: now also C38.2, Q7.2 (S), R66.2, TP8.1
- net Status: now also R62.1, U7.12 (STATUS)
- new net: J16.3 (Sense-), R67.1
- new net: Q6.1 (G), TP7.1, U7.11 (OUT)
- new net: D14.2 (A), R63.1
- new net: C39.2, Q7.1 (G), R67.2
- new net: C35.1, U7.2 (KEEP)
- new net: R61.2, U7.3 (PEAK)
- new net: R58.2, U7.4 (HOLD)
- new net: R59.2, U7.5 (OSC)
- new net: C36.1, D13.1 (K), R60.1, U7.7 (VIN)
- new net: Q6.2 (S), R64.2, R65.2
- new net Econ_Sense: C37.1, R65.1, U7.9 (SENSE)

Commit message: Embedded contactor economizer datasheet and fixed symbols for LM74502DDFR and LM7450HDDFR
Parts:
- renumbered C37 to C1, C39 to C?, C36 to C?, C34 to C?, C35 to C?, C38 to C?, D13 to D1, D14 to D?, D15 to D?, J16 to J?, Q7 to Q?, Q6 to Q?, R65 to R1, R63 to R?, R66 to R?, R58 to R?, R60 to R?, R61 to R?, R64 to R?, R59 to R?, R67 to R?, TP7 to TP?, TP8 to TP?, U7 to U?

Commit message: Rev a fixes (#84)
* updated buck block

* tp symbol + usb fixes

* fixes

* updated .gitignore

* updated conns
Parts:
- removed TP?: ctrl, TestPoint:TestPoint_THTPad_D3.0mm_Drill1.5mm, symbol Connector:TestPoint
- removed TP?: Sense, TestPoint:TestPoint_THTPad_D3.0mm_Drill1.5mm, symbol Connector:TestPoint
- C?: LCSC P/N (none) -> C14663; Mouser Part Number 963-HMK107B7104KA-T -> (none)
- C?: Mouser Part Number 963-UMK107BJ105KA-T -> (none)
- D1, D?: LCSC P/N (none) -> C6326606; Manufactuerer Vishay General Semiconductor -> (none)
- D?: LCSC P/N (none) -> C84263; Manufactuerer NATIONSTAR -> (none)
- Q? (x2): LCSC P/N (none) -> C67272
Other:
- moved on the sheet: C1, C?, D1, D?, J?, Q?, R1, R62, R?, U?
