File: LHRS_Design_Blocks.kicad_blocks/12VBuckBoost.kicad_block/12VBuckBoost.kicad_sch (KiCad schematic)
At the start: 18 parts, among them IC1 TPS552872RYQR

Commit message: Embedded data sheets in symbol, fixed 12V Buck Design Block schematic issues caused by merge, made edits to 12V Buck Boost Design Block
Parts:
- added C96, C97: 0.1u, Capacitor_SMD:C_1206_3216Metric, symbol Device:C
- added NT1: NetTie_2, symbol Device:NetTie_2
- C1, C2, C3, C4, C5: footprint (none) -> Capacitor_SMD:C_1206_3216Metric; LCSC P/N (none) -> C5448976; P/N (none) -> GGM31CD70J226KE02L
- C10: value C -> 45p; footprint (none) -> Capacitor_SMD:C_0603_1608Metric_Pad1.08x0.95mm_HandSolder; LCSC P/N (none) -> C105622; P/N (none) -> CL10C470JB8NNNC
- C6: footprint (none) -> Capacitor_SMD:C_0805_2012Metric_Pad1.18x1.45mm_HandSolder; LCSC P/N (none) -> C105911; P/N (none) -> -- mixed values --
- C7: footprint Package_SO:SOIC-8_3.9x4.9mm_P1.27mm -> Capacitor_SMD:C_1206_3216Metric; LCSC P/N (none) -> C14663; P/N (none) -> MLASH168SB7104KTNA01
- C8: footprint (none) -> Capacitor_SMD:C_1206_3216Metric; LCSC P/N (none) -> C14663; P/N (none) -> MLASH168SB7104KTNA01
- C9: footprint (none) -> Capacitor_SMD:C_0603_1608Metric_Pad1.08x0.95mm_HandSolder; LCSC P/N (none) -> C282075; P/N (none) -> 0603N910J500CT
- L1: footprint Package_SO:SOIC-20W_7.5x12.8mm_P1.27mm -> LHRS_Passives:74439369082; P/N (none) -> 74439369082
- R1: footprint (none) -> Resistor_SMD:R_0603_1608Metric_Pad0.98x0.95mm_HandSolder; LCSC P/N (none) -> C25803; P/N (none) -> CRCW0603100KFKEE
- R2: footprint (none) -> Resistor_SMD:R_0603_1608Metric_Pad0.98x0.95mm_HandSolder; LCSC P/N (none) -> C1854558; P/N (none) -> RNCF0603BTE11K1
- R3: footprint (none) -> Resistor_SMD:R_0603_1608Metric_Pad0.98x0.95mm_HandSolder; LCSC P/N (none) -> C22841; P/N (none) -> CR0603-FX-1431ELF
- R4: footprint (none) -> Resistor_SMD:R_1210_3225Metric; LCSC P/N (none) -> C7467372; P/N (none) -> ERJ-8CWJR013V
- R5: footprint (none) -> Resistor_SMD:R_0603_1608Metric_Pad0.98x0.95mm_HandSolder; LCSC P/N (none) -> C4117233; P/N (none) -> CR0603-FX-4992ELF
- R6: renamed from R4; footprint (none) -> Resistor_SMD:R_0603_1608Metric_Pad0.98x0.95mm_HandSolder; now not fitted
Connections:
- net AGND: now also NT1.2; no longer C1.2, C2.2, C3.2, C4.2, C5.2, IC1.9 (PGND_1)
- net VIN: now also C96.1
- net at IC1.8 (SW1), L1.1: now also C7.1; no longer C7.2
- net at IC1.20 (BOOT1): now also C7.2; no longer C7.1
- net at C2.1, C3.1, C4.1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: now also C97.1
- net PGND: now reaches IC1.22 (PGND_2)
- net PGND: now also C1.2, C2.2, C3.2, C4.2, C5.2, IC1.23 (PGND_3), IC1.9 (PGND_1), C96.2, C97.2, NT1.1
Other:
- note added: "C1"
- note added: "C2"
- note added: "C3"
- note added: "C4"
- note added: "C5"
- note added: "C6"
- note added: "C7"
- note added: "f_C is upper bounded by the lower of 1/10 f_SW and 1/5 f_RHPZ. R_COUT is the ESR of C2, C3, C4, C5, and C6. The datasheet states C7 can be left open if it's below 10 pF. If R_COUT is less than 0.165 mOhms, C7 can be left open. EN/UVLO: Programmable undervoltage lockout. Logic high enables (>1.15V) & logic low turns it into shutdown mode. Can be used for undervoltage lockout. PG: Power good. When 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"
- note removed: "f_C is upper bounded by the lower of 1/10 f_SW and 1/5 f_RHPZ. R_COUT is the ESR of C2, C3, C4, C5, and C6. The datasheet states C10 can be left open if it's below 10 pF. If R_COUT is less than 0.165 mOhms, C10 can be left open. EN/UVLO: Programmable undervoltage lockout. Logic high enables & logic low turns it into shutdown mode. PG: Power good. When VOUT > 95% of the setting output voltage, hig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"

Commit message: Fixed 12V Buck Boost Capacitors having the wrong P/N and footprint. Found P/N and LCSC P/N for 12V Power Mux. 5k resistors have been changed to 5.1k to use the standard parts list.
Parts:
- C1, C2, C3, C4, C5: footprint Capacitor_SMD:C_1206_3216Metric -> Capacitor_SMD:C_1210_3225Metric_Pad1.33x2.70mm_HandSolder; LCSC P/N C5448976 -> C778721; P/N GGM31CD70J226KE02L -> GMK325BJ226MM-P
- C6: P/N -- mixed values -- -> C0805B475K050T
- R1, R2, R3, R4, R5, R6: symbol Device:R_US -> Device:R
Changed lines of the file:
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@@
 			)
 		)
-		(property "P/N" "-- mixed values --"
+		(property "P/N" "C0805B475K050T"
 			(at 120.65 41.91 0)
 			(hide yes)
@@
 			)
 		)
-		(property "Footprint" "Capacitor_SMD:C_1206_3216Metric"
+		(property "Footprint" "Capacitor_SMD:C_1210_3225Metric_Pad1.33x2.70mm_HandSolder"
 			(at 209.2452 43.18 0)
 			(hide yes)
@@
 			)
 		)
-		(property "LCSC P/N" "C5448976 "
+		(property "LCSC P/N" "C778721"
 			(at 208.28 39.37 0)
 			(hide yes)
@@
 			)
 		)
-		(property "P/N" "GGM31CD70J226KE02L "
+		(property "P/N" "GMK325BJ226MM-P"
 			(at 208.28 39.37 0)
 			(hide yes)
@@
 	)
 	(symbol
-		(lib_id "Device:R_US")
+		(lib_id "Device:R")
 		(at 241.3 59.69 0)
 		(unit 1)
@@
 		)
 		(property "Footprint" "Resistor_SMD:R_0603_1608Metric_Pad0.98x0.95mm_HandSolder"
-			(at 242.316 59.944 90)
+			(at 239.522 59.69 90)
 			(hide yes)
 			(show_name no)
@@
 			)
 		)
-		(property "Description" "Resistor, US symbol"
+		(property "Description" "Resistor"
 			(at 241.3 59.69 0)
 			(hide yes)
@@
 	)
 	(symbol
-		(lib_id "Device:R_US")
+		(lib_id "Device:R")
 		(at 208.28 62.23 0)
 		(unit 1)
@@
 		)
 		(property "Footprint" "Resistor_SMD:R_0603_1608Metric_Pad0.98x0.95mm_HandSolder"
-			(at 209.296 62.484 90)
+			(at 206.502 62.23 90)
 			(hide yes)
 			(show_name no)
@@
 			)
 		)
-		(property "Description" "Resistor, US symbol"
+		(property "Description" "Resistor"
 			(at 208.28 62.23 0)
 			(hide yes)
@@
 	)
 	(symbol
-		(lib_id "Device:R_US")
+		(lib_id "Device:R")
 		(at 173.99 67.31 180)
 		(unit 1)
@@
 		)
 		(property "Footprint" "Resistor_SMD:R_0603_1608Metric_Pad0.98x0.95mm_HandSolder"
-			(at 172.974 67.056 90)
+			(at 175.768 67.31 90)
 			(hide yes)
 			(show_name no)
@@
 			)
 		)
-		(property "Description" "Resistor, US symbol"
+		(property "Description" "Resistor"
 			(at 173.99 67.31 0)
 			(hide yes)
@@
 			)
 		)
-		(property "Footprint" "Capacitor_SMD:C_1206_3216Metric"
+		(property "Footprint" "Capacitor_SMD:C_1210_3225Metric_Pad1.33x2.70mm_HandSolder"
 			(at 197.8152 43.18 0)
 			(hide yes)
@@
 			)
 		)
-		(property "LCSC P/N" "C5448976 "
+		(property "LCSC P/N" "C778721"
 			(at 196.85 39.37 0)
 			(hide yes)
@@
 			)
 		)
-		(property "P/N" "GGM31CD70J226KE02L "
+		(property "P/N" "GMK325BJ226MM-P"
 			(at 196.85 39.37 0)
 			(hide yes)
@@
 	)
 	(symbol
-		(lib_id "Device:R_US")
+		(lib_id "Device:R")
 		(at 241.3 46.99 180)
 		(unit 1)
@@
 		)
 		(property "Footprint" "Resistor_SMD:R_0603_1608Metric_Pad0.98x0.95mm_HandSolder"
-			(at 240.284 46.736 90)
+			(at 243.078 46.99 90)
 			(hide yes)
 			(show_name no)
@@
 			)
 		)
-		(property "Description" "-- mixed values --"
+		(property "Description" "Resistor"
 			(at 241.3 46.99 0)
 			(hide yes)
@@
 			)
 		)
-		(property "Footprint" "Capacitor_SMD:C_1206_3216Metric"
+		(property "Footprint" "Capacitor_SMD:C_1210_3225Metric_Pad1.33x2.70mm_HandSolder"
 			(at 174.9552 43.18 0)
 			(hide yes)
@@
 			)
 		)
-		(property "LCSC P/N" "C5448976 "
+		(property "LCSC P/N" "C778721"
 			(at 173.99 39.37 0)
 			(hide yes)
@@
 			)
 		)
-		(property "P/N" "GGM31CD70J226KE02L "
+		(property "P/N" "GMK325BJ226MM-P"
 			(at 173.99 39.37 0)
 			(hide yes)
@@
 			)
 		)
-		(property "Footprint" "Capacitor_SMD:C_1206_3216Metric"
+		(property "Footprint" "Capacitor_SMD:C_1210_3225Metric_Pad1.33x2.70mm_HandSolder"
 			(at 96.2152 43.18 0)
 			(hide yes)
@@
 			)
 		)
-		(property "LCSC P/N" "C5448976 "
+		(property "LCSC P/N" "C778721"
 			(at 95.25 39.37 0)
 			(hide yes)
@@
 			)
 		)
-		(property "P/N" "GGM31CD70J226KE02L "
+		(property "P/N" "GMK325BJ226MM-P"
 			(at 95.25 39.37 0)
 			(hide yes)
@@
 			)
 		)
-		(property "Footprint" "Capacitor_SMD:C_1206_3216Metric"
+		(property "Footprint" "Capacitor_SMD:C_1210_3225Metric_Pad1.33x2.70mm_HandSolder"
 			(at 186.3852 43.18 0)
 			(hide yes)
@@
 			)
 		)
-		(property "LCSC P/N" "C5448976 "
+		(property "LCSC P/N" "C778721"
 			(at 185.42 39.37 0)
 			(hide yes)
@@
 			)
 		)
-		(property "P/N" "GGM31CD70J226KE02L "
+		(property "P/N" "GMK325BJ226MM-P"
 			(at 185.42 39.37 0)
 			(hide yes)
@@
 	)
 	(symbol
-		(lib_id "Device:R_US")
+		(lib_id "Device:R")
 		(at 229.87 35.56 90)
 		(unit 1)
@@
 		)
 		(property "Footprint" "Resistor_SMD:R_1210_3225Metric"
-			(at 230.124 34.544 90)
+			(at 229.87 37.338 90)
 			(hide yes)
 			(show_name no)
@@
 			)
 		)
-		(property "Description" "Resistor, US symbol"
+		(property "Description" "Resistor"
 			(at 229.87 35.56 0)
 			(hide yes)
@@
 	)
 	(symbol
-		(lib_id "Device:R_US")
+		(lib_id "Device:R")
 		(at 120.65 69.85 0)
 		(mirror x)
@@
 		)
 		(property "Footprint" "Resistor_SMD:R_0603_1608Metric_Pad0.98x0.95mm_HandSolder"
-			(at 121.666 69.596 90)
+			(at 118.872 69.85 90)
 			(hide yes)
 			(show_name no)
@@
 			)
 		)
-		(property "Description" "Resistor, US symbol"
+		(property "Description" "Resistor"
 			(at 120.65 69.85 0)
 			(hide yes)

Commit message: fixes
Parts:
- IC1: Height 1 -> (none); Manufacturer_Name Texas Instruments -> (none); Manufacturer_Part_Number TPS552872RYQR -> (none); Mouser Part Number 595-TPS552872RYQR -> (none); Mouser Price/Stock https://www.mouser.co.uk/ProductDetail/Texas-Instruments/TP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 -> (none); P/N (none) -> TPS552872RYQR
Changed lines of the file:
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@@
 			)
 		)
-		(property "Height" "1"
-			(at 154.94 430.48 0)
+		(property "P/N" "TPS552872RYQR"
+			(at 120.65 35.56 0)
 			(hide yes)
 			(show_name no)
@@
 					(size 1.27 1.27)
 				)
-				(justify left top)
 			)
 		)
-		(property "Mouser Part Number" "595-TPS552872RYQR"
-			(at 154.94 530.48 0)
-			(hide yes)
-			(show_name no)
-			(do_not_autoplace no)
-			(effects
-				(font
-					(size 1.27 1.27)
-				)
-				(justify left top)
-			)
-		)
-		(property "Mouser Price/Stock" "https://www.mouser.co.uk/ProductDetail/Texas-Instruments/TPS552872RYQR?qs=HoCaDK9Nz5dA1e3xUGl6lQ%3D%3D"
-			(at 154.94 630.48 0)
-			(hide yes)
-			(show_name no)
-			(do_not_autoplace no)
-			(effects
-				(font
-					(size 1.27 1.27)
-				)
-				(justify left top)
-			)
-		)
-		(property "Manufacturer_Name" "Texas Instruments"
-			(at 154.94 730.48 0)
-			(hide yes)
-			(show_name no)
-			(do_not_autoplace no)
-			(effects
-				(font
-					(size 1.27 1.27)
-				)
-				(justify left top)
-			)
-		)
-		(property "Manufacturer_Part_Number" "TPS552872RYQR"
-			(at 154.94 830.48 0)
-			(hide yes)
-			(show_name no)
-			(do_not_autoplace no)
-			(effects
-				(font
-					(size 1.27 1.27)
-				)
-				(justify left top)
-			)
-		)
