File: LHRS_Design_Blocks.kicad_blocks/12VBuckBoost.kicad_block/12VBuckBoost.kicad_sch (KiCad schematic)
At the start: 21 parts, among them IC1 TPS552872RYQR

Commit message: Rev a fixes (#84)
* updated buck block

* tp symbol + usb fixes

* fixes

* updated .gitignore

* updated conns
Parts:
- IC1: Height 1 -> (none); Manufacturer_Name Texas Instruments -> (none); Manufacturer_Part_Number TPS552872RYQR -> (none); Mouser Part Number 595-TPS552872RYQR -> (none); Mouser Price/Stock https://www.mouser.co.uk/ProductDetail/Texas-Instruments/TP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 -> (none); P/N (none) -> TPS552872RYQR
