File: LHRS_Design_Blocks.kicad_blocks/CAN_Transceiver.kicad_block/CAN_Transceiver.kicad_sch (KiCad schematic)
At the start: 9 parts, among them IC1 TCAN3413DR

Commit message: UTSVT to LHRS
Parts:
- D1: footprint UTSVT_Passives:CDSOT23-T24CAN -> LHRS_Passives:CDSOT23-T24CAN
- IC1: footprint UTSVT_Passives:TCAN3413DR -> LHRS_Passives:TCAN3413DR
Changed lines of the file:
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@@
 			)
 		)
-		(property "Footprint" "UTSVT_Passives:CDSOT23-T24CAN"
+		(property "Footprint" "LHRS_Passives:CDSOT23-T24CAN"
 			(at 204.47 149.53 0)
 			(effects
@@
 			)
 		)
-		(property "Footprint" "UTSVT_Passives:TCAN3413DR"
+		(property "Footprint" "LHRS_Passives:TCAN3413DR"
 			(at 140.97 166.04 0)
 			(effects

Commit message: Rev a fixes (#84)
* updated buck block

* tp symbol + usb fixes

* fixes

* updated .gitignore

* updated conns
Parts:
- D1: Height 1.17 -> (none); Manufacturer_Name Bourns -> (none); Mouser Part Number 652-CDSOT23-T24CAN -> (none); Mouser Price/Stock https://www.mouser.co.uk/ProductDetail/Bourns/CDSOT23-T24CA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 -> (none)
- IC1: Height 1.75 -> (none); Manufacturer_Name Texas Instruments -> (none); Mouser Part Number 595-TCAN3413DR -> (none); Mouser Price/Stock - -> (none)
Connections:
- net 3.3v renamed 3V3
