File: LHRS_Design_Blocks.kicad_blocks/USB_PD.kicad_block/USB_PD.kicad_sch (KiCad schematic)
At the start: 38 parts, among them IC1 CYPD3177-24LQXQ, Q1 SI7997DP-T1-GE3, Q2 SI7997DP-T1-GE3, Q3 IRLML0030

Commit message: UTSVT to LHRS
Parts:
- D4: symbol utsvt_power:SMBJ24A-E3_52 -> lhrs_power:SMBJ24A-E3_52
- D5, D6: symbol utsvt_power:SMBJ10A-E3_52 -> lhrs_power:SMBJ10A-E3_52
- IC1: footprint UTSVT_ICs:CYPD3177-24LQXQ -> LHRS_ICs:CYPD3177-24LQXQ; symbol utsvt_ics:CYPD3177-24LQXQ -> lhrs_ics:CYPD3177-24LQXQ
- Q1, Q2: footprint UTSVT_ICs:SI7997DP-T1-GE3 -> LHRS_ICs:SI7997DP-T1-GE3; symbol utsvt_ics:SI7997DP-T1-GE3 -> lhrs_ics:SI7997DP-T1-GE3
Changed lines of the file:
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@@
 	)
 	(symbol
-		(lib_id "utsvt_ics:SI7997DP-T1-GE3")
+		(lib_id "lhrs_ics:SI7997DP-T1-GE3")
 		(at 110.49 171.45 0)
 		(mirror y)
@@
 			)
 		)
-		(property "Footprint" "UTSVT_ICs:SI7997DP-T1-GE3"
+		(property "Footprint" "LHRS_ICs:SI7997DP-T1-GE3"
 			(at 86.36 266.37 0)
 			(effects
@@
 	)
 	(symbol
-		(lib_id "utsvt_power:SMBJ10A-E3_52")
+		(lib_id "lhrs_power:SMBJ10A-E3_52")
 		(at 95.25 139.7 270)
 		(unit 1)
@@
 	)
 	(symbol
-		(lib_id "utsvt_ics:SI7997DP-T1-GE3")
+		(lib_id "lhrs_ics:SI7997DP-T1-GE3")
 		(at 72.39 171.45 0)
 		(unit 1)
@@
 			)
 		)
-		(property "Footprint" "UTSVT_ICs:SI7997DP-T1-GE3"
+		(property "Footprint" "LHRS_ICs:SI7997DP-T1-GE3"
 			(at 96.52 266.37 0)
 			(effects
@@
 	)
 	(symbol
-		(lib_id "utsvt_power:SMBJ24A-E3_52")
+		(lib_id "lhrs_power:SMBJ24A-E3_52")
 		(at 35.56 48.26 90)
 		(mirror x)
@@
 	)
 	(symbol
-		(lib_id "utsvt_ics:SI7997DP-T1-GE3")
+		(lib_id "lhrs_ics:SI7997DP-T1-GE3")
 		(at 110.49 138.43 0)
 		(mirror y)
@@
 			)
 		)
-		(property "Footprint" "UTSVT_ICs:SI7997DP-T1-GE3"
+		(property "Footprint" "LHRS_ICs:SI7997DP-T1-GE3"
 			(at 86.36 233.35 0)
 			(effects
@@
 	)
 	(symbol
-		(lib_id "utsvt_ics:CYPD3177-24LQXQ")
+		(lib_id "lhrs_ics:CYPD3177-24LQXQ")
 		(at 137.16 67.31 0)
 		(unit 1)
@@
 			)
 		)
-		(property "Footprint" "UTSVT_ICs:CYPD3177-24LQXQ"
+		(property "Footprint" "LHRS_ICs:CYPD3177-24LQXQ"
 			(at 173.99 152.07 0)
 			(effects
@@
 	(symbol
 		(lib_name "SI7997DP-T1-GE3_1")
-		(lib_id "utsvt_ics:SI7997DP-T1-GE3")
+		(lib_id "lhrs_ics:SI7997DP-T1-GE3")
 		(at 72.39 138.43 0)
 		(unit 1)
@@
 			)
 		)
-		(property "Footprint" "UTSVT_ICs:SI7997DP-T1-GE3"
+		(property "Footprint" "LHRS_ICs:SI7997DP-T1-GE3"
 			(at 96.52 233.35 0)
 			(effects
@@
 	)
 	(symbol
-		(lib_id "utsvt_power:SMBJ10A-E3_52")
+		(lib_id "lhrs_power:SMBJ10A-E3_52")
 		(at 95.25 172.72 270)
 		(unit 1)

Commit message: Rev a fixes (#84)
* updated buck block

* tp symbol + usb fixes

* fixes

* updated .gitignore

* updated conns
Parts:
- C1: Mfg GRM21BR61H106KE43K -> (none)
- D2: renamed from D4; Height 2.44 -> (none); Manufacturer_Name Vishay -> (none); Mouser Part Number 625-SMBJ24A-E3 -> (none); Mouser Price/Stock https://www.mouser.co.uk/ProductDetail/Vishay-General-Semic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 -> (none)
- D3: renamed from D5; Height 2.44 -> (none); Manufacturer_Name Vishay -> (none); Mouser Part Number 625-SMBJ10A-E3 -> (none); Mouser Price/Stock https://www.mouser.co.uk/ProductDetail/Vishay-General-Semic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 -> (none)
- D4: renamed from D6; Height 2.44 -> (none); Manufacturer_Name Vishay -> (none); Mouser Part Number 625-SMBJ10A-E3 -> (none); Mouser Price/Stock https://www.mouser.co.uk/ProductDetail/Vishay-General-Semic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 -> (none)
- D5: renamed from D7; Color Red -> (none); Mfg NCD0603R1 -> (none)
- IC1: Height 0.6 -> (none); Manufacturer_Name Infineon -> (none); Mouser Part Number 727-CYPD3177-24LQXQ -> (none); Mouser Price/Stock https://www.mouser.co.uk/ProductDetail/Infineon-Technologie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 -> (none)
- Q1, Q2: Manufacturer_Name Vishay -> (none); Mouser Part Number 781-SI7997DP-T1-GE3 -> (none); Mouser Price/Stock https://www.mouser.co.uk/ProductDetail/Vishay-Semiconductor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 -> (none)
- R1: renamed from R7; Mfg CRCW06035K10FKEC -> (none)
- R2: renamed from R8; Mfg CRCW06035K10FKEC -> (none)
- renumbered R16 to R10, R17 to R11, R18 to R12, R19 to R13, R20 to R14, R9 to R3, R10 to R4, R11 to R5, R12 to R6, R13 to R7, R14 to R8, R15 to R9, TP19 to TP10, TP20 to TP11, TP15 to TP3, TP16 to TP8, TP17 to TP9
