File: LHRS_Design_Blocks.kicad_blocks/LDO.kicad_block/LDO.kicad_sch (KiCad schematic)
At the start: 5 parts, among them U1 MCP1826S

Commit message: Rev a fixes (#84)
* updated buck block

* tp symbol + usb fixes

* fixes

* updated .gitignore

* updated conns
Parts:
- removed TP_3.3V1: 3.3V, TestPoint:TestPoint_Loop_D1.80mm_Drill1.0mm_Beaded, symbol Connector:TestPoint
- U1: LCSC MFG P/N LM39100S-3.3 -> (none)

Commit message: replaced old diode with standardized part
Parts:
- D1: value SBA130CH-AU_R1_000A1 -> 1N5819HW-7-F; footprint Diode_SMD:D_SOD-323_HandSoldering -> Diode_SMD:D_SOD-123
Changed lines of the file:
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@@
 			)
 		)
-		(property "Value" "SBA130CH-AU_R1_000A1"
+		(property "Value" "1N5819HW-7-F"
 			(at 133.604 59.69 0)
 			(show_name no)
@@
 			)
 		)
-		(property "Footprint" "Diode_SMD:D_SOD-323_HandSoldering"
+		(property "Footprint" "Diode_SMD:D_SOD-123"
 			(at 133.35 63.5 90)
 			(hide yes)
@@
 			)
 		)
-		(property "Datasheet" "https://www.mouser.com/datasheet/3/3736/1/11145663EF9055F8C188C22CC003165FC5A818A8439A953D3A6E1D8FCBF51DA1.pdf"
+		(property "Datasheet" "https://www.diodes.com/assets/Datasheets/1N5819HW.pdf"
 			(at 133.35 63.5 90)
 			(hide yes)
