File: LHRS_Design_Blocks.kicad_blocks/IMUs.kicad_block/IMUs.kicad_sch (KiCad schematic)
At the start: 12 parts, among them IC3 MMC5983MA, U4 ASM330LHHX, U7 TPD4E05U06DQA, U8 TPD4E05U06DQA

Commit message: IMU Details
Parts:
- renumbered C25 to C42, C41 to C43, C26 to C44, C27 to C45, C40 to C48, C28 to C49, R25 to R35, U4 to U5, U7 to U6
Other:
- note added: "ESD Protection"
- note added: "MAG_DRDY is an interupt letting MCU know when a new reading is ready"
- note added: "Max Voltage: 3.6V Min Voltage: 1.71V Typ Current: 1.3mA Max Current: 1.6mA"
- note added: "Max Voltage: 3.6V Min Voltage: 2.8V Typ Current: 450uA Max Current: 450uA"
- note removed: "SPI Protection"
Changed lines of the file:
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@@
 		)
 	)
+	(text "Max Voltage: 3.6V\n\nMin Voltage: 1.71V\n\nTyp Current: 1.3mA\n\nMax Current: 1.6mA\n"
+		(exclude_from_sim no)
+		(at 61.214 146.304 0)
+		(effects
+			(font
+				(size 1.27 1.27)
+			)
+		)
+	)
+	(text "Max Voltage: 3.6V\n\nMin Voltage: 2.8V\n\nTyp Current: 450uA\n\nMax Current: 450uA\n"
+		(exclude_from_sim no)
+		(at 153.67 88.392 0)
+		(effects
+			(font
+				(size 1.27 1.27)
+			)
+		)
+	)
+	(text "MAG_DRDY is an interupt letting MCU know when a new reading is ready"
+		(exclude_from_sim no)
+		(at 60.96 136.906 0)
+		(effects
+			(font
+				(size 1.27 1.27)
+			)
+		)
+	)
 	(text "3-Axis Magnetometer"
 		(exclude_from_sim no)
@@
 		)
 	)
-	(text "SPI Protection"
+	(text "ESD Protection"
 		(exclude_from_sim no)
-		(at 181.61 110.49 0)
+		(at 181.864 110.49 0)
 		(effects
 			(font
@@
 	)
 	(image
-		(at 74.93 127)
-		(scale 0.384416)
+		(at 72.39 97.79)
+		(scale 0.280196)
 		(data "iVBORw0KGgoAAAANSUhEUgAABnIAAAT4CAYAAAAsDFyTAAAMUmlDQ1BJQ0MgUHJvZmlsZQAASImV"
 			"VwdYU8kWnlvSgNACCEgJvYkiUgJICT303kQlJAFCCTEhqIgNXVRwLahYsKKLIgpWmh0bKoti74sF"
@@
 				)
 			)
+			(project "SuspensionBoard"
+				(path "/f9dc491a-b8c6-4623-9728-13837ac4bba3/ab14ffa7-4ae1-4464-91d5-9b05f92e5082"
+					(reference "IC3")
+					(unit 1)
+				)
+			)
 		)
 	)
@@
 				)
 			)
+			(project "SuspensionBoard"
+				(path "/f9dc491a-b8c6-4623-9728-13837ac4bba3/ab14ffa7-4ae1-4464-91d5-9b05f92e5082"
+					(reference "U8")
+					(unit 1)
+				)
+			)
 		)
 	)
@@
 		(in_pos_files yes)
 		(dnp no)
-		(property "Reference" "C26"
+		(property "Reference" "C44"
 			(at 88.9 51.054 0)
 			(show_name no)
@@
 				)
 			)
+			(project "SuspensionBoard"
+				(path "/f9dc491a-b8c6-4623-9728-13837ac4bba3/ab14ffa7-4ae1-4464-91d5-9b05f92e5082"
+					(reference "C44")
+					(unit 1)
+				)
+			)
 		)
 	)
@@
 		(in_pos_files yes)
 		(dnp no)
-		(property "Reference" "C25"
+		(property "Reference" "C42"
 			(at 22.86 45.974 0)
 			(show_name no)
@@
 				)
 			)
+			(project "SuspensionBoard"
+				(path "/f9dc491a-b8c6-4623-9728-13837ac4bba3/ab14ffa7-4ae1-4464-91d5-9b05f92e5082"
+					(reference "C42")
+					(unit 1)
+				)
+			)
 		)
 	)
@@
 		(in_pos_files yes)
 		(dnp no)
-		(property "Reference" "C28"
+		(property "Reference" "C49"
 			(at 209.804 26.67 0)
 			(show_name no)
@@
 				)
 			)
+			(project "SuspensionBoard"
+				(path "/f9dc491a-b8c6-4623-9728-13837ac4bba3/ab14ffa7-4ae1-4464-91d5-9b05f92e5082"
+					(reference "C49")
+					(unit 1)
+				)
+			)
 		)
 	)
@@
 		(dnp no)
 		(fields_autoplaced yes)
-		(property "Reference" "U7"
+		(property "Reference" "U6"
 			(at 194.31 116.84 0)
 			(show_name no)
@@
 				)
 			)
+			(project "SuspensionBoard"
+				(path "/f9dc491a-b8c6-4623-9728-13837ac4bba3/ab14ffa7-4ae1-4464-91d5-9b05f92e5082"
+					(reference "U6")
+					(unit 1)
+				)
+			)
 		)
 	)
@@
 		(in_pos_files yes)
 		(dnp no)
-		(property "Reference" "C27"
+		(property "Reference" "C45"
 			(at 183.134 83.82 0)
 			(show_name no)
@@
 				)
 			)
+			(project "SuspensionBoard"
+				(path "/f9dc491a-b8c6-4623-9728-13837ac4bba3/ab14ffa7-4ae1-4464-91d5-9b05f92e5082"
+					(reference "C45")
+					(unit 1)
+				)
+			)
 		)
 	)
@@
 		(dnp no)
 		(fields_autoplaced yes)
-		(property "Reference" "U4"
+		(property "Reference" "U5"
 			(at 63.5 22.86 0)
 			(show_name no)
@@
 				)
 			)
+			(project "SuspensionBoard"
+				(path "/f9dc491a-b8c6-4623-9728-13837ac4bba3/ab14ffa7-4ae1-4464-91d5-9b05f92e5082"
+					(reference "U5")
+					(unit 1)
+				)
+			)
 		)
 	)
@@
 		(in_pos_files yes)
 		(dnp no)
-		(property "Reference" "R25"
+		(property "Reference" "R35"
 			(at 172.466 20.574 90)
 			(show_name no)
@@
 				)
 			)
+			(project "SuspensionBoard"
+				(path "/f9dc491a-b8c6-4623-9728-13837ac4bba3/ab14ffa7-4ae1-4464-91d5-9b05f92e5082"
+					(reference "R35")
+					(unit 1)
+				)
+			)
 		)
 	)
@@
 		(in_pos_files yes)
 		(dnp no)
-		(property "Reference" "C40"
+		(property "Reference" "C48"
 			(at 207.264 63.5 0)
 			(show_name no)
@@
 				)
 			)
+			(project "SuspensionBoard"
+				(path "/f9dc491a-b8c6-4623-9728-13837ac4bba3/ab14ffa7-4ae1-4464-91d5-9b05f92e5082"
+					(reference "C48")
+					(unit 1)
+				)
+			)
 		)
 	)
@@
 				)
 			)
+			(project "SuspensionBoard"
+				(path "/f9dc491a-b8c6-4623-9728-13837ac4bba3/ab14ffa7-4ae1-4464-91d5-9b05f92e5082"
+					(reference "R33")
+					(unit 1)
+				)
+			)
 		)
 	)
@@
 		(in_pos_files yes)
 		(dnp no)
-		(property "Reference" "#PWR020"
+		(property "Reference" "#PWR01"
 			(at 218.44 154.94 0)
 			(hide yes)
@@
 				)
 			)
+			(project "SuspensionBoard"
+				(path "/f9dc491a-b8c6-4623-9728-13837ac4bba3/ab14ffa7-4ae1-4464-91d5-9b05f92e5082"
+					(reference "#PWR01")
+					(unit 1)
+				)
+			)
 		)
 	)
@@
 		(dnp no)
 		(fields_autoplaced yes)
-		(property "Reference" "C41"
+		(property "Reference" "C43"
 			(at 96.52 24.1299 0)
 			(show_name no)
@@
 					(unit 1)
 				)
+			)
+			(project "SuspensionBoard"
+				(path "/f9dc491a-b8c6-4623-9728-13837ac4bba3/ab14ffa7-4ae1-4464-91d5-9b05f92e5082"
+					(reference "C43")
+					(unit 1)
+				)

Commit message: cleaning up for merge
Parts:
- C25: renamed from C42; value 100nF -> 100n; footprint RF_Converter:Balun_Johanson_0900PC15J0013 -> Capacitor_SMD:C_0603_1608Metric_Pad1.08x0.95mm_HandSolder
- C26: renamed from C44; value 100nF -> 100n; footprint RF_Converter:Balun_Johanson_0900PC15J0013 -> Capacitor_SMD:C_0603_1608Metric_Pad1.08x0.95mm_HandSolder
- C27: renamed from C45; value 10uF -> 10u; footprint (none) -> Capacitor_SMD:C_0603_1608Metric_Pad1.08x0.95mm_HandSolder
- C28: renamed from C49; value 1uF -> 1u; footprint (none) -> Capacitor_SMD:C_0603_1608Metric_Pad1.08x0.95mm_HandSolder
- C40: renamed from C48; value 100nF -> 100n; footprint (none) -> Capacitor_SMD:C_0603_1608Metric_Pad1.08x0.95mm_HandSolder
- C41: renamed from C43; value 10uF -> 10u
- R25: renamed from R35; footprint (none) -> Resistor_SMD:R_0603_1608Metric_Pad0.98x0.95mm_HandSolder
- R33: footprint (none) -> Resistor_SMD:R_0603_1608Metric_Pad0.98x0.95mm_HandSolder
- renumbered U5 to U4, U6 to U7
Other:
- note added: "ADD EXTERNAL SPI DAMPNING R's IF NEEDED SPI CLK: 10MHz ---> 22 Ohm RECOMMENDED"
